File: GuitarPedal1590b/pcb/SSD1306_Screen_SPI.kicad_sch (KiCad schematic)
At the start: 1 part, among them U6 OLED_DISPLAY_SSD1306_SPI

Commit message: Added some missing custom symbols and footprints
Parts:
- U6: symbol Keiths_Symbols:OLED_DISPLAY_SSD1306_SPI -> GuitarPedal1590b:OLED_DISPLAY_SSD1306_SPI
Changed lines of the file:
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@@
     )
   )
-  (symbol (lib_id "Keiths_Symbols:OLED_DISPLAY_SSD1306_SPI") (at 138.43 102.87 0) (unit 1)
+  (symbol (lib_id "GuitarPedal1590b:OLED_DISPLAY_SSD1306_SPI") (at 138.43 102.87 0) (unit 1)
     (in_bom yes) (on_board yes) (dnp no)
     (property "Reference" "U6" (at 137.16 100.33 0)
