File: GuitarPedal1590b/pcb/DaisySeedPedal1590b.kicad_pcb (KiCad board)
At the start: 2 copper layers, 54 x 106 mm, 61 parts, among them J1 Barrel_Jack, J2 AUDIO_IN_TRS, J3 AUDIO_OUT_TRS, J4 MIDI IN JACK, J5 MIDI OUT JACK, SW1 Toggle_Switch_A, SW2 Toggle_Switch_B, U1 LD1117S50TR_SOT223, U2 PDS1-S5-S5-M, U3 MCP6004, U4 OPA1652AID, U5 H11L1

Commit message: Updated project to KiCad 7
Parts:
- A1: footprint DaisySeed:Electrosmith_Daisy_Seed -> Module:Electrosmith_Daisy_Seed
- U1: footprint Package_TO_SOT_SMD:TO-252-2 -> Package_TO_SOT_SMD:TO-252-3_TabPin2
- U4: footprint OPA1652AID:SOIC127P599X175-8N -> Package_SO:SOIC-8_3.9x4.9mm_P1.27mm
- moved U1 1.60 mm to (93.0, 57.6)
Connections:
- A1 pad 7: unconnected-(A1-Pad7) -> OLED_DISPLAY_SPI_RESET
Routing:
- net +5V: track 14.1 -> 20.4 mm

Commit message: Updated resistors on LEDs to be 1K
Make them a tad dimmer!
Parts:
- R19, R20: value 220R -> 1K
Changed lines of the file:
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@@
         (effects (font (size 0.8 0.8) (thickness 0.15)))
     )
-    (fp_text value "220R" (at 3.81 0.15 90) (layer "F.Fab") hide
+    (fp_text value "1K" (at 3.81 0.15 90) (layer "F.Fab") hide
         (effects (font (size 1 1) (thickness 0.15)))
     )
@@
         (effects (font (size 0.8 0.8) (thickness 0.15)))
     )
-    (fp_text value "220R" (at 3.81 0.05 90) (layer "F.Fab") hide
-        (effects (font (size 1 1) (thickness 0.15)))
-    )
+    (fp_text value "1K" (at 3.81 0.05 90) (layer "F.Fab") hide
+        (effects (font (size 1 1) (thickness 0.15)))
+    )

Commit message: KiCad 7 fixes
Had to update some footprints and symbols to address issues related to ugprading to KiCad 7.0
Parts:
- D2: value 1N914 -> 1N4148

Commit message: Guitar Pedal 1590b Rev 3
Drastically cleaned up the PCB layout for the 1590B guitar pedal.  Updated it to be a 4 Layer board and replaced all SMD parts with through-hole parts.  Much easier to build now!
Parts:
- removed SW1: Toggle_Switch_A, Connector_PinHeader_2.54mm:PinHeader_1x03_P2.54mm_Vertical
- removed SW2: Toggle_Switch_B, Connector_PinHeader_2.54mm:PinHeader_1x03_P2.54mm_Vertical
- FS1: value Foot_Switch_A -> Foot_Switch_1
- FS2: value Foot_Switch_B -> Foot_Switch_2
- J1: footprint Connector_PinHeader_2.54mm:PinHeader_1x02_P2.54mm_Vertical -> GuitarPedal1590b:Generic_PowerJack
- LED1: value LED_A -> LED_1
- LED2: value LED_B -> LED_2
- POT1: value POT_10K_A -> 10K; footprint Connector_PinHeader_2.54mm:PinHeader_1x03_P2.54mm_Vertical -> GuitarPedal1590b:Pot_RightAngle_LongPin_16mm
- POT2: value POT_10K_B -> 10K; footprint Connector_PinHeader_2.54mm:PinHeader_1x03_P2.54mm_Vertical -> GuitarPedal1590b:Pot_RightAngle_LongPin_16mm
- POT3: value POT_10K_C -> 10K; footprint Connector_PinHeader_2.54mm:PinHeader_1x03_P2.54mm_Vertical -> GuitarPedal1590b:Pot_RightAngle_LongPin_16mm
- POT4: value POT_10K_D -> 10K; footprint Connector_PinHeader_2.54mm:PinHeader_1x03_P2.54mm_Vertical -> GuitarPedal1590b:Pot_RightAngle_LongPin_16mm
- U1: value LD1117S50TR_SOT223 -> L4931CZ50; footprint Package_TO_SOT_SMD:TO-252-3_TabPin2 -> Package_TO_SOT_THT:TO-92_Inline_Wide
- U2: value PDS1-S5-S5-M -> PDS1-S5-S5-D; footprint PDS1-S5-S5-M:CONV_PDS1-S5-S5-M -> PDS1-S5-S5-D:CONV_PDS1-S5-S5-D
- U4: value OPA1652AID -> OPA2134; footprint Package_SO:SOIC-8_3.9x4.9mm_P1.27mm -> Package_DIP:DIP-8_W7.62mm
- moved FS1 64.0 mm to (93.5, 130.0), turned to 90 degrees
- moved FS2 58.8 mm to (118.0, 130.0), turned to 90 degrees
- moved POT3 39.9 mm to (89.0, 86.0)
- moved LED2 39.5 mm to (108.3, 103.5), turned to -90 degrees
- moved POT1 33.8 mm to (89.0, 61.0)
- moved LED1 26.3 mm to (108.3, 89.5), turned to -90 degrees
- moved R19 20.9 mm to (103.2, 61.0), turned to 0 degrees
- moved U4 20.8 mm to (111.0, 119.0), turned to -90 degrees
- moved R20 18.2 mm to (103.2, 57.8), turned to 0 degrees
- moved C8 14.7 mm to (118.5, 120.0), turned to -90 degrees
- moved POT2 14.6 mm to (125.0, 61.0)
- moved J5 13.0 mm to (107.0, 30.8)
- moved POT4 12.3 mm to (125.0, 86.0)
- moved C4 11.7 mm to (87.5, 63.5)
- moved L1 11.4 mm to (93.8, 63.8)
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Connections:
- net Net-(A1-ADC_0) renamed POT_1
- net Net-(A1-ADC_1) renamed POT_2
- net Net-(A1-ADC_2) renamed POT_3
- net Net-(A1-ADC_3) renamed POT_4
- A1 pad 10: OLED_DISPLAY_SPI_DC -> unconnected-(A1-SPI1_POCI-Pad10)
- A1 pad 11: OLED_DISPLAY_SPI_MOSI -> unconnected-(A1-SPI1_PICO-Pad11)
- A1 pad 14: MIDI_OUT -> unconnected-(A1-USART1_TX-Pad14)
- A1 pad 15: MIDI_IN -> unconnected-(A1-USART1_RX-Pad15)
- A1 pad 26: Net-(A1-ADC_4) -> unconnected-(A1-ADC_4-Pad26)
- A1 pad 27: Net-(A1-ADC_5) -> unconnected-(A1-ADC_5-Pad27)
- A1 pad 29: Net-(A1-DAC_OUT2) -> LED_1
- A1 pad 30: Net-(A1-DAC_OUT1) -> LED_2
- A1 pad 31: Net-(A1-SAI2_MCLK) -> unconnected-(A1-SAI2_MCLK-Pad31)
- A1 pad 32: Net-(A1-SAI2_SD_B) -> unconnected-(A1-SAI2_SD_B-Pad32)
- A1 pad 36: unconnected-(A1-USB_D_--Pad36) -> MIDI_OUT
- A1 pad 37: unconnected-(A1-USB_D_+-Pad37) -> MIDI_IN
- A1 pad 6: unconnected-(A1-SD_CMD-Pad6) -> FOOT_SWITCH_2
- A1 pad 7: OLED_DISPLAY_SPI_RESET -> FOOT_SWITCH_1
- A1 pad 8: OLED_DISPLAY_SPI_CS -> unconnected-(A1-SPI1_CS-Pad8)
- A1 pad 9: OLED_DISPLAY_SPI_SCK -> unconnected-(A1-SPI1_SCK-Pad9)
- FS1 pad 2: Net-(A1-ADC_4) -> FOOT_SWITCH_1
- FS2 pad 2: Net-(A1-ADC_5) -> FOOT_SWITCH_2
- R19 pad 1: Net-(LED2-A) -> Net-(LED1-A)
- R19 pad 2: Net-(A1-DAC_OUT1) -> LED_1
- R20 pad 1: Net-(LED1-A) -> Net-(LED2-A)
- R20 pad 2: Net-(A1-DAC_OUT2) -> LED_2
- U1 pad 1: GND -> +5V
- U1 pad 2: +5V -> GND
- U2 pad 4: GND -> /Power/VIN
Routing:
- net FOOT_SWITCH_1: track 0.00 -> 130.3 mm
- net FOOT_SWITCH_2: track 0.00 -> 111.2 mm
- net Net-(LED2-A): track 9.30 -> 47.9 mm
- net POT_1: track 4.95 -> 37.2 mm, vias 0 -> 1
- net MIDI_OUT: track 28.3 -> 4.08 mm
- net Net-(A1-SAI2_SD_B): track 21.9 -> 0.00 mm
- net Net-(LED1-A): track 9.30 -> 29.6 mm
- net Net-(U4A--): track 11.1 -> 30.7 mm
- net MIDI_IN: track 37.5 -> 20.2 mm
- net Net-(A1-SAI2_MCLK): track 17.0 -> 0.00 mm
- net +3.3VA: track 17.0 -> 0.00 mm
- net +9V: track 47.9 -> 64.5 mm
- net POT_3: track 15.4 -> 30.4 mm
- net MIDI_OUT_JACK_PIN4: track 38.6 -> 23.7 mm
- net POT_2: track 9.85 -> 22.4 mm
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- added copper zone on In2.Cu, net +3.3V
- added copper zone on In2.Cu, net +3.3VA
- added copper zone on In2.Cu, net +5V_ISOLATED_POWER
- added copper zone on In1.Cu, net GND
- removed copper zone on F.Cu, net +3.3V
- removed copper zone on F.Cu, net +5V_ISOLATED_POWER
- removed copper zone on B.Cu, net GND
Other:
- copper layers 2 -> 4
- board text added: "Daisy Seed 1590b Guitar Pedal Made by Keith Shepherd 3/17/2023 (Rev 3)"
- board text removed: "Daisy Seed Guitar Pedal (Rev 2) Made by Keith Shepherd 1/22/2023"

Commit message: Fixed minor issue with power jack footprint
Changed lines of the file:
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@@
     (pad "2" thru_hole oval (at -6 0 270) (size 2.3 4.5) (drill oval 0.8 3) (layers "*.Cu" "*.Mask")
       (net 46 "POWER_JACK_PWR") (pintype "passive"))
-    (pad "3" thru_hole oval (at -3.125 4.65) (size 2.3 4) (drill oval 0.8 2.5) (layers "*.Cu" "*.Mask")
+    (pad "3" thru_hole oval (at -2.5 4.65) (size 2.3 4) (drill oval 0.8 2.5) (layers "*.Cu" "*.Mask")
       (net 47 "GND") (pintype "passive"))
   )
@@
   (segment (start 120.91 44.69) (end 120.91 46.225) (width 0.25) (layer "F.Cu") (net 6))
   (segment (start 114.62 40.115) (end 115.47 39.265) (width 0.25) (layer "F.Cu") (net 6))
-  (segment (start 94.4125 30.5375) (end 110.1225 30.5375) (width 0.9) (layer "F.Cu") (net 8))
-  (segment (start 89.3875 37.133084) (end 89.3875 35.5625) (width 0.9) (layer "F.Cu") (net 8))
-  (segment (start 110.1225 30.5375) (end 114.62 35.035) (width 0.9) (layer "F.Cu") (net 8))
   (segment (start 81.75 48.5) (end 81.75 49.43) (width 0.9) (layer "F.Cu") (net 8))
-  (segment (start 88.88 41.415584) (end 89.75 40.545584) (width 0.9) (layer "F.Cu") (net 8))
   (segment (start 89.75 48.5) (end 88.3 47.05) (width 0.9) (layer "F.Cu") (net 8))
-  (segment (start 89.3875 35.5625) (end 94.4125 30.5375) (width 0.9) (layer "F.Cu") (net 8))
+  (segment (start 94.491916 30.5375) (end 110.1225 30.5375) (width 0.9) (layer "F.Cu") (net 8))
   (segment (start 86.13 42.75) (end 84.5 42.75) (width 0.9) (layer "F.Cu") (net 8))
   (segment (start 88.3 47.05) (end 83.2 47.05) (width 0.9) (layer "F.Cu") (net 8))
+  (segment (start 110.1225 30.5375) (end 114.62 35.035) (width 0.9) (layer "F.Cu") (net 8))
   (segment (start 81.75 49.43) (end 85.96 53.64) (width 0.9) (layer "F.Cu") (net 8))
-  (segment (start 88.88 45.25) (end 88.88 41.415584) (width 0.9) (layer "F.Cu") (net 8))
+  (segment (start 88.88 42.040584) (end 89.5 41.420584) (width 0.9) (layer "F.Cu") (net 8))
   (segment (start 88.88 45.25) (end 88.63 45.25) (width 0.9) (layer "F.Cu") (net 8))
   (segment (start 88.88 45.25) (end 88.88 47.63) (width 0.9) (layer "F.Cu") (net 8))
-  (segment (start 89.75 37.495584) (end 89.3875 37.133084) (width 0.9) (layer "F.Cu") (net 8))
-  (segment (start 89.75 40.545584) (end 89.75 37.495584) (width 0.9) (layer "F.Cu") (net 8))
+  (segment (start 89.5 41.420584) (end 89.5 37.245584) (width 0.9) (layer "F.Cu") (net 8))
   (segment (start 83.2 47.05) (end 81.75 48.5) (width 0.9) (layer "F.Cu") (net 8))
   (segment (start 88.63 45.25) (end 86.13 42.75) (width 0.9) (layer "F.Cu") (net 8))
+  (segment (start 89.25 35.779416) (end 94.491916 30.5375) (width 0.9) (layer "F.Cu") (net 8))
+  (segment (start 89.5 37.245584) (end 89.25 36.995584) (width 0.9) (layer "F.Cu") (net 8))
+  (segment (start 89.25 36.995584) (end 89.25 35.779416) (width 0.9) (layer "F.Cu") (net 8))
   (segment (start 88.88 47.63) (end 89.75 48.5) (width 0.9) (layer "F.Cu") (net 8))
+  (segment (start 88.88 45.25) (end 88.88 42.040584) (width 0.9) (layer "F.Cu") (net 8))
   (segment (start 87.5 63.5) (end 93.5 63.5) (width 0.9) (layer "F.Cu") (net 9))
   (segment (start 86.700001 62.700001) (end 86.700001 57.979999) (width 0.9) (layer "F.Cu") (net 9))

Commit message: Updated 1590b PCB layout (Rev 4)
Updated the layout of the PCB to move some of the components a little farther from the edge of the PCB.  Also swapped the locations of the LEDs to be more consistent with my other projects.  FS1 and LED1 are now the default for enabling and disabling the effect.
Parts:
- moved R16 22.0 mm to (103.2, 45.0), turned to 0 degrees
- moved R17 15.2 mm to (103.2, 48.2), turned to 0 degrees
- moved LED1 14.0 mm to (108.3, 103.5)
- moved LED2 14.0 mm to (108.3, 89.5)
- moved D2 10.8 mm to (122.2, 44.4), turned to 0 degrees
- moved C17 8.51 mm to (123.5, 55.8), turned to 0 degrees
- moved U5 8.15 mm to (129.8, 52.5), turned to 180 degrees
- moved C3 6.25 mm to (88.0, 48.5), turned to 180 degrees
- moved R15 4.27 mm to (125.2, 33.8), turned to -90 degrees
- moved C1 2.55 mm to (84.0, 45.2)
- moved R18 2.14 mm to (119.2, 53.6)
- moved C2 1.25 mm to (91.0, 48.5)
- moved C4 1.25 mm to (88.8, 63.5)
- moved C5 1.25 mm to (88.8, 67.0)
- moved R1 1.13 mm to (121.2, 108.0)
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Routing:
- net Net-(LED2-A): track 47.9 -> 32.8 mm
- net Net-(LED1-A): track 29.6 -> 43.6 mm
- net MIDI_OUT_JACK_PIN4: track 23.7 -> 11.7 mm
- net MIDI_IN: track 20.2 -> 11.3 mm
- net Net-(D2-K): track 6.83 -> 15.5 mm
- net MIDI_IN_JACK_PIN5: track 8.84 -> 16.1 mm
- net +9V: track 64.3 -> 57.2 mm
- net MIDI_OUT_JACK_PIN5: track 15.8 -> 10.3 mm
- net MIDI_OUT: track 4.08 -> 7.12 mm
- net POT_1: track 37.2 -> 34.9 mm
- net Net-(U3D-+): track 24.8 -> 26.5 mm
- net FOOT_SWITCH_1: track 130.3 -> 131.7 mm
- net MIDI_IN_JACK_PIN4: track 2.95 -> 4.00 mm
- net /Power/VIN: track 20.9 -> 19.9 mm
- net AUDIO_IN_JACK_LEFT: track 26.6 -> 25.6 mm
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Other:
- board text added: "Daisy Seed 1590b Guitar Pedal Made by Keith Shepherd 4/12/2023 (Rev 4)"
- board text removed: "Daisy Seed 1590b Guitar Pedal Made by Keith Shepherd 3/17/2023 (Rev 3)"

Commit message: Switched LED and FS placement on the 125B pcb layout
Parts:
- moved FS1 24.5 mm to (118.0, 130.0)
- moved FS2 24.5 mm to (93.5, 130.0)
- moved LED2 2.57 mm to (105.7, 89.5), turned to 90 degrees
- moved LED1 2.54 mm to (105.8, 103.5), turned to 90 degrees
Routing:
- net FOOT_SWITCH_2: track 111.7 -> 137.1 mm
- net FOOT_SWITCH_1: track 131.7 -> 107.2 mm
- net Net-(LED1-A): track 43.6 -> 44.6 mm
- net Net-(LED2-A): track 32.8 -> 33.9 mm
Changed lines of the file:
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@@
   )
   (footprint "Connector_PinHeader_2.54mm:PinHeader_1x02_P2.54mm_Vertical" (layer "F.Cu")
-    (at 108.29 103.5 -90)
+    (at 105.75 103.5 90)
     (descr "Through hole straight pin header, 1x02, 2.54mm pitch, single row")
     (tags "Through hole pin header THT 1x02 2.54mm single row")
@@
     (property "ki_keywords" "LED diode")
     (attr through_hole)
-    (fp_text reference "LED1" (at 2.5 1.29) (layer "F.SilkS")
+    (fp_text reference "LED1" (at -2.5 1.25) (layer "F.SilkS")
         (effects (font (size 1 1) (thickness 0.15)))
     )
@@
     (fp_line (start 1.27 3.81) (end -1.27 3.81)
       (stroke (width 0.1) (type solid)) (layer "F.Fab"))
-    (pad "1" thru_hole rect (at 0 0 270) (size 1.7 1.7) (drill 1) (layers "*.Cu" "*.Mask")
+    (pad "1" thru_hole rect (at 0 0 90) (size 1.7 1.7) (drill 1) (layers "*.Cu" "*.Mask")
       (net 47 "GND") (pinfunction "K") (pintype "passive"))
-    (pad "2" thru_hole oval (at 0 2.54 270) (size 1.7 1.7) (drill 1) (layers "*.Cu" "*.Mask")
+    (pad "2" thru_hole oval (at 0 2.54 90) (size 1.7 1.7) (drill 1) (layers "*.Cu" "*.Mask")
       (net 69 "Net-(LED1-A)") (pinfunction "A") (pintype "passive"))
     (model "${KICAD6_3DMODEL_DIR}/Connector_PinHeader_2.54mm.3dshapes/PinHeader_1x02_P2.54mm_Vertical.wrl"
@@
   )
   (footprint "Connector_PinHeader_2.54mm:PinHeader_1x02_P2.54mm_Vertical" (layer "F.Cu")
-    (at 118 130 90)
+    (at 93.5 130 90)
     (descr "Through hole straight pin header, 1x02, 2.54mm pitch, single row")
     (tags "Through hole pin header THT 1x02 2.54mm single row")
@@
   )
   (footprint "Connector_PinHeader_2.54mm:PinHeader_1x02_P2.54mm_Vertical" (layer "F.Cu")
-    (at 108.29 89.5 -90)
+    (at 105.725 89.5 90)
     (descr "Through hole straight pin header, 1x02, 2.54mm pitch, single row")
     (tags "Through hole pin header THT 1x02 2.54mm single row")
@@
     (property "ki_keywords" "LED diode")
     (attr through_hole)
-    (fp_text reference "LED2" (at -2.5 1.29) (layer "F.SilkS")
+    (fp_text reference "LED2" (at 2.5 1.29) (layer "F.SilkS")
         (effects (font (size 1 1) (thickness 0.15)))
     )
@@
     (fp_line (start 1.27 3.81) (end -1.27 3.81)
       (stroke (width 0.1) (type solid)) (layer "F.Fab"))
-    (pad "1" thru_hole rect (at 0 0 270) (size 1.7 1.7) (drill 1) (layers "*.Cu" "*.Mask")
+    (pad "1" thru_hole rect (at 0 0 90) (size 1.7 1.7) (drill 1) (layers "*.Cu" "*.Mask")
       (net 47 "GND") (pinfunction "K") (pintype "passive"))
-    (pad "2" thru_hole oval (at 0 2.54 270) (size 1.7 1.7) (drill 1) (layers "*.Cu" "*.Mask")
+    (pad "2" thru_hole oval (at 0 2.54 90) (size 1.7 1.7) (drill 1) (layers "*.Cu" "*.Mask")
       (net 70 "Net-(LED2-A)") (pinfunction "A") (pintype "passive"))
     (model "${KICAD6_3DMODEL_DIR}/Connector_PinHeader_2.54mm.3dshapes/PinHeader_1x02_P2.54mm_Vertical.wrl"
@@
   )
   (footprint "Connector_PinHeader_2.54mm:PinHeader_1x02_P2.54mm_Vertical" (layer "F.Cu")
-    (at 93.46 130 90)
+    (at 118 130 90)
     (descr "Through hole straight pin header, 1x02, 2.54mm pitch, single row")
     (tags "Through hole pin header THT 1x02 2.54mm single row")
@@
     (effects (font (size 1 1) (thickness 0.15)))
   )
-  (segment (start 105.863299 50.8) (end 104.199009 50.8) (width 0.25) (layer "B.Cu") (net 1))
-  (segment (start 131.85 129.15) (end 133.25 127.75) (width 0.25) (layer "B.Cu") (net 1))
+  (segment (start 104.199009 50.8) (end 99.38 45.980991) (width 0.25) (layer "B.Cu") (net 1))
   (segment (start 133.25 77.403299) (end 114.916701 59.07) (width 0.25) (layer "B.Cu") (net 1))
-  (segment (start 114.133299 59.07) (end 105.863299 50.8) (width 0.25) (layer "B.Cu") (net 1))
+  (segment (start 131.85 129.15) (end 133.25 127.75) (width 0.25) (layer "B.Cu") (net 1))
   (segment (start 114.916701 59.07) (end 114.133299 59.07) (width 0.25) (layer "B.Cu") (net 1))
   (segment (start 133.25 127.75) (end 133.25 77.403299) (width 0.25) (layer "B.Cu") (net 1))
-  (segment (start 120.54 130) (end 121.39 129.15) (width 0.25) (layer "B.Cu") (net 1))
+  (segment (start 126.25 129.15) (end 131.85 129.15) (width 0.25) (layer "B.Cu") (net 1))
+  (segment (start 124.225 131.175) (end 126.25 129.15) (width 0.25) (layer "B.Cu") (net 1))
+  (segment (start 96.04 130) (end 97.215 131.175) (width 0.25) (layer "B.Cu") (net 1))
+  (segment (start 105.863299 50.8) (end 104.199009 50.8) (width 0.25) (layer "B.Cu") (net 1))
+  (segment (start 97.215 131.175) (end 124.225 131.175) (width 0.25) (layer "B.Cu") (net 1))
+  (segment (start 114.133299 59.07) (end 105.863299 50.8) (width 0.25) (layer "B.Cu") (net 1))
   (segment (start 99.38 45.980991) (end 99.38 45.195) (width 0.25) (layer "B.Cu") (net 1))
-  (segment (start 121.39 129.15) (end 131.85 129.15) (width 0.25) (layer "B.Cu") (net 1))
-  (segment (start 104.199009 50.8) (end 99.38 45.980991) (width 0.25) (layer "B.Cu") (net 1))
-  (segment (start 130.225991 128.675) (end 97.325 128.675) (width 0.25) (layer "B.Cu") (net 2))
-  (segment (start 114.916701 61.61) (end 132.8 79.493299) (width 0.25) (layer "B.Cu") (net 2))
-  (segment (start 99.38 47.910991) (end 113.079009 61.61) (width 0.25) (layer "B.Cu") (net 2))
-  (segment (start 132.8 126.100991) (end 130.225991 128.675) (width 0.25) (layer "B.Cu") (net 2))
-  (segment (start 97.325 128.675) (end 96 130) (width 0.25) (layer "B.Cu") (net 2))
-  (segment (start 113.079009 61.61) (end 114.916701 61.61) (width 0.25) (layer "B.Cu") (net 2))
   (segment (start 99.38 47.735) (end 99.38 47.910991) (width 0.25) (layer "B.Cu") (net 2))
+  (segment (start 121.865 128.675) (end 120.54 130) (width 0.25) (layer "B.Cu") (net 2))
+  (segment (start 130.225991 128.675) (end 121.865 128.675) (width 0.25) (layer "B.Cu") (net 2))
+  (segment (start 132.8 126.100991) (end 130.225991 128.675) (width 0.25) (layer "B.Cu") (net 2))
+  (segment (start 114.916701 61.61) (end 132.8 79.493299) (width 0.25) (layer "B.Cu") (net 2))
   (segment (start 132.8 79.493299) (end 132.8 126.100991) (width 0.25) (layer "B.Cu") (net 2))
+  (segment (start 113.079009 61.61) (end 114.916701 61.61) (width 0.25) (layer "B.Cu") (net 2))
+  (segment (start 99.38 47.910991) (end 113.079009 61.61) (width 0.25) (layer "B.Cu") (net 2))
   (segment (start 110.81 47.06863) (end 114.62 43.25863) (width 0.25) (layer "F.Cu") (net 5))
   (segment (start 110.81 48.2) (end 110.81 47.06863) (width 0.25) (layer "F.Cu") (net 5))
@@
   (segment (start 129.8 52.525) (end 129.8 52) (width 0.25) (layer "F.Cu") (net 68))
   (segment (start 122.22 44.4) (end 125.2 41.42) (width 0.25) (layer "F.Cu") (net 68))
-  (segment (start 104.575 102.325) (end 104.575 65.325) (width 0.25) (layer "F.Cu") (net 69))
-  (segment (start 105.75 103.5) (end 104.575 102.325) (width 0.25) (layer "F.Cu") (net 69))
-  (segment (start 103.19 63.94) (end 104.575 65.325) (width 0.25) (layer "F.Cu") (net 69))
-  (segment (start 103.19 61) (end 103.19 63.94) (width 0.25) (layer "F.Cu") (net 69))
-  (segment (start 105.75 60.31) (end 105.75 89.5) (width 0.25) (layer "F.Cu") (net 70))
-  (segment (start 103.19 57.75) (end 105.75 60.31) (width 0.25) (layer "F.Cu") (net 70))
+  (segment (start 104.25 62.06) (end 104.25 99.46) (width 0.25) (layer "F.Cu") (net 69))
+  (segment (start 103.19 61) (end 104.25 62.06) (width 0.25) (layer "F.Cu") (net 69))
+  (segment (start 104.25 99.46) (end 108.29 103.5) (width 0.25) (layer "F.Cu") (net 69))
+  (segment (start 103.19 57.75) (end 108.265 62.825) (width 0.25) (layer "F.Cu") (net 70))
+  (segment (start 108.265 62.825) (end 108.265 89.5) (width 0.25) (layer "F.Cu") (net 70))
   (segment (start 120.844009 127.435) (end 118.625 125.215991) (width 0.25) (layer "F.Cu") (net 71))
   (segment (start 127.75 126.25) (end 126.565 127.435) (width 0.25) (layer "F.Cu") (net 71))

Commit message: Minor updates to PCB
Parts:
- moved J2 0.25 mm to (120.8, 96.5)
- moved J3 0.25 mm to (93.2, 96.5)
Routing:
- net +3.3VA: track 0.00 -> 89.3 mm, vias 0 -> 1
- net POT_4: track 18.4 -> 59.0 mm
- net +3.3V: track 0.00 -> 38.1 mm
- net POT_3: track 30.4 -> 68.2 mm
- net +5V_ISOLATED_POWER: track 16.2 -> 40.3 mm, vias 1 -> 0
- net FOOT_SWITCH_1: track 107.2 -> 119.3 mm
- net FOOT_SWITCH_2: track 137.1 -> 148.2 mm
- net POT_1: track 34.9 -> 42.2 mm, vias 1 -> 0
- net Net-(LED1-A): track 44.6 -> 46.8 mm
- net POT_2: track 22.4 -> 20.3 mm
- net Net-(LED2-A): track 33.9 -> 35.7 mm
- net Net-(U3D-+): track 26.5 -> 25.9 mm
- net MIDI_OUT_JACK_PIN4: track 11.7 -> 11.1 mm
- net GND: vias 0 -> 1
- added copper zone on F.Cu, net +5V_ISOLATED_POWER
- added copper zone on In2.Cu, net GND
- removed copper zone on In2.Cu, net +3.3V
- removed copper zone on In2.Cu, net +3.3VA
- removed copper zone on In2.Cu, net +5V_ISOLATED_POWER
Other:
- board text added: "Daisy Seed 1590b Guitar Pedal Made by Keith Shepherd 5/23/2023 (Rev 4)"
- board text removed: "Daisy Seed 1590b Guitar Pedal Made by Keith Shepherd 4/12/2023 (Rev 4)"
