File: GuitarPedal1590b/pcb/DaisySeedPedal1590b.kicad_pcb (KiCad board)
At the start: 4 copper layers, 54 x 106 mm, 59 parts, among them J1 Barrel_Jack, J2 AUDIO_IN_TRS, J3 AUDIO_OUT_TRS, J4 MIDI IN JACK, J5 MIDI OUT JACK, U1 L4931CZ50, U2 PDS1-S5-S5-D, U3 MCP6004, U4 OPA2134, U5 H11L1

Commit message: Updated 1590B PCB and software
Updated the PCB to properly ground the inputs and outputs when no plug is inserted in the jack.  Fixed a noise issue caused by having the LED update function in the main loop instead of the audio callback.
Connections:
- J2 pad RN: unconnected-(J2-PadRN) -> GND
- J2 pad TN: unconnected-(J2-PadTN) -> GND
- J3 pad RN: unconnected-(J3-PadRN) -> GND
- J3 pad TN: unconnected-(J3-PadTN) -> GND
Other:
- board text added: "Daisy Seed 1590b Guitar Pedal Made by Keith Shepherd 6/3/2023 (Rev 5)"
- board text removed: "Daisy Seed 1590b Guitar Pedal Made by Keith Shepherd 5/23/2023 (Rev 4)"
