File: GuitarPedal1590b/pcb/DaisySeedPedal1590b.kicad_sch (KiCad schematic)
At the start: 18 parts, among them J1 Barrel_Jack, J2 AUDIO_IN_TRS, J3 AUDIO_OUT_TRS, J4 MIDI IN JACK, J5 MIDI OUT JACK, SW1 Toggle_Switch_A, SW2 Toggle_Switch_B

Commit message: Updated project to KiCad 7
Parts:
- A1: footprint DaisySeed:Electrosmith_Daisy_Seed -> Module:Electrosmith_Daisy_Seed
Connections:
- net OLED_DISPLAY_SPI_RESET: now also A1.7 (SDMMC1_CK)

Commit message: Updated resistors on LEDs to be 1K
Make them a tad dimmer!
Parts:
- R19, R20: value 220R -> 1K
Changed lines of the file:
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@@
       (effects (font (size 1.27 1.27)))
     )
-    (property "Value" "220R" (at 72.39 111.76 90)
+    (property "Value" "1K" (at 72.39 111.76 90)
       (effects (font (size 1.27 1.27)))
     )
@@
       (effects (font (size 1.27 1.27)))
     )
-    (property "Value" "220R" (at 45.72 116.84 90)
-      (effects (font (size 1.27 1.27)))
-    )
+    (property "Value" "1K" (at 45.72 116.84 90)
+      (effects (font (size 1.27 1.27)))
+    )

Commit message: KiCad 7 fixes
Had to update some footprints and symbols to address issues related to ugprading to KiCad 7.0
Parts:
- A1: symbol Electrosmith_Daisy_Seed:Electrosmith_Daisy_Seed_Rev4 -> MCU_Module:Electrosmith_Daisy_Seed_Rev4
- J4, J5: symbol Connector:AudioJack4 -> Connector_Audio:AudioJack4
Changed lines of the file:
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@@
     )
   )
-  (symbol (lib_id "Electrosmith_Daisy_Seed:Electrosmith_Daisy_Seed_Rev4") (at 152.4 95.25 0) (unit 1)
+  (symbol (lib_id "MCU_Module:Electrosmith_Daisy_Seed_Rev4") (at 152.4 95.25 0) (unit 1)
     (in_bom yes) (on_board yes) (dnp no) (fields_autoplaced)
     (property "Reference" "A1" (at 156.9594 130.81 0)
@@
     )
   )
-  (symbol (lib_id "Connector:AudioJack4") (at 236.22 148.59 180) (unit 1)
+  (symbol (lib_id "Connector_Audio:AudioJack4") (at 236.22 148.59 180) (unit 1)
     (in_bom yes) (on_board yes) (dnp no) (fields_autoplaced)
     (property "Reference" "J5" (at 238.76 157.48 0)
       (effects (font (size 1.27 1.27)))
     )
-    (property "Value" "MIDI OUT JACK" (at 238.76 154.94 0)
+    (property "Value" "MIDI OUT JACK" (at 236.22 154.94 0)
       (effects (font (size 1.27 1.27)))
     )
@@
     )
   )
-  (symbol (lib_id "power:GND") (at 227.33 99.06 0) (unit 1)
-    (in_bom yes) (on_board yes) (dnp no) (fields_autoplaced)
-    (property "Reference" "#PWR0110" (at 227.33 105.41 0)
-      (effects (font (size 1.27 1.27)) hide)
-    )
-    (property "Value" "GND" (at 227.33 104.14 0)
-      (effects (font (size 1.27 1.27)))
-    )
-    (property "Footprint" "" (at 227.33 99.06 0)
-      (effects (font (size 1.27 1.27)) hide)
-    )
-    (property "Datasheet" "" (at 227.33 99.06 0)
-      (effects (font (size 1.27 1.27)) hide)
-    )
-    (pin "1")
-    (instances
-      (project "DaisySeedPedal1590b"
-        (path "/1d54e6f4-7c7a-4f03-b2db-a136bdff5b99"
-          (reference "#PWR0110") (unit 1)
-        )
-      )
-    )
-  )
   (symbol (lib_id "power:GND") (at 73.66 83.82 90) (unit 1)
     (in_bom yes) (on_board yes) (dnp no) (fields_autoplaced)
@@
         (path "/1d54e6f4-7c7a-4f03-b2db-a136bdff5b99"
           (reference "#PWR0108") (unit 1)
+        )
+      )
+    )
+  )
+  (symbol (lib_id "power:GND") (at 227.33 99.06 0) (unit 1)
+    (in_bom yes) (on_board yes) (dnp no) (fields_autoplaced)
+    (property "Reference" "#PWR018" (at 227.33 105.41 0)
+      (effects (font (size 1.27 1.27)) hide)
+    )
+    (property "Value" "GND" (at 227.33 102.87 0)
+      (effects (font (size 1.27 1.27)))
+    )
+    (property "Footprint" "" (at 227.33 99.06 0)
+      (effects (font (size 1.27 1.27)) hide)
+    )
+    (property "Datasheet" "" (at 227.33 99.06 0)
+      (effects (font (size 1.27 1.27)) hide)
+    )
+    (pin "1")
+    (instances
+      (project "DaisySeedPedal1590b"
+        (path "/1d54e6f4-7c7a-4f03-b2db-a136bdff5b99"
+          (reference "#PWR018") (unit 1)
         )
       )
@@
     )
   )
-  (symbol (lib_id "Connector:AudioJack4") (at 220.98 121.92 0) (mirror x) (unit 1)
+  (symbol (lib_id "Connector_Audio:AudioJack4") (at 220.98 121.92 0) (mirror x) (unit 1)
     (in_bom yes) (on_board yes) (dnp no) (fields_autoplaced)
     (property "Reference" "J4" (at 218.44 130.81 0)

Commit message: Guitar Pedal 1590b Rev 3
Drastically cleaned up the PCB layout for the 1590B guitar pedal.  Updated it to be a 4 Layer board and replaced all SMD parts with through-hole parts.  Much easier to build now!
Parts:
- removed FS1: Foot_Switch_A, Connector_PinHeader_2.54mm:PinHeader_1x02_P2.54mm_Vertical, symbol Switch:SW_Push
- removed FS2: Foot_Switch_B, Connector_PinHeader_2.54mm:PinHeader_1x02_P2.54mm_Vertical, symbol Switch:SW_Push
- removed LED1: LED_A, Connector_PinHeader_2.54mm:PinHeader_1x02_P2.54mm_Vertical, symbol Device:LED
- removed LED2: LED_B, Connector_PinHeader_2.54mm:PinHeader_1x02_P2.54mm_Vertical, symbol Device:LED
- removed POT1: POT_10K_A, Connector_PinHeader_2.54mm:PinHeader_1x03_P2.54mm_Vertical, symbol Device:R_Potentiometer_US
- removed POT2: POT_10K_B, Connector_PinHeader_2.54mm:PinHeader_1x03_P2.54mm_Vertical, symbol Device:R_Potentiometer_US
- removed POT3: POT_10K_C, Connector_PinHeader_2.54mm:PinHeader_1x03_P2.54mm_Vertical, symbol Device:R_Potentiometer_US
- removed POT4: POT_10K_D, Connector_PinHeader_2.54mm:PinHeader_1x03_P2.54mm_Vertical, symbol Device:R_Potentiometer_US
- removed R19, R20: 1K, Resistor_THT:R_Axial_DIN0207_L6.3mm_D2.5mm_P7.62mm_Horizontal, symbol Device:R
- removed SW1: Toggle_Switch_A, Connector_PinHeader_2.54mm:PinHeader_1x03_P2.54mm_Vertical, symbol Switch:SW_SPDT
- removed SW2: Toggle_Switch_B, Connector_PinHeader_2.54mm:PinHeader_1x03_P2.54mm_Vertical, symbol Switch:SW_SPDT
- J1: footprint Connector_PinHeader_2.54mm:PinHeader_1x02_P2.54mm_Vertical -> GuitarPedal1590b:Generic_PowerJack; symbol Connector:Barrel_Jack -> Connector:Barrel_Jack_Switch
Connections:
- net GND: now also J1.3
- net MIDI_IN: now also A1.37 (USB_D_+); no longer A1.15 (USART1_RX)
- net MIDI_OUT: now also A1.36 (USB_D_-); no longer A1.14 (USART1_TX)
- net POT_1: now reaches A1.22 (ADC_0)
- net POT_2: now reaches A1.23 (ADC_1)
- net POT_3: now reaches A1.24 (ADC_2)
- net POT_4: now reaches A1.25 (ADC_3)
- net LED_1: now reaches A1.29 (DAC_OUT2)
- net LED_2: now reaches A1.30 (DAC_OUT1)
- net FOOT_SWITCH_2: now reaches A1.6 (SD_CMD)
- net OLED_DISPLAY_SPI_CS: no longer names the net of A1.8 (SPI1_CS)
- net OLED_DISPLAY_SPI_DC: no longer names the net of A1.10 (SPI1_POCI)
- net OLED_DISPLAY_SPI_MOSI: no longer names the net of A1.11 (SPI1_PICO)
- net OLED_DISPLAY_SPI_RESET renamed FOOT_SWITCH_1
- net OLED_DISPLAY_SPI_SCK: no longer names the net of A1.9 (SPI1_SCK)
- no-connect marks 20 -> 27
Other:
- removed sheet SSD1306 Screen SPI
- added sheet Controls (Controls.kicad_sch)

Commit message: Updated 1590B PCB and software
Updated the PCB to properly ground the inputs and outputs when no plug is inserted in the jack.  Fixed a noise issue caused by having the LED update function in the main loop instead of the audio callback.
Connections:
- net GND: now also J2.RN, J2.TN, J3.RN, J3.TN
- no-connect marks 27 -> 23
Changed lines of the file:
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@@
   (title_block
     (title "Daisy Seed Guitar Pedal 1590B")
-    (date "2023-04-12")
-    (rev "4")
+    (date "2023-06-03")
+    (rev "5")
     (company "Made by Keith Shepherd (kshep@mac.com)")
     (comment 1 "https://github.com/electro-smith/Hardware/blob/master/reference/daisy_petal/")
     (comment 2 "Schematic loosly based on the Electro-Smith Daisy Petal Reference Hardware Rev 5")
   )
+  (junction (at 231.14 67.31) (diameter 0) (color 0 0 0 0)
+  )
   (junction (at 231.14 69.85) (diameter 0) (color 0 0 0 0)
+  )
+  (junction (at 231.14 88.9) (diameter 0) (color 0 0 0 0)
   )
   (junction (at 152.4 133.35) (diameter 0) (color 0 0 0 0)
   )
   (junction (at 236.22 39.37) (diameter 0) (color 0 0 0 0)
+  )
+  (junction (at 231.14 62.23) (diameter 0) (color 0 0 0 0)
+  )
+  (junction (at 231.14 93.98) (diameter 0) (color 0 0 0 0)
   )
   (junction (at 231.14 96.52) (diameter 0) (color 0 0 0 0)
@@
   (no_connect (at 127 118.11))
   (no_connect (at 177.8 102.87))
-  (no_connect (at 231.14 83.82))
-  (no_connect (at 231.14 57.15))
   (no_connect (at 127 97.79))
   (no_connect (at 127 95.25))
   (no_connect (at 177.8 90.17))
   (no_connect (at 177.8 82.55))
-  (no_connect (at 231.14 88.9))
   (no_connect (at 177.8 113.03))
   (no_connect (at 177.8 97.79))
@@
   (no_connect (at 177.8 100.33))
   (no_connect (at 177.8 115.57))
-  (no_connect (at 231.14 62.23))
   (no_connect (at 177.8 110.49))
   (no_connect (at 127 100.33))
@@
   )
   (wire (pts (xy 226.06 36.83) (xy 227.33 36.83))
+    (stroke (width 0) (type default))
+  )
+  (wire (pts (xy 231.14 88.9) (xy 231.14 93.98))
     (stroke (width 0) (type default))
   )
@@
     (stroke (width 0) (type default))
   )
+  (wire (pts (xy 231.14 83.82) (xy 231.14 88.9))
+    (stroke (width 0) (type default))
+  )
   (wire (pts (xy 234.95 69.85) (xy 234.95 72.39))
     (stroke (width 0) (type default))
@@
   )
   (wire (pts (xy 236.22 39.37) (xy 248.92 39.37))
+    (stroke (width 0) (type default))
+  )
+  (wire (pts (xy 231.14 57.15) (xy 231.14 62.23))
     (stroke (width 0) (type default))
   )
@@
     (stroke (width 0) (type default))
   )
+  (wire (pts (xy 231.14 62.23) (xy 231.14 67.31))
+    (stroke (width 0) (type default))
+  )
