File: GuitarPedal1590b/pcb/Midi_InOut.kicad_sch (KiCad schematic)
At the start: 7 parts, among them U5 H11L1

Commit message: KiCad 7 fixes
Had to update some footprints and symbols to address issues related to ugprading to KiCad 7.0
Parts:
- D2: value 1N914 -> 1N4148; symbol Diode:1N914 -> Diode:1N4148
Changed lines of the file:
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@@
     )
   )
-  (symbol (lib_id "Diode:1N914") (at 127 95.25 270) (unit 1)
+  (symbol (lib_id "Diode:1N4148") (at 127 95.25 270) (unit 1)
     (in_bom yes) (on_board yes) (dnp no) (fields_autoplaced)
     (property "Reference" "D2" (at 129.54 93.9799 90)
       (effects (font (size 1.27 1.27)) (justify left))
     )
-    (property "Value" "1N914" (at 129.54 96.5199 90)
+    (property "Value" "1N4148" (at 129.54 96.5199 90)
       (effects (font (size 1.27 1.27)) (justify left))
     )
-    (property "Footprint" "Diode_THT:D_DO-35_SOD27_P7.62mm_Horizontal" (at 122.555 95.25 0)
+    (property "Footprint" "Diode_THT:D_DO-35_SOD27_P7.62mm_Horizontal" (at 127 95.25 0)
       (effects (font (size 1.27 1.27)) hide)
     )
-    (property "Datasheet" "http://www.vishay.com/docs/85622/1n914.pdf" (at 127 95.25 0)
+    (property "Datasheet" "https://assets.nexperia.com/documents/data-sheet/1N4148_1N4448.pdf" (at 127 95.25 0)
       (effects (font (size 1.27 1.27)) hide)
     )
