File: GuitarPedal1590b/pcb/Power.kicad_sch (KiCad schematic)
At the start: 10 parts, among them U1 LD1117S50TR_SOT223, U2 PDS1-S5-S5-M

Commit message: Updated project to KiCad 7
Parts:
- U1: footprint Package_TO_SOT_SMD:TO-252-2 -> Package_TO_SOT_SMD:TO-252-3_TabPin2

Commit message: KiCad 7 fixes
Had to update some footprints and symbols to address issues related to ugprading to KiCad 7.0
Changed lines of the file:
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@@
-    (effects (font (size 1.27 1.27)) (justify left bottom))
-  )
-  (label "EXT_PWR" (at 48.26 100.33 0) (fields_autoplaced)
     (effects (font (size 1.27 1.27)) (justify left bottom))
   )
@@
       (effects (font (size 1.27 1.27)) hide)
     )
+    (property "Sim.Device" "D" (at 68.58 100.33 0)
+      (effects (font (size 1.27 1.27)) hide)
+    )
+    (property "Sim.Pins" "1=K 2=A" (at 68.58 100.33 0)
+      (effects (font (size 1.27 1.27)) hide)
+    )
     (pin "1")
     (pin "2")
@@
   (symbol (lib_id "PDS1-S5-S5-M:PDS1-S5-S5-M") (at 176.53 102.87 0) (unit 1)
     (in_bom yes) (on_board yes) (dnp no) (fields_autoplaced)
-    (property "Reference" "U2" (at 176.53 90.17 0)
-      (effects (font (size 1.27 1.27)))
-    )
-    (property "Value" "PDS1-S5-S5-M" (at 176.53 92.71 0)
-      (effects (font (size 1.27 1.27)))
-    )
+    (property "Reference" "U2" (at 176.53 91.44 0)
+      (effects (font (size 1.27 1.27)))
+    )
+    (property "Value" "PDS1-S5-S5-M" (at 176.53 93.98 0)
+      (effects (font (size 1.27 1.27)))
+    )

Commit message: Guitar Pedal 1590b Rev 3
Drastically cleaned up the PCB layout for the 1590B guitar pedal.  Updated it to be a 4 Layer board and replaced all SMD parts with through-hole parts.  Much easier to build now!
Parts:
- U1: value LD1117S50TR_SOT223 -> L4931CZ50; footprint Package_TO_SOT_SMD:TO-252-3_TabPin2 -> Package_TO_SOT_THT:TO-92_Inline_Wide; symbol Regulator_Linear:LD1117S50TR_SOT223 -> Regulator_Linear:L78L05_TO92
- U2: value PDS1-S5-S5-M -> PDS1-S5-S5-D; footprint PDS1-S5-S5-M:CONV_PDS1-S5-S5-M -> PDS1-S5-S5-D:CONV_PDS1-S5-S5-D; symbol PDS1-S5-S5-M:PDS1-S5-S5-M -> PDS1-S5-S5-D:PDS1-S5-S5-D; DESCRIPTION PDS1 Series 1 W 12 VDC 84 mA Surface Mount DC-DC Isolated C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 -> Module DC-DC 12VIN 1-OUT 12V 0.083A 1W 4-Pin DIP; MP PDS1-S12-S12-M -> PDS1-S12-S12-D; PACKAGE SMD-8 CUI -> DIP-7 CUI; PRICE 4.02 USD -> 3.88 USD
Connections:
- net +5V: now also U1.1 (VO); no longer U1.2 (VO)
- net GND: now also U1.2 (GND), U2.7 (0V); no longer U1.1 (GND), U2.4 (0V)
- net VIN: now also U2.4 (VIN); no longer U2.2 (VIN)
Changed lines of the file:
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@@
   (title_block
     (title "Daisy Seed Guitar Pedal 1590B")
-    (date "2023-01-22")
-    (rev "2")
+    (date "2023-03-17")
+    (rev "3")
     (company "Made by Keith Shepherd (kshep@mac.com)")
     (comment 1 "https://github.com/electro-smith/Hardware/blob/master/reference/daisy_petal/")
@@
     )
   )
-  (symbol (lib_id "Regulator_Linear:LD1117S50TR_SOT223") (at 118.11 100.33 0) (unit 1)
+  (symbol (lib_id "Regulator_Linear:L78L05_TO92") (at 118.11 100.33 0) (unit 1)
     (in_bom yes) (on_board yes) (dnp no) (fields_autoplaced)
     (property "Reference" "U1" (at 118.11 92.71 0)
       (effects (font (size 1.27 1.27)))
     )
-    (property "Value" "LD1117S50TR_SOT223" (at 118.11 95.25 0)
-      (effects (font (size 1.27 1.27)))
-    )
-    (property "Footprint" "Package_TO_SOT_SMD:TO-252-3_TabPin2" (at 118.11 95.25 0)
-      (effects (font (size 1.27 1.27)) hide)
-    )
-    (property "Datasheet" "http://www.st.com/st-web-ui/static/active/en/resource/technical/document/datasheet/CD00000544.pdf" (at 120.65 106.68 0)
+    (property "Value" "L4931CZ50" (at 118.11 95.25 0)
+      (effects (font (size 1.27 1.27)))
+    )
+    (property "Footprint" "Package_TO_SOT_THT:TO-92_Inline_Wide" (at 118.11 94.615 0)
+      (effects (font (size 1.27 1.27) italic) hide)
+    )
+    (property "Datasheet" "http://www.st.com/content/ccc/resource/technical/document/datasheet/15/55/e5/aa/23/5b/43/fd/CD00000446.pdf/files/CD00000446.pdf/jcr:content/translations/en.CD00000446.pdf" (at 118.11 101.6 0)
       (effects (font (size 1.27 1.27)) hide)
     )
@@
     )
   )
-  (symbol (lib_id "PDS1-S5-S5-M:PDS1-S5-S5-M") (at 176.53 102.87 0) (unit 1)
+  (symbol (lib_id "PDS1-S5-S5-D:PDS1-S5-S5-D") (at 176.53 102.87 0) (unit 1)
     (in_bom yes) (on_board yes) (dnp no) (fields_autoplaced)
     (property "Reference" "U2" (at 176.53 91.44 0)
       (effects (font (size 1.27 1.27)))
     )
-    (property "Value" "PDS1-S5-S5-M" (at 176.53 93.98 0)
-      (effects (font (size 1.27 1.27)))
-    )
-    (property "Footprint" "PDS1-S5-S5-M:CONV_PDS1-S5-S5-M" (at 176.53 102.87 0)
-      (effects (font (size 1.27 1.27)) (justify bottom) hide)
+    (property "Value" "PDS1-S5-S5-D" (at 176.53 93.98 0)
+      (effects (font (size 1.27 1.27)))
+    )
+    (property "Footprint" "PDS1-S5-S5-D:CONV_PDS1-S5-S5-D" (at 176.53 102.87 0)
+      (effects (font (size 1.27 1.27)) (justify left bottom) hide)
     )
     (property "Datasheet" "" (at 176.53 102.87 0)
-      (effects (font (size 1.27 1.27)) hide)
+      (effects (font (size 1.27 1.27)) (justify left bottom) hide)
     )
     (property "MF" "CUI" (at 176.53 102.87 0)
-      (effects (font (size 1.27 1.27)) (justify bottom) hide)
-    )
-    (property "PRICE" "4.02 USD" (at 176.53 102.87 0)
-      (effects (font (size 1.27 1.27)) (justify bottom) hide)
+      (effects (font (size 1.27 1.27)) (justify left bottom) hide)
+    )
+    (property "PRICE" "3.88 USD" (at 176.53 102.87 0)
+      (effects (font (size 1.27 1.27)) (justify left bottom) hide)
     )
     (property "AVAILABILITY" "Bad" (at 176.53 102.87 0)
-      (effects (font (size 1.27 1.27)) (justify bottom) hide)
-    )
-    (property "PACKAGE" "SMD-8 CUI" (at 176.53 102.87 0)
-      (effects (font (size 1.27 1.27)) (justify bottom) hide)
-    )
-    (property "MP" "PDS1-S12-S12-M" (at 176.53 102.87 0)
-      (effects (font (size 1.27 1.27)) (justify bottom) hide)
-    )
-    (property "DESCRIPTION" "PDS1 Series 1 W 12 VDC 84 mA Surface Mount DC-DC Isolated Converter" (at 176.53 102.87 0)
-      (effects (font (size 1.27 1.27)) (justify bottom) hide)
-    )
-    (pin "1")
-    (pin "2")
+      (effects (font (size 1.27 1.27)) (justify left bottom) hide)
+    )
+    (property "PACKAGE" "DIP-7 CUI" (at 176.53 102.87 0)
+      (effects (font (size 1.27 1.27)) (justify left bottom) hide)
+    )
+    (property "MP" "PDS1-S12-S12-D" (at 176.53 102.87 0)
+      (effects (font (size 1.27 1.27)) (justify left bottom) hide)
+    )
+    (property "DESCRIPTION" "Module DC-DC 12VIN 1-OUT 12V 0.083A 1W 4-Pin DIP" (at 176.53 102.87 0)
+      (effects (font (size 1.27 1.27)) (justify left bottom) hide)
+    )
+    (pin "1")
     (pin "4")
     (pin "5")
-    (instances
-      (project "DaisySeedPedal1590b"
+    (pin "7")
+    (instances
+      (project "DaisySeedPedal1590b"
