File: GuitarPedal125b/pcb/DaisySeedPedal125b.kicad_pcb (KiCad board)
At the start: 4 copper layers, 60 x 94 mm, 79 parts, among them J1 Barrel_Jack_Switch, J2 AUDIO_IN_TRS, J3 AUDIO_OUT_TRS, J4 MIDI IN JACK, J5 MIDI OUT JACK, K1 G6K-2, K2 G6K-2, Q1 SS8050, U1 LD1117S50TR_SOT223, U2 PDS1-S5-S5-M, U3 MCP6004, U4 OPA1652AID, U5 H11L1, U6 OLED_DISPLAY_SSD1306_SPI

Commit message: Updated PCB to use 5v power for the relay instead of 9v
Connections:
- D3 pad 1: +9V -> +5V_ISOLATED_POWER
- D4 pad 1: +9V -> +5V_ISOLATED_POWER
- K1 pad 1: +9V -> +5V_ISOLATED_POWER
- K2 pad 1: +9V -> +5V_ISOLATED_POWER
Routing:
- net +9V: track 113.8 -> 53.6 mm
- net +5V_ISOLATED_POWER: track 49.4 -> 57.8 mm

Commit message: Updating some missing footprints
Parts:
- A1: footprint DaisySeed:Electrosmith_Daisy_Seed -> Module:Electrosmith_Daisy_Seed
- J1: footprint Keiths_Reusable_Footprints:CaliforniaJOS_PowerJack -> GuitarPedal125B:CaliforniaJOS_PowerJack
- U6: footprint Keiths_Reusable_Footprints:HiLetgo_OLED_SPI -> GuitarPedal125B:HiLetgo_OLED_SPI
Changed lines of the file:
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@@
     )
   )
-  (footprint "DaisySeed:Electrosmith_Daisy_Seed" (layer "F.Cu")
+  (footprint "Module:Electrosmith_Daisy_Seed" (layer "F.Cu")
     (at 114.25 83.25 90)
     (descr "Embedded platform for audio applications. 96kHz / 24-bit audio hardware. 64MB of SDRAM for up to 10 minute long audio. ARM Cortex-M7 MCU, running at 480MHz. 31 total GPIO pins with configurable functionality. 12-bit Digital to Analog Converters (x2). SD card interfaces. PWM outputs. Serial Protocols for connecting external sensors and devices (SPI, UART, I2S, I2C). Dedicated VIN pin for power. Micro USB port, and additional USB pins for full OTG-support as host and device. https://static1.squarespace.com/static/58d03fdc1b10e3bf442567b8/t/6227e6236f02fb68d1577146/1646781988478/Daisy_Seed_datasheet_v1.0.3.pdf")
@@
     (property "ki_keywords" "Electrosmith Daisy Seed Microcontroller Module ARM Cortex-M7")
     (attr through_hole)
-    (fp_text reference "A1" (at 2.5 -0.25 90) (layer "F.SilkS")
-        (effects (font (size 0.8 0.8) (thickness 0.15)))
+    (fp_text reference "A1" (at 7.62 -3.6 90) (layer "F.SilkS")
+        (effects (font (size 1 1) (thickness 0.15)))
     )
-    (fp_text value "Electrosmith_Daisy_Seed_Rev4" (at 7.12 23.455) (layer "F.Fab") hide
+    (fp_text value "Electrosmith_Daisy_Seed_Rev4" (at 7.62 51 90) (layer "F.Fab")
         (effects (font (size 1 1) (thickness 0.15)))
     )
-    (fp_text user "${REFERENCE}" (at 2.5 -0.25 90) (layer "F.Fab")
+    (fp_text user "${REFERENCE}" (at 7.62 22 90) (layer "F.Fab")
         (effects (font (size 1 1) (thickness 0.15)))
     )
@@
     )
   )
-  (footprint "Keiths_Reusable_Footprints:CaliforniaJOS_PowerJack" (layer "F.Cu")
+  (footprint "GuitarPedal125B:CaliforniaJOS_PowerJack" (layer "F.Cu")
     (at 132.4375 53.3375 -90)
     (property "Sheetfile" "DaisySeedPedal125b.kicad_sch")
@@
         (effects (font (size 1 1) (thickness 0.15)))
     )
-    (fp_text value "Barrel_Jack_Switch" (at -15.8375 -0.0625 unlocked) (layer "F.Fab")
+    (fp_text value "Barrel_Jack_Switch" (at -5.1 6.8 -90 unlocked) (layer "F.Fab")
         (effects (font (size 1 1) (thickness 0.15)))
     )
@@
     )
   )
-  (footprint "Keiths_Reusable_Footprints:HiLetgo_OLED_SPI" (layer "B.Cu")
+  (footprint "GuitarPedal125B:HiLetgo_OLED_SPI" (layer "B.Cu")
     (at 142 89 180)
     (property "Sheetfile" "SSD1306_Screen_SPI.kicad_sch")
     (property "Sheetname" "SSD1306 Screen SPI")
     (attr through_hole)
-    (fp_text reference "U6" (at 0 8.25 unlocked) (layer "B.SilkS")
+    (fp_text reference "U6" (at 0 0 unlocked) (layer "B.SilkS")
         (effects (font (size 1 1) (thickness 0.15)) (justify mirror))
     )
-    (fp_text value "OLED_DISPLAY_SSD1306_SPI" (at -0.25 10 unlocked) (layer "B.Fab")
+    (fp_text value "OLED_DISPLAY_SSD1306_SPI" (at 0 2.25 unlocked) (layer "B.Fab")
         (effects (font (size 1 1) (thickness 0.15)) (justify mirror))
     )
-    (fp_text user "${REFERENCE}" (at 0 8.25) (layer "B.Fab")
+    (fp_text user "${REFERENCE}" (at 0 0) (layer "B.Fab")
         (effects (font (size 1 1) (thickness 0.15)) (justify mirror))
     )

Commit message: 125B Guitar Pedal Rev 2
Updated the 125B Guitar Pedal to fix some issues, upgrade from 3 to 6 knobs and reposition the screen, and make it easier to manufacture with JLCPCB.
Parts:
- removed C20, C21: 10NF, Capacitor_SMD:C_0805_2012Metric
- removed ENC2: RotaryEncoder_Switch, PEC11R-4XXXK-SXXXX:PEC11R-4XXXK-SXXXX
- removed R24, R25, R28, R29: 10K, Resistor_SMD:R_0805_2012Metric
- added POT4: 10K, GuitarPedal125B:Potentiometer_Bourns_PRS11R, B.Cu at (159.5, 70.5)
- added POT5: 10K, GuitarPedal125B:Potentiometer_Bourns_PRS11R, B.Cu at (139.5, 70.5)
- added POT6: 10K, GuitarPedal125B:Potentiometer_Bourns_PRS11R, B.Cu at (119.5, 70.5)
- ENC1: footprint PEC11R-4XXXK-SXXXX:PEC11R-4XXXK-SXXXX -> Rotary_Encoder:RotaryEncoder_Alps_EC11E-Switch_Vertical_H20mm
- J1: footprint GuitarPedal125B:CaliforniaJOS_PowerJack -> GuitarPedal125B:Generic_PowerJack
- K1, K2: footprint Relay_THT:Relay_DPDT_Omron_G6K-2P-Y -> Relay_SMD:Relay_DPDT_Omron_G6K-2G-Y
- POT1, POT2, POT3: footprint RD901F:RD901F4015R1B10K00DL1 -> GuitarPedal125B:Potentiometer_Bourns_PRS11R
- R19, R20: value 220R -> 1K
- U5: footprint Package_DIP:DIP-6_W7.62mm -> Package_DIP:DIP-6_W8.89mm_SMDSocket_LongPads
- moved LED2 53.3 mm to (124.8, 125.0), turned to 90 degrees
- moved LED1 53.3 mm to (159.2, 125.0), turned to -90 degrees
- moved C19 46.6 mm to (121.8, 85.0)
- moved R26 46.6 mm to (115.0, 85.0)
- moved R22 42.2 mm to (117.2, 85.0), turned to 90 degrees
- moved R23 42.1 mm to (124.0, 84.9), turned to -90 degrees
- moved C18 37.8 mm to (119.5, 85.0)
- moved R27 37.8 mm to (126.2, 84.9)
- moved ENC1 33.1 mm to (139.5, 111.3), turned to -90 degrees
- moved R17 28.9 mm to (162.2, 57.8)
- moved C12 19.1 mm to (160.2, 95.3), turned to 90 degrees
- moved C9 17.6 mm to (131.3, 95.3), turned to 90 degrees
- moved R1 17.6 mm to (129.1, 95.3), turned to 90 degrees
- moved R4 17.6 mm to (133.6, 95.3), turned to 90 degrees
- moved R10 17.3 mm to (160.2, 99.0), turned to -90 degrees
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Connections:
- A1 pad 13: ENCODER_1_A -> unconnected-(A1-I2C1_SDA-Pad13)
- A1 pad 14: ENCODER_1_B -> unconnected-(A1-USART1_TX-Pad14)
- A1 pad 15: ENCODER_1_CLICK -> unconnected-(A1-USART1_RX-Pad15)
- A1 pad 2: ENCODER_2_CLICK -> DISABLE_AUDIO_BYPASS
- A1 pad 25: unconnected-(A1-ADC_3-Pad25) -> POT_4
- A1 pad 26: unconnected-(A1-ADC_4-Pad26) -> POT_5
- A1 pad 27: unconnected-(A1-ADC_5-Pad27) -> POT_6
- A1 pad 3: ENCODER_2_A -> ENCODER_1_A
- A1 pad 4: ENCODER_2_B -> ENCODER_1_B
- A1 pad 5: FOOT_SWITCH_2 -> ENCODER_1_CLICK
- A1 pad 6: FOOT_SWITCH_1 -> FOOT_SWITCH_2
- A1 pad 7: DISABLE_AUDIO_BYPASS -> FOOT_SWITCH_1
Routing:
- net Net-(LED2-A): track 3.88 -> 118.2 mm, vias 0 -> 1
- net Net-(LED1-A): track 3.53 -> 67.2 mm, vias 0 -> 1
- net Net-(ENC1-PadA): track 4.33 -> 55.6 mm, vias 0 -> 1
- net Net-(ENC1-PadB): track 4.37 -> 49.1 mm, vias 0 -> 1
- net ENCODER_1_CLICK: track 14.8 -> 54.1 mm
- net MIDI_OUT: track 10.3 -> 43.9 mm
- net AUDIO_OUT_BUFFER_RIGHT: track 35.0 -> 5.22 mm, vias 1 -> 0
- net MIDI_OUT_JACK_PIN5: track 35.0 -> 6.12 mm, vias 1 -> 0
- net POT_6: track 0.00 -> 26.8 mm
- net Net-(U3D-+): track 33.2 -> 8.45 mm, vias 2 -> 0
- net +3.3VA: track 58.1 -> 81.6 mm
- net AUDIO_OUT_JACK_LEFT: track 30.3 -> 52.6 mm, vias 1 -> 2
- net ENCODER_1_B: track 26.3 -> 5.65 mm
- net /Audio Input Buffer/V_AUDIOBIAS: track 26.1 -> 6.05 mm, vias 2 -> 0
- net AUDIO_OUT_BUFFER_LEFT: track 24.7 -> 5.34 mm, vias 1 -> 0
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Other:
- board text added: "Daisy Seed Guitar Pedal 125B (Rev 2) Made by Keith Shepherd 3/11/2023"
- board text removed: "Daisy Seed Guitar Pedal 125B (Rev 1) Made by Keith Shepherd 2/6/2023"

Commit message: Fixed minor issue with power jack footprint
Parts:
- moved J1 0.09 mm to (132.4, 53.2)
Changed lines of the file:
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@@
   )
   (footprint "GuitarPedal125B:Generic_PowerJack" (layer "F.Cu")
-    (at 132.4375 53.3375 -90)
+    (at 132.4375 53.25 -90)
     (property "Sheetfile" "DaisySeedPedal125b.kicad_sch")
     (property "Sheetname" "")
@@
     (pad "2" thru_hole oval (at -6 0 270) (size 2.3 4.5) (drill oval 0.8 3) (layers "*.Cu" "*.Mask")
       (net 12 "POWER_JACK_PWR") (pintype "passive"))
-    (pad "3" thru_hole oval (at -3.125 4.65) (size 2.3 4) (drill oval 0.8 2.5) (layers "*.Cu" "*.Mask")
+    (pad "3" thru_hole oval (at -2.5 4.65) (size 2.3 4) (drill oval 0.8 2.5) (layers "*.Cu" "*.Mask")
       (net 41 "GND") (pintype "passive"))
   )
@@
   (segment (start 145.5 97.386396) (end 145.5 110.275) (width 0.25) (layer "B.Cu") (net 5))
   (segment (start 124.5 92) (end 140.113604 92) (width 0.25) (layer "B.Cu") (net 5))
-  (segment (start 138.6 45.9) (end 133.875 45.9) (width 0.9) (layer "F.Cu") (net 12))
-  (segment (start 133.875 45.9) (end 132.4375 47.3375) (width 0.9) (layer "F.Cu") (net 12))
+  (segment (start 133.7875 45.9) (end 132.4375 47.25) (width 0.9) (layer "F.Cu") (net 12))
+  (segment (start 138.6 45.9) (end 133.7875 45.9) (width 0.9) (layer "F.Cu") (net 12))
   (segment (start 143.967588 71.75) (end 143.275 71.057412) (width 0.25) (layer "B.Cu") (net 13))
   (segment (start 152.63 71.75) (end 143.967588 71.75) (width 0.25) (layer "B.Cu") (net 13))

Commit message: Switched LED and FS placement on the 125B pcb layout
Parts:
- moved LED2 37.0 mm to (161.8, 125.0)
- moved LED1 34.5 mm to (124.8, 125.0), turned to 90 degrees
- moved FS2 9.00 mm to (146.5, 132.2), turned to 90 degrees
- moved FS1 3.96 mm to (140.0, 132.2), turned to 90 degrees
- moved J4 0.75 mm to (121.8, 41.2)
- moved J5 0.75 mm to (162.2, 41.2)
Routing:
- net Net-(LED1-A): track 67.2 -> 120.1 mm
- net Net-(LED2-A): track 118.2 -> 70.9 mm
- net FOOT_SWITCH_1: track 57.3 -> 69.5 mm
- net FOOT_SWITCH_2: track 61.9 -> 59.3 mm
- net MIDI_OUT_JACK_PIN5: track 6.12 -> 6.87 mm
- net MIDI_IN_JACK_PIN5: track 16.5 -> 17.3 mm
- net MIDI_IN_JACK_PIN4: track 8.75 -> 9.50 mm
Other:
- board text added: "Daisy Seed Guitar Pedal 125B (Rev 3) Made by Keith Shepherd 4/14/2023"
- board text removed: "Daisy Seed Guitar Pedal 125B (Rev 2) Made by Keith Shepherd 3/11/2023"

Commit message: Updated H11L1 footprint
Parts:
- U5: footprint Package_DIP:DIP-6_W8.89mm_SMDSocket_LongPads -> GuitarPedal125B:SOP-6_2.54mm
Routing:
- net MIDI_IN_JACK_PIN5: track 17.3 -> 14.3 mm
- net GND: track 51.4 -> 50.8 mm

Commit message: 125B Rev 4 PCB
Updated hardware design for the 125B PCB to include hardware muting.  This allows the signal to be muted during true bypass relay switching, which reduces any popping that might happen otherwise.

Updated the example software to use the hardware mute when using the bypass.  Also, added basic menu support to the OLED screen with some settings for the Tremolo and hardware device.
Parts:
- added R24: 1K, Resistor_SMD:R_0805_2012Metric, F.Cu at (159.0, 105.5)
- added R25: 1K, Resistor_SMD:R_0805_2012Metric, F.Cu at (164.0, 105.5)
- added U7: CPC1018N, Package_SO:SOP-4_3.8x4.1mm_P2.54mm, F.Cu at (159.0, 110.5)
- added U8: CPC1018N, Package_SO:SOP-4_3.8x4.1mm_P2.54mm, F.Cu at (164.0, 110.5)
- moved J2 0.15 mm to (125.4, 125.0)
- moved J3 0.15 mm to (158.6, 125.0)
Connections:
- A1 pad 13: unconnected-(A1-I2C1_SDA-Pad13) -> ENABLE_AUDIO_MUTE
Routing:
- net ENABLE_AUDIO_MUTE: track 0.00 -> 26.4 mm, vias 0 -> 1
- net AUDIO_OUT_JACK_LEFT: track 52.6 -> 62.0 mm
- net AUDIO_OUT_JACK_RIGHT: track 49.2 -> 57.1 mm
- net GND: track 50.8 -> 55.8 mm, vias 35 -> 39
- net Net-(R24-Pad2): track 0.00 -> 3.15 mm
- net Net-(R25-Pad2): track 0.00 -> 2.40 mm
Other:
- board text added: "Daisy Seed Guitar Pedal 125B (Rev 4) Made by Keith Shepherd 5/5/2023"
- board text removed: "Daisy Seed Guitar Pedal 125B (Rev 3) Made by Keith Shepherd 4/14/2023"
