File: GuitarPedal125b/pcb/DaisySeedPedal125b.kicad_pcb (KiCad board)
At the start: 4 copper layers, 60 x 94 mm, 79 parts, among them J1 Barrel_Jack_Switch, J2 AUDIO_IN_TRS, J3 AUDIO_OUT_TRS, J4 MIDI IN JACK, J5 MIDI OUT JACK, K1 G6K-2, K2 G6K-2, Q1 SS8050, U1 LD1117S50TR_SOT223, U2 PDS1-S5-S5-M, U3 MCP6004, U4 OPA1652AID, U5 H11L1, U6 OLED_DISPLAY_SSD1306_SPI, U7 CPC1018N, U8 CPC1018N

Commit message: 125B Rev 5
Minor updates.  Adjusted screen placement slightly to ease assembly. Also grounded TRS jacks better when plug isn't in place.  Adjusted pot footprint mounting holes to be slightly larger to ease installation.
Parts:
- moved R13 5.58 mm to (130.2, 107.0), turned to 180 degrees
- moved C15 3.42 mm to (133.6, 109.8), turned to 90 degrees
- moved R11 3.39 mm to (135.8, 109.8), turned to -90 degrees
- moved U6 1.25 mm to (142.0, 98.0)
Connections:
- J2 pad RN: unconnected-(J2-PadRN) -> GND
- J2 pad TN: unconnected-(J2-PadTN) -> GND
- J3 pad RN: unconnected-(J3-PadRN) -> GND
- J3 pad TN: unconnected-(J3-PadTN) -> GND
Routing:
- net Net-(LED2-A): track 70.9 -> 80.1 mm
- net +5V_ISOLATED_POWER: track 43.1 -> 48.5 mm
- net Net-(LED1-A): track 120.1 -> 124.9 mm
- net Net-(U4B--): track 24.5 -> 19.9 mm
- net BYPASS_LEFT_RETURN: track 23.0 -> 18.8 mm
- net +3.3V: track 3.54 -> 5.54 mm
- net OLED_DISPLAY_SPI_RESET: track 5.86 -> 4.61 mm
- net OLED_DISPLAY_SPI_MOSI: track 5.70 -> 4.45 mm
- net OLED_DISPLAY_SPI_DC: track 4.81 -> 3.56 mm
- net OLED_DISPLAY_SPI_CS: track 5.70 -> 4.45 mm
- net OLED_DISPLAY_SPI_SCK: track 15.3 -> 14.6 mm
- net GND: track 55.8 -> 55.4 mm, vias 39 -> 40
Other:
- board text added: "Daisy Seed Guitar Pedal 125B (Rev 5) Made by Keith Shepherd 6/30/2023"
- board text removed: "Daisy Seed Guitar Pedal 125B (Rev 4) Made by Keith Shepherd 5/5/2023"
