File: GuitarPedal125b/pcb/Audio_Output_Buffer.kicad_sch (KiCad schematic)
At the start: 15 parts, among them U4 OPA1652AID

Commit message: 125B Guitar Pedal Rev 2
Updated the 125B Guitar Pedal to fix some issues, upgrade from 3 to 6 knobs and reposition the screen, and make it easier to manufacture with JLCPCB.
Parts:
- U4: symbol OPA1652AID:OPA1652AID -> Amplifier_Operational:OPA1612AxD; MANUFACTURER Texas Instruments -> (none); MAXIMUM_PACKAGE_HEIGHT 1.75mm -> (none); PARTREV B -> (none); SNAPEDA_PACKAGE_ID 10438 -> (none); STANDARD IPC 7351B -> (none)
Changed lines of the file:
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@@
   (title_block
     (title "Daisy Seed Guitar Pedal 125B")
-    (date "2023-01-27")
-    (rev "1")
+    (date "2023-03-12")
+    (rev "2")
     (company "Made by Keith Shepherd (kshep@mac.com)")
     (comment 1 "https://github.com/electro-smith/Hardware/blob/master/reference/daisy_petal/")
     (comment 2 "Schematic from the Electro-Smith Daisy Petal Reference Hardware Rev 5")
   )
+  (junction (at 175.26 106.68) (diameter 0) (color 0 0 0 0)
+  )
+  (junction (at 147.32 106.68) (diameter 0) (color 0 0 0 0)
+  )
+  (junction (at 152.4 153.67) (diameter 0) (color 0 0 0 0)
+  )
   (junction (at 137.16 153.67) (diameter 0) (color 0 0 0 0)
   )
-  (junction (at 175.26 106.68) (diameter 0) (color 0 0 0 0)
-  )
-  (junction (at 152.4 153.67) (diameter 0) (color 0 0 0 0)
-  )
   (junction (at 175.26 67.31) (diameter 0) (color 0 0 0 0)
   )
   (junction (at 114.3 104.14) (diameter 0) (color 0 0 0 0)
   )
+  (junction (at 114.3 64.77) (diameter 0) (color 0 0 0 0)
+  )
+  (junction (at 147.32 67.31) (diameter 0) (color 0 0 0 0)
+  )
+  (junction (at 152.4 138.43) (diameter 0) (color 0 0 0 0)
+  )
   (junction (at 137.16 138.43) (diameter 0) (color 0 0 0 0)
   )
-  (junction (at 114.3 64.77) (diameter 0) (color 0 0 0 0)
-  )
-  (junction (at 147.32 67.31) (diameter 0) (color 0 0 0 0)
-  )
-  (junction (at 147.32 106.68) (diameter 0) (color 0 0 0 0)
-  )
-  (junction (at 152.4 138.43) (diameter 0) (color 0 0 0 0)
-  )
   (wire (pts (xy 171.45 106.68) (xy 175.26 106.68))
     (stroke (width 0) (type default))
@@
     (stroke (width 0) (type default))
   )
+  (wire (pts (xy 142.24 67.31) (xy 147.32 67.31))
+    (stroke (width 0) (type default))
+  )
   (wire (pts (xy 165.1 149.86) (xy 165.1 153.67))
     (stroke (width 0) (type default))
@@
   )
   (wire (pts (xy 191.77 67.31) (xy 191.77 82.55))
+    (stroke (width 0) (type default))
+  )
+  (wire (pts (xy 142.24 106.68) (xy 147.32 106.68))
     (stroke (width 0) (type default))
   )
@@
     )
   )
-  (symbol (lib_id "OPA1652AID:OPA1652AID") (at 134.62 106.68 0) (unit 1)
+  (symbol (lib_id "Amplifier_Operational:OPA1612AxD") (at 134.62 106.68 0) (unit 1)
     (in_bom yes) (on_board yes) (dnp no) (fields_autoplaced)
     (property "Reference" "U4" (at 137.16 96.52 0)
@@
       (effects (font (size 1.27 1.27)))
     )
-    (property "Footprint" "Package_SO:SOIC-8_3.9x4.9mm_P1.27mm" (at 104.14 101.6 0)
-      (effects (font (size 1.27 1.27)) (justify bottom) hide)
-    )
-    (property "Datasheet" "" (at 134.62 106.68 0)
-      (effects (font (size 1.27 1.27)) hide)
-    )
-    (property "STANDARD" "IPC 7351B" (at 104.14 106.68 0)
-      (effects (font (size 1.27 1.27)) (justify bottom) hide)
-    )
-    (property "PARTREV" "B" (at 104.14 111.76 0)
-      (effects (font (size 1.27 1.27)) (justify bottom) hide)
-    )
-    (property "MANUFACTURER" "Texas Instruments" (at 104.14 104.14 0)
-      (effects (font (size 1.27 1.27)) (justify bottom) hide)
-    )
-    (property "SNAPEDA_PACKAGE_ID" "10438" (at 104.14 114.3 0)
-      (effects (font (size 1.27 1.27)) (justify bottom) hide)
-    )
-    (property "MAXIMUM_PACKAGE_HEIGHT" "1.75mm" (at 104.14 109.22 0)
-      (effects (font (size 1.27 1.27)) (justify bottom) hide)
+    (property "Footprint" "Package_SO:SOIC-8_3.9x4.9mm_P1.27mm" (at 134.62 106.68 0)
+      (effects (font (size 1.27 1.27)) hide)
+    )
+    (property "Datasheet" "http://www.ti.com/lit/ds/symlink/opa1652.pdf" (at 134.62 106.68 0)
+      (effects (font (size 1.27 1.27)) hide)
     )
     (pin "1")
@@
     )
   )
-  (symbol (lib_id "OPA1652AID:OPA1652AID") (at 134.62 146.05 0) (unit 3)
+  (symbol (lib_id "Amplifier_Operational:OPA1612AxD") (at 139.7 146.05 0) (unit 3)
     (in_bom yes) (on_board yes) (dnp no)
-    (property "Reference" "U4" (at 139.7 144.5126 0)
-      (effects (font (size 1.27 1.27)) (justify left))
-    )
-    (property "Value" "OPA1652AID" (at 139.7 148.59 0)
-      (effects (font (size 1.27 1.27)) (justify left))
-    )
-    (property "Footprint" "Package_SO:SOIC-8_3.9x4.9mm_P1.27mm" (at 104.14 140.97 0)
-      (effects (font (size 1.27 1.27)) (justify bottom) hide)
-    )
-    (property "Datasheet" "" (at 134.62 146.05 0)
-      (effects (font (size 1.27 1.27)) hide)
-    )
-    (property "STANDARD" "IPC 7351B" (at 104.14 146.05 0)
-      (effects (font (size 1.27 1.27)) (justify bottom) hide)
-    )
-    (property "PARTREV" "B" (at 104.14 151.13 0)
-      (effects (font (size 1.27 1.27)) (justify bottom) hide)
-    )
-    (property "MANUFACTURER" "Texas Instruments" (at 104.14 143.51 0)
-      (effects (font (size 1.27 1.27)) (justify bottom) hide)
-    )
-    (property "SNAPEDA_PACKAGE_ID" "10438" (at 104.14 153.67 0)
-      (effects (font (size 1.27 1.27)) (justify bottom) hide)
-    )
-    (property "MAXIMUM_PACKAGE_HEIGHT" "1.75mm" (at 104.14 148.59 0)
-      (effects (font (size 1.27 1.27)) (justify bottom) hide)
+    (property "Reference" "U4" (at 125.73 144.78 0)
+      (effects (font (size 1.27 1.27)) (justify left))
+    )
+    (property "Value" "OPA1652AID" (at 121.92 148.59 0)
+      (effects (font (size 1.27 1.27)) (justify left))
+    )
+    (property "Footprint" "Package_SO:SOIC-8_3.9x4.9mm_P1.27mm" (at 139.7 146.05 0)
+      (effects (font (size 1.27 1.27)) hide)
+    )
+    (property "Datasheet" "http://www.ti.com/lit/ds/symlink/opa1652.pdf" (at 139.7 146.05 0)
+      (effects (font (size 1.27 1.27)) hide)
     )
     (pin "1")
@@
     )
   )
-  (symbol (lib_id "OPA1652AID:OPA1652AID") (at 134.62 67.31 0) (unit 2)
+  (symbol (lib_id "Amplifier_Operational:OPA1612AxD") (at 134.62 67.31 0) (unit 2)
     (in_bom yes) (on_board yes) (dnp no) (fields_autoplaced)
     (property "Reference" "U4" (at 137.16 57.15 0)
@@
       (effects (font (size 1.27 1.27)))
     )
-    (property "Footprint" "Package_SO:SOIC-8_3.9x4.9mm_P1.27mm" (at 104.14 62.23 0)
-      (effects (font (size 1.27 1.27)) (justify bottom) hide)
-    )
-    (property "Datasheet" "" (at 134.62 67.31 0)
-      (effects (font (size 1.27 1.27)) hide)
-    )
-    (property "STANDARD" "IPC 7351B" (at 104.14 67.31 0)
-      (effects (font (size 1.27 1.27)) (justify bottom) hide)
-    )
-    (property "PARTREV" "B" (at 104.14 72.39 0)
-      (effects (font (size 1.27 1.27)) (justify bottom) hide)
-    )
-    (property "MANUFACTURER" "Texas Instruments" (at 104.14 64.77 0)
-      (effects (font (size 1.27 1.27)) (justify bottom) hide)
-    )
-    (property "SNAPEDA_PACKAGE_ID" "10438" (at 104.14 74.93 0)
-      (effects (font (size 1.27 1.27)) (justify bottom) hide)
-    )
-    (property "MAXIMUM_PACKAGE_HEIGHT" "1.75mm" (at 104.14 69.85 0)
-      (effects (font (size 1.27 1.27)) (justify bottom) hide)
-    )
-    (pin "1")
+    (property "Footprint" "Package_SO:SOIC-8_3.9x4.9mm_P1.27mm" (at 134.62 67.31 0)
+      (effects (font (size 1.27 1.27)) hide)
+    )
+    (property "Datasheet" "http://www.ti.com/lit/ds/symlink/opa1652.pdf" (at 134.62 67.31 0)
+      (effects (font (size 1.27 1.27)) hide)
+    )
+    (pin "1")
