File: GuitarPedal125b/pcb/Audio_True_Bypass_Stereo.kicad_sch (KiCad schematic)
At the start: 6 parts, among them K1 G6K-2, K2 G6K-2, Q1 SS8050

Commit message: Updated PCB to use 5v power for the relay instead of 9v
Connections:
- net +9V renamed +5V_ISOLATED_POWER
Changed lines of the file:
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@@
+    )
+  )
+  (global_label "+5V_ISOLATED_POWER" (shape input) (at 135.89 40.64 90) (fields_autoplaced)
+    (effects (font (size 1.27 1.27)) (justify left))
+    (property "Intersheetrefs" "${INTERSHEET_REFS}" (at 135.89 16.8095 90)
+      (effects (font (size 1.27 1.27)) (justify left) hide)
     )
   )
@@
         )
       )
-    )
-  )
-  (symbol (lib_id "power:+9V") (at 135.89 40.64 0) (unit 1)
-    (in_bom yes) (on_board yes) (dnp no) (fields_autoplaced)
-    (property "Reference" "#PWR019" (at 135.89 44.45 0)
-      (effects (font (size 1.27 1.27)) hide)
-    )
-    (property "Value" "+9V" (at 135.89 35.56 0)
-      (effects (font (size 1.27 1.27)))
-    )
-    (property "Footprint" "" (at 135.89 40.64 0)
-      (effects (font (size 1.27 1.27)) hide)
-    )
-    (property "Datasheet" "" (at 135.89 40.64 0)
-      (effects (font (size 1.27 1.27)) hide)
-    )
-    (pin "1")
-    (instances
-      (project "DaisySeedPedal125b"
-        (path "/1d54e6f4-7c7a-4f03-b2db-a136bdff5b99/d5b1af0e-2179-4bcd-8e24-55fd6680ab7e"
-          (reference "#PWR019") (unit 1)
-        )
-      )

Commit message: 125B Guitar Pedal Rev 2
Updated the 125B Guitar Pedal to fix some issues, upgrade from 3 to 6 knobs and reposition the screen, and make it easier to manufacture with JLCPCB.
Parts:
- D3, D4: symbol Device:D -> Diode:1N4007
- K1, K2: footprint Relay_THT:Relay_DPDT_Omron_G6K-2P-Y -> Relay_SMD:Relay_DPDT_Omron_G6K-2G-Y
Other:
- company: (none) -> Made by Keith Shepherd (kshep@mac.com)
- title: (none) -> Daisy Seed Guitar Pedal 125B
Changed lines of the file:
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@@
 (kicad_sch (version 20230121) (generator eeschema)
   (paper "USLetter")
+  (title_block
+    (title "Daisy Seed Guitar Pedal 125B")
+    (date "2023-03-12")
+    (rev "2")
+    (company "Made by Keith Shepherd (kshep@mac.com)")
+  )
   (junction (at 135.89 63.5) (diameter 0) (color 0 0 0 0)
   )
@@
       (effects (font (size 1.27 1.27)))
     )
-    (property "Footprint" "Relay_THT:Relay_DPDT_Omron_G6K-2P-Y" (at 124.46 73.66 0)
+    (property "Footprint" "Relay_SMD:Relay_DPDT_Omron_G6K-2G-Y" (at 124.46 73.66 0)
       (effects (font (size 1.27 1.27)) (justify left) hide)
     )
@@
     )
   )
-  (symbol (lib_id "Device:D") (at 124.46 46.99 180) (unit 1)
+  (symbol (lib_id "Diode:1N4007") (at 124.46 46.99 180) (unit 1)
     (in_bom yes) (on_board yes) (dnp no) (fields_autoplaced)
     (property "Reference" "D3" (at 124.46 40.64 0)
@@
       (effects (font (size 1.27 1.27)))
     )
-    (property "Footprint" "Diode_SMD:D_SOD-123F" (at 124.46 46.99 0)
-      (effects (font (size 1.27 1.27)) hide)
-    )
-    (property "Datasheet" "~" (at 124.46 46.99 0)
+    (property "Footprint" "Diode_SMD:D_SOD-123F" (at 124.46 42.545 0)
+      (effects (font (size 1.27 1.27)) hide)
+    )
+    (property "Datasheet" "http://www.vishay.com/docs/88503/1n4001.pdf" (at 124.46 46.99 0)
       (effects (font (size 1.27 1.27)) hide)
     )
@@
       (effects (font (size 1.27 1.27)))
     )
-    (property "Footprint" "Relay_THT:Relay_DPDT_Omron_G6K-2P-Y" (at 124.46 130.81 0)
+    (property "Footprint" "Relay_SMD:Relay_DPDT_Omron_G6K-2G-Y" (at 124.46 130.81 0)
       (effects (font (size 1.27 1.27)) (justify left) hide)
     )
@@
     )
   )
-  (symbol (lib_id "Device:D") (at 124.46 104.14 180) (unit 1)
+  (symbol (lib_id "Diode:1N4007") (at 124.46 104.14 180) (unit 1)
     (in_bom yes) (on_board yes) (dnp no) (fields_autoplaced)
     (property "Reference" "D4" (at 124.46 97.79 0)
@@
       (effects (font (size 1.27 1.27)))
     )
-    (property "Footprint" "Diode_SMD:D_SOD-123F" (at 124.46 104.14 0)
-      (effects (font (size 1.27 1.27)) hide)
-    )
-    (property "Datasheet" "~" (at 124.46 104.14 0)
-      (effects (font (size 1.27 1.27)) hide)
-    )
+    (property "Footprint" "Diode_SMD:D_SOD-123F" (at 124.46 99.695 0)
+      (effects (font (size 1.27 1.27)) hide)
+    )
+    (property "Datasheet" "http://www.vishay.com/docs/88503/1n4001.pdf" (at 124.46 104.14 0)
+      (effects (font (size 1.27 1.27)) hide)
+    )

Commit message: 125B Rev 4 PCB
Updated hardware design for the 125B PCB to include hardware muting.  This allows the signal to be muted during true bypass relay switching, which reduces any popping that might happen otherwise.

Updated the example software to use the hardware mute when using the bypass.  Also, added basic menu support to the OLED screen with some settings for the Tremolo and hardware device.
Parts:
- added R24, R25: 1K, Resistor_SMD:R_0805_2012Metric, symbol Device:R
- added U7, U8: CPC1018N, Package_SO:SOP-4_3.8x4.1mm_P2.54mm, symbol Relay_SolidState:CPC1017N
Connections:
- net AUDIO_OUT_JACK_LEFT: now also U7.4
- net AUDIO_OUT_JACK_RIGHT: now also U8.4
- net GND: now also U7.2, U7.3, U8.2, U8.3
- new net: R24.2, U7.1
- new net: R25.2, U8.1
- new net ENABLE_AUDIO_MUTE: R24.1, R25.1
