File: GuitarPedal125b/pcb/Controls.kicad_sch (KiCad schematic)
At the start: 23 parts

Commit message: 125B Guitar Pedal Rev 2
Updated the 125B Guitar Pedal to fix some issues, upgrade from 3 to 6 knobs and reposition the screen, and make it easier to manufacture with JLCPCB.
Parts:
- removed C20, C21: 10NF, Capacitor_SMD:C_0805_2012Metric, symbol Device:C
- removed ENC2: RotaryEncoder_Switch, PEC11R-4XXXK-SXXXX:PEC11R-4XXXK-SXXXX, symbol Device:RotaryEncoder_Switch
- removed R24, R25, R28, R29: 10K, Resistor_SMD:R_0805_2012Metric, symbol Device:R
- added POT4, POT5, POT6: 10K, GuitarPedal125B:Potentiometer_Bourns_PRS11R, symbol Device:R_Potentiometer_US
- ENC1: footprint PEC11R-4XXXK-SXXXX:PEC11R-4XXXK-SXXXX -> Rotary_Encoder:RotaryEncoder_Alps_EC11E-Switch_Vertical_H20mm
- POT1, POT2, POT3: footprint RD901F:RD901F4015R1B10K00DL1 -> GuitarPedal125B:Potentiometer_Bourns_PRS11R
- R19, R20: value 220R -> 1K
Connections:
- net +3.3VA: now also POT4.3, POT5.3, POT6.3
- net GND: now also POT4.1, POT5.1, POT6.1
- new net POT_4: POT4.2
- new net POT_5: POT5.2
- new net POT_6: POT6.2
Other:
- company: (none) -> Made by Keith Shepherd (kshep@mac.com)
- title: (none) -> Daisy Seed Guitar Pedal 125B
