File: GuitarPedal125b/pcb/DaisySeedPedal125b.kicad_sch (KiCad schematic)
At the start: 6 parts, among them J1 Barrel_Jack_Switch, J2 AUDIO_IN_TRS, J3 AUDIO_OUT_TRS, J4 MIDI IN JACK, J5 MIDI OUT JACK

Commit message: Updating some missing footprints
Parts:
- A1: footprint DaisySeed:Electrosmith_Daisy_Seed -> Module:Electrosmith_Daisy_Seed
- J1: footprint Keiths_Reusable_Footprints:CaliforniaJOS_PowerJack -> GuitarPedal125B:CaliforniaJOS_PowerJack
Changed lines of the file:
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@@
       (effects (font (size 1.27 1.27)) (justify left))
     )
-    (property "Footprint" "DaisySeed:Electrosmith_Daisy_Seed" (at 147.32 144.78 0)
+    (property "Footprint" "Module:Electrosmith_Daisy_Seed" (at 147.32 144.78 0)
       (effects (font (size 1.27 1.27)) hide)
     )
@@
       (effects (font (size 1.27 1.27)) (justify right))
     )
-    (property "Footprint" "Keiths_Reusable_Footprints:CaliforniaJOS_PowerJack" (at 219.71 35.814 0)
+    (property "Footprint" "GuitarPedal125B:CaliforniaJOS_PowerJack" (at 219.71 35.814 0)
       (effects (font (size 1.27 1.27)) hide)
     )

Commit message: Updating missing symbol libraries
Parts:
- A1: symbol Electrosmith_Daisy_Seed:Electrosmith_Daisy_Seed_Rev4 -> MCU_Module:Electrosmith_Daisy_Seed_Rev4
Changed lines of the file:
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@@
     )
   )
-  (symbol (lib_id "Electrosmith_Daisy_Seed:Electrosmith_Daisy_Seed_Rev4") (at 128.27 109.22 0) (unit 1)
+  (symbol (lib_id "MCU_Module:Electrosmith_Daisy_Seed_Rev4") (at 128.27 109.22 0) (unit 1)
     (in_bom yes) (on_board yes) (dnp no) (fields_autoplaced)
     (property "Reference" "A1" (at 132.8294 144.78 0)

Commit message: 125B Guitar Pedal Rev 2
Updated the 125B Guitar Pedal to fix some issues, upgrade from 3 to 6 knobs and reposition the screen, and make it easier to manufacture with JLCPCB.
Parts:
- J1: footprint GuitarPedal125B:CaliforniaJOS_PowerJack -> GuitarPedal125B:Generic_PowerJack
- J4, J5: symbol Connector:AudioJack4 -> Connector_Audio:AudioJack4
Connections:
- net ENCODER_2_A is gone; now on net ENCODER_1_A: A1.3 (SD_DATA_2)
- net ENCODER_2_B is gone; now on net ENCODER_1_B: A1.4 (SD_DATA_1)
- net ENCODER_2_CLICK is gone; now on net DISABLE_AUDIO_BYPASS: A1.2 (SD_DATA_3)
- net DISABLE_AUDIO_BYPASS: no longer A1.7 (SD_CLK)
- net ENCODER_1_A: no longer A1.13 (I2C1_SDA)
- net ENCODER_1_B: no longer A1.14 (USART1_TX)
- net ENCODER_1_CLICK: now also A1.5 (SD_DATA_0); no longer A1.15 (USART1_RX)
- net FOOT_SWITCH_1: now also A1.7 (SD_CLK); no longer A1.6 (SD_CMD)
- net FOOT_SWITCH_2: now also A1.6 (SD_CMD); no longer A1.5 (SD_DATA_0)
- net POT_4: now reaches A1.25 (ADC_3)
- net POT_5: now reaches A1.26 (ADC_4)
- net POT_6: now reaches A1.27 (ADC_5)

Commit message: 125B Rev 4 PCB
Updated hardware design for the 125B PCB to include hardware muting.  This allows the signal to be muted during true bypass relay switching, which reduces any popping that might happen otherwise.

Updated the example software to use the hardware mute when using the bypass.  Also, added basic menu support to the OLED screen with some settings for the Tremolo and hardware device.
Connections:
- net ENABLE_AUDIO_MUTE: now reaches A1.13 (I2C1_SDA)
- no-connect marks 16 -> 15
Other:
- moved on the sheet: J4, J5

Commit message: 125B Rev 5
Minor updates.  Adjusted screen placement slightly to ease assembly. Also grounded TRS jacks better when plug isn't in place.  Adjusted pot footprint mounting holes to be slightly larger to ease installation.
Connections:
- net GND: now also J2.RN, J2.TN, J3.RN, J3.TN
- no-connect marks 15 -> 11
Changed lines of the file:
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@@
   (title_block
     (title "Daisy Seed Guitar Pedal 125B")
-    (date "2023-04-15")
-    (rev "4")
+    (date "2023-06-30")
+    (rev "5")
     (company "Made by Keith Shepherd (kshep@mac.com)")
     (comment 1 "https://github.com/electro-smith/Hardware/blob/master/reference/daisy_petal/")
@@
   (junction (at 128.27 147.32) (diameter 0) (color 0 0 0 0)
   )
+  (junction (at 231.14 88.9) (diameter 0) (color 0 0 0 0)
+  )
+  (junction (at 231.14 93.98) (diameter 0) (color 0 0 0 0)
+  )
   (junction (at 231.14 96.52) (diameter 0) (color 0 0 0 0)
   )
+  (junction (at 231.14 67.31) (diameter 0) (color 0 0 0 0)
+  )
   (junction (at 240.03 39.37) (diameter 0) (color 0 0 0 0)
   )
-  (no_connect (at 231.14 83.82))
-  (no_connect (at 231.14 57.15))
+  (junction (at 231.14 62.23) (diameter 0) (color 0 0 0 0)
+  )
   (no_connect (at 153.67 93.98))
   (no_connect (at 102.87 127))
   (no_connect (at 102.87 132.08))
   (no_connect (at 153.67 96.52))
-  (no_connect (at 231.14 88.9))
   (no_connect (at 153.67 83.82))
   (no_connect (at 102.87 129.54))
@@
   (no_connect (at 228.6 123.19))
   (no_connect (at 102.87 114.3))
-  (no_connect (at 231.14 62.23))
   (no_connect (at 102.87 134.62))
   (no_connect (at 102.87 124.46))
@@
     (stroke (width 0) (type default))
   )
+  (wire (pts (xy 231.14 88.9) (xy 231.14 93.98))
+    (stroke (width 0) (type default))
+  )
   (wire (pts (xy 229.87 144.78) (xy 233.68 144.78))
     (stroke (width 0) (type default))
@@
     (stroke (width 0) (type default))
   )
+  (wire (pts (xy 231.14 83.82) (xy 231.14 88.9))
+    (stroke (width 0) (type default))
+  )
   (wire (pts (xy 232.41 128.27) (xy 232.41 125.73))
     (stroke (width 0) (type default))
@@
     (stroke (width 0) (type default))
   )
+  (wire (pts (xy 228.6 86.36) (xy 231.14 86.36))
+    (stroke (width 0) (type default))
+  )
   (wire (pts (xy 125.73 147.32) (xy 128.27 147.32))
     (stroke (width 0) (type default))
@@
     (stroke (width 0) (type default))
   )
+  (wire (pts (xy 231.14 57.15) (xy 231.14 62.23))
+    (stroke (width 0) (type default))
+  )
   (wire (pts (xy 128.27 58.42) (xy 128.27 71.12))
     (stroke (width 0) (type default))
@@
     (stroke (width 0) (type default))
   )
+  (wire (pts (xy 231.14 62.23) (xy 231.14 67.31))
+    (stroke (width 0) (type default))
+  )
   (wire (pts (xy 229.87 147.32) (xy 233.68 147.32))
     (stroke (width 0) (type default))
@@
     (stroke (width 0) (type default))
   )
-  (global_label "AUDIO_OUT_JACK_LEFT" (shape input) (at 231.14 86.36 180) (fields_autoplaced)
-    (effects (font (size 1.27 1.27)) (justify right))
-    (property "Intersheetrefs" "${INTERSHEET_REFS}" (at 207.7417 86.2806 0)
+  (wire (pts (xy 228.6 91.44) (xy 231.14 91.44))
+    (stroke (width 0) (type default))
+  )
+  (global_label "AUDIO_OUT_JACK_LEFT" (shape input) (at 228.6 86.36 180) (fields_autoplaced)
+    (effects (font (size 1.27 1.27)) (justify right))
+    (property "Intersheetrefs" "${INTERSHEET_REFS}" (at 205.2017 86.2806 0)
       (effects (font (size 1.27 1.27)) (justify right) hide)
     )
@@
     )
   )
-  (global_label "AUDIO_OUT_JACK_RIGHT" (shape input) (at 231.14 91.44 180) (fields_autoplaced)
-    (effects (font (size 1.27 1.27)) (justify right))
-    (property "Intersheetrefs" "${INTERSHEET_REFS}" (at 206.5321 91.3606 0)
-      (effects (font (size 1.27 1.27)) (justify right) hide)
-    )
+  (global_label "AUDIO_OUT_JACK_RIGHT" (shape input) (at 228.6 91.44 180) (fields_autoplaced)
+    (effects (font (size 1.27 1.27)) (justify right))
+    (property "Intersheetrefs" "${INTERSHEET_REFS}" (at 203.9921 91.3606 0)
+      (effects (font (size 1.27 1.27)) (justify right) hide)
+    )
