File: GuitarPedal125b/pcb/Midi_InOut.kicad_sch (KiCad schematic)
At the start: 7 parts, among them U5 H11L1

Commit message: 125B Guitar Pedal Rev 2
Updated the 125B Guitar Pedal to fix some issues, upgrade from 3 to 6 knobs and reposition the screen, and make it easier to manufacture with JLCPCB.
Parts:
- D2: symbol Diode:1N914 -> Diode:1N4148
- U5: footprint Package_DIP:DIP-6_W7.62mm -> Package_DIP:DIP-6_W8.89mm_SMDSocket_LongPads
Changed lines of the file:
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@@
   (title_block
     (title "Daisy Seed Guitar Pedal 125B")
-    (date "2023-01-27")
-    (rev "1")
+    (date "2023-03-12")
+    (rev "2")
     (company "Made by Keith Shepherd (kshep@mac.com)")
     (comment 1 "https://diyelectromusic.wordpress.com/2022/08/29/3v3-midi-module-pcb/")
@@
     )
   )
-  (symbol (lib_id "Diode:1N914") (at 127 95.25 270) (unit 1)
+  (symbol (lib_id "Diode:1N4148") (at 127 95.25 270) (unit 1)
     (in_bom yes) (on_board yes) (dnp no) (fields_autoplaced)
     (property "Reference" "D2" (at 129.54 93.9799 90)
@@
       (effects (font (size 1.27 1.27)) (justify left))
     )
-    (property "Footprint" "Diode_SMD:D_SOD-123" (at 122.555 95.25 0)
-      (effects (font (size 1.27 1.27)) hide)
-    )
-    (property "Datasheet" "http://www.vishay.com/docs/85622/1n914.pdf" (at 127 95.25 0)
+    (property "Footprint" "Diode_SMD:D_SOD-123" (at 127 95.25 0)
+      (effects (font (size 1.27 1.27)) hide)
+    )
+    (property "Datasheet" "https://assets.nexperia.com/documents/data-sheet/1N4148_1N4448.pdf" (at 127 95.25 0)
       (effects (font (size 1.27 1.27)) hide)
     )
@@
       (effects (font (size 1.27 1.27)))
     )
-    (property "Footprint" "Package_DIP:DIP-6_W7.62mm" (at 142.494 95.25 0)
-      (effects (font (size 1.27 1.27)) hide)
-    )
+    (property "Footprint" "Package_DIP:DIP-6_W8.89mm_SMDSocket_LongPads" (at 142.494 95.25 0)
+      (effects (font (size 1.27 1.27)) hide)
+    )

Commit message: Updated H11L1 footprint
Parts:
- U5: footprint Package_DIP:DIP-6_W8.89mm_SMDSocket_LongPads -> GuitarPedal125B:SOP-6_2.54mm
Changed lines of the file:
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@@
       (effects (font (size 1.27 1.27)))
     )
-    (property "Footprint" "Package_DIP:DIP-6_W8.89mm_SMDSocket_LongPads" (at 142.494 95.25 0)
+    (property "Footprint" "GuitarPedal125B:SOP-6_2.54mm" (at 142.494 95.25 0)
       (effects (font (size 1.27 1.27)) hide)
     )
