File: GuitarPedal125b/pcb/Power.kicad_sch (KiCad schematic)
At the start: 10 parts, among them U1 LD1117S50TR_SOT223, U2 PDS1-S5-S5-M

Commit message: 125B Guitar Pedal Rev 2
Updated the 125B Guitar Pedal to fix some issues, upgrade from 3 to 6 knobs and reposition the screen, and make it easier to manufacture with JLCPCB.
Parts:
- D1: symbol Device:D -> Diode:1N5817
Changed lines of the file:
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@@
   (title_block
     (title "Daisy Seed Guitar Pedal 125B")
-    (date "2023-01-27")
-    (rev "1")
+    (date "2023-03-12")
+    (rev "2")
     (company "Made by Keith Shepherd (kshep@mac.com)")
     (comment 1 "https://github.com/electro-smith/Hardware/blob/master/reference/daisy_petal/")
@@
   )
   (label "VIN" (at 153.67 100.33 0) (fields_autoplaced)
-    (effects (font (size 1.27 1.27)) (justify left bottom))
-  )
-  (label "EXT_PWR" (at 48.26 100.33 0) (fields_autoplaced)
     (effects (font (size 1.27 1.27)) (justify left bottom))
   )
@@
     )
   )
-  (symbol (lib_id "Device:D") (at 68.58 100.33 180) (unit 1)
+  (symbol (lib_id "Diode:1N5817") (at 68.58 100.33 180) (unit 1)
     (in_bom yes) (on_board yes) (dnp no)
     (property "Reference" "D1" (at 68.58 97.79 0)
@@
       (effects (font (size 1.27 1.27)))
     )
-    (property "Footprint" "Diode_SMD:D_SOD-123" (at 68.58 100.33 0)
-      (effects (font (size 1.27 1.27)) hide)
-    )
-    (property "Datasheet" "~" (at 68.58 100.33 0)
-      (effects (font (size 1.27 1.27)) hide)
-    )
+    (property "Footprint" "Diode_SMD:D_SOD-123" (at 68.58 95.885 0)
+      (effects (font (size 1.27 1.27)) hide)
+    )
+    (property "Datasheet" "http://www.vishay.com/docs/88525/1n5817.pdf" (at 68.58 100.33 0)
+      (effects (font (size 1.27 1.27)) hide)
+    )
