File: GuitarPedal125b/pcb/SSD1306_Screen_SPI.kicad_sch (KiCad schematic)
At the start: 1 part, among them U6 OLED_DISPLAY_SSD1306_SPI

Commit message: Updating some missing footprints
Parts:
- U6: footprint Keiths_Reusable_Footprints:HiLetgo_OLED_SPI -> GuitarPedal125B:HiLetgo_OLED_SPI
Changed lines of the file:
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@@
       (effects (font (size 1.27 1.27)) (justify left))
     )
-    (property "Footprint" "Keiths_Reusable_Footprints:HiLetgo_OLED_SPI" (at 138.43 102.87 0)
+    (property "Footprint" "GuitarPedal125B:HiLetgo_OLED_SPI" (at 138.43 102.87 0)
       (effects (font (size 1.27 1.27)) hide)
     )

Commit message: Updating missing symbol libraries
Parts:
- U6: symbol Keiths_Symbols:OLED_DISPLAY_SSD1306_SPI -> GuitarPedal125B:OLED_DISPLAY_SSD1306_SPI
Changed lines of the file:
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@@
     )
   )
-  (symbol (lib_id "Keiths_Symbols:OLED_DISPLAY_SSD1306_SPI") (at 138.43 102.87 0) (unit 1)
+  (symbol (lib_id "GuitarPedal125B:OLED_DISPLAY_SSD1306_SPI") (at 138.43 102.87 0) (unit 1)
     (in_bom yes) (on_board yes) (dnp no)
     (property "Reference" "U6" (at 137.16 100.33 0)
