File: Hardware/GuitarPedal1590b/pcb/DaisySeedPedal1590b.kicad_pcb (KiCad board)
At the start: 4 copper layers, 54 x 106 mm, 59 parts, among them J1 Barrel_Jack, J2 AUDIO_IN_TRS, J3 AUDIO_OUT_TRS, J4 MIDI IN JACK, J5 MIDI OUT JACK, U1 L4931CZ50, U2 PDS1-S5-S5-D, U3 MCP6004, U4 OPA2134, U5 H11L1

Commit message: Updated 1590b Schematic Rev 6
* Added a DNP SMD Resistor pad to optionally bypass the PDS1 isolated power components.
Parts:
- added R21: DNP, Resistor_SMD:R_0805_2012Metric, F.Cu at (94.6, 73.0)
Routing:
- net +5V: track 17.6 -> 27.6 mm
- net +5V_ISOLATED_POWER: track 40.3 -> 46.2 mm
Other:
- board text added: "Daisy Seed 1590b Guitar Pedal Made by Keith Shepherd 11/12/2023 (Rev 6)"
- board text removed: "Daisy Seed 1590b Guitar Pedal Made by Keith Shepherd 6/3/2023 (Rev 5)"
Changed lines of the file:
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@@
       (drillshape 0)
       (scaleselection 1)
-      (outputdirectory "../../../../Desktop/DaisySeedPedal1590-Rev5-gerbers/")
+      (outputdirectory "/Users/kshep/Desktop/DaisySeedPedal1590b-Rev6-gerbers/")
     )
   )
@@
     )
   )
+  (footprint "Resistor_SMD:R_0805_2012Metric" (layer "F.Cu")
+    (at 94.6 73 -90)
+    (descr "Resistor SMD 0805 (2012 Metric), square (rectangular) end terminal, IPC_7351 nominal, (Body size source: IPC-SM-782 page 72, https://www.pcb-3d.com/wordpress/wp-content/uploads/ipc-sm-782a_amendment_1_and_2.pdf), generated with kicad-footprint-generator")
+    (tags "resistor")
+    (property "Sheetfile" "Power.kicad_sch")
+    (property "Sheetname" "Power")
+    (property "ki_description" "Resistor")
+    (property "ki_keywords" "R res resistor")
+    (attr smd)
+    (fp_text reference "R21" (at 0 1.6 90) (layer "F.SilkS")
+        (effects (font (size 0.8 0.8) (thickness 0.15)))
+    )
+    (fp_text value "DNP" (at 0 1.65 90) (layer "F.Fab")
+        (effects (font (size 1 1) (thickness 0.15)))
+    )
+    (fp_text user "${REFERENCE}" (at 0 0 90) (layer "F.Fab")
+        (effects (font (size 0.5 0.5) (thickness 0.08)))
+    )
+    (fp_line (start -0.227064 -0.735) (end 0.227064 -0.735)
+      (stroke (width 0.12) (type solid)) (layer "F.SilkS"))
+    (fp_line (start -0.227064 0.735) (end 0.227064 0.735)
+      (stroke (width 0.12) (type solid)) (layer "F.SilkS"))
+    (fp_line (start -1.68 -0.95) (end 1.68 -0.95)
+      (stroke (width 0.05) (type solid)) (layer "F.CrtYd"))
+    (fp_line (start -1.68 0.95) (end -1.68 -0.95)
+      (stroke (width 0.05) (type solid)) (layer "F.CrtYd"))
+    (fp_line (start 1.68 -0.95) (end 1.68 0.95)
+      (stroke (width 0.05) (type solid)) (layer "F.CrtYd"))
+    (fp_line (start 1.68 0.95) (end -1.68 0.95)
+      (stroke (width 0.05) (type solid)) (layer "F.CrtYd"))
+    (fp_line (start -1 -0.625) (end 1 -0.625)
+      (stroke (width 0.1) (type solid)) (layer "F.Fab"))
+    (fp_line (start -1 0.625) (end -1 -0.625)
+      (stroke (width 0.1) (type solid)) (layer "F.Fab"))
+    (fp_line (start 1 -0.625) (end 1 0.625)
+      (stroke (width 0.1) (type solid)) (layer "F.Fab"))
+    (fp_line (start 1 0.625) (end -1 0.625)
+      (stroke (width 0.1) (type solid)) (layer "F.Fab"))
+    (pad "1" smd roundrect (at -0.9125 0 270) (size 1.025 1.4) (layers "F.Cu" "F.Paste" "F.Mask") (roundrect_rratio 0.243902439)
+      (net 9 "+5V") (pintype "passive"))
+    (pad "2" smd roundrect (at 0.9125 0 270) (size 1.025 1.4) (layers "F.Cu" "F.Paste" "F.Mask") (roundrect_rratio 0.243902439)
+      (net 10 "+5V_ISOLATED_POWER") (pintype "passive"))
+    (model "${KICAD6_3DMODEL_DIR}/Resistor_SMD.3dshapes/R_0805_2012Metric.wrl"
+      (offset (xyz 0 0 0))
+      (scale (xyz 1 1 1))
+      (rotate (xyz 0 0 0))
+    )
+  )
   (gr_line (start 146.75 83) (end 71 83)
     (stroke (width 0.15) (type default)) (layer "Dwgs.User"))
@@
     )
     (stroke (width 0.1) (type solid)) (fill none) (layer "Edge.Cuts"))
-  (gr_text "Daisy Seed 1590b Guitar Pedal\n\nMade by Keith Shepherd\n\n6/3/2023 (Rev 5)" (at 107.6 96.5) (layer "B.SilkS")
+  (gr_text "Daisy Seed 1590b Guitar Pedal\n\nMade by Keith Shepherd\n\n11/12/2023 (Rev 6)" (at 107.6 96.5) (layer "B.SilkS")
     (effects (font (size 1 1) (thickness 0.15)) (justify mirror))
   )
@@
   (segment (start 110.1225 30.5375) (end 114.62 35.035) (width 0.9) (layer "F.Cu") (net 8))
   (segment (start 93.5 63.5) (end 93.75 63.75) (width 0.9) (layer "F.Cu") (net 9))
+  (segment (start 93.75 63.75) (end 96.2 66.2) (width 0.9) (layer "F.Cu") (net 9))
+  (segment (start 96.2 66.2) (end 96.2 70.4875) (width 0.9) (layer "F.Cu") (net 9))
   (segment (start 88.75 63.5) (end 86.700001 61.450001) (width 0.9) (layer "F.Cu") (net 9))
+  (segment (start 96.2 70.4875) (end 94.6 72.0875) (width 0.9) (layer "F.Cu") (net 9))
   (segment (start 86.700001 61.450001) (end 86.700001 57.979999) (width 0.9) (layer "F.Cu") (net 9))
   (segment (start 88.75 63.5) (end 93.5 63.5) (width 0.9) (layer "F.Cu") (net 9))
@@
   (segment (start 81.25 97.5) (end 91.5 87.25) (width 0.9) (layer "F.Cu") (net 10))
   (segment (start 91.5 83.7226) (end 94.7226 80.5) (width 0.9) (layer "F.Cu") (net 10))
+  (segment (start 94.6 73.9125) (end 93.5 75.0125) (width 0.9) (layer "F.Cu") (net 10))
   (segment (start 81.25 97.5) (end 81.25 110.5) (width 0.9) (layer "F.Cu") (net 10))
   (segment (start 93.62 79.37) (end 94.75 80.5) (width 0.9) (layer "F.Cu") (net 10))
   (segment (start 90.56 79.37) (end 93.62 79.37) (width 0.9) (layer "F.Cu") (net 10))
+  (segment (start 93.5 75.0125) (end 93.5 79.25) (width 0.9) (layer "F.Cu") (net 10))
+  (segment (start 93.5 79.25) (end 93.62 79.37) (width 0.9) (layer "F.Cu") (net 10))
   (segment (start 91.5 87.25) (end 91.5 83.7226) (width 0.9) (layer "F.Cu") (net 10))
   (segment (start 99.5 118.54) (end 99.5 118.74) (width 0.25) (layer "F.Cu") (net 15))
