File: Hardware/GuitarPedal1590b/pcb/Power.kicad_sch (KiCad schematic)
At the start: 10 parts, among them U1 L4931CZ50, U2 PDS1-S5-S5-D

Commit message: Updated 1590b Schematic Rev 6
* Added a DNP SMD Resistor pad to optionally bypass the PDS1 isolated power components.
Parts:
- added R21: DNP, Resistor_SMD:R_0805_2012Metric, symbol Device:R
Connections:
- net +5V: now also R21.1
- net +5V_ISOLATED_POWER: now also R21.2
Changed lines of the file:
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@@
   (title_block
     (title "Daisy Seed Guitar Pedal 1590B")
-    (date "2023-06-03")
-    (rev "5")
+    (date "2023-11-12")
+    (rev "6")
     (company "Made by Keith Shepherd (kshep@mac.com)")
     (comment 1 "https://github.com/electro-smith/Hardware/blob/master/reference/daisy_petal/")
@@
   (junction (at 132.08 100.33) (diameter 0) (color 0 0 0 0)
   )
-  (junction (at 129.54 100.33) (diameter 0) (color 0 0 0 0)
-  )
   (junction (at 132.08 111.76) (diameter 0) (color 0 0 0 0)
   )
@@
   (junction (at 200.66 100.33) (diameter 0) (color 0 0 0 0)
   )
+  (junction (at 127 100.33) (diameter 0) (color 0 0 0 0)
+  )
   (wire (pts (xy 76.2 100.33) (xy 88.9 100.33))
     (stroke (width 0) (type default))
@@
     (stroke (width 0) (type default))
   )
+  (wire (pts (xy 180.34 86.36) (xy 200.66 86.36))
+    (stroke (width 0) (type default))
+  )
   (wire (pts (xy 151.13 115.57) (xy 200.66 115.57))
     (stroke (width 0) (type default))
@@
     (stroke (width 0) (type default))
   )
+  (wire (pts (xy 200.66 86.36) (xy 200.66 100.33))
+    (stroke (width 0) (type default))
+  )
   (wire (pts (xy 191.77 100.33) (xy 200.66 100.33))
     (stroke (width 0) (type default))
@@
     (stroke (width 0) (type default))
   )
-  (wire (pts (xy 125.73 100.33) (xy 129.54 100.33))
+  (wire (pts (xy 125.73 100.33) (xy 127 100.33))
     (stroke (width 0) (type default))
   )
@@
     (stroke (width 0) (type default))
   )
+  (wire (pts (xy 132.08 86.36) (xy 172.72 86.36))
+    (stroke (width 0) (type default))
+  )
   (wire (pts (xy 73.66 100.33) (xy 76.2 100.33))
     (stroke (width 0) (type default))
@@
     (stroke (width 0) (type default))
   )
-  (wire (pts (xy 129.54 90.17) (xy 129.54 100.33))
+  (wire (pts (xy 127 90.17) (xy 127 100.33))
     (stroke (width 0) (type default))
   )
@@
     (stroke (width 0) (type default))
   )
-  (wire (pts (xy 129.54 100.33) (xy 132.08 100.33))
+  (wire (pts (xy 127 100.33) (xy 132.08 100.33))
     (stroke (width 0) (type default))
   )
@@
   )
   (wire (pts (xy 151.13 111.76) (xy 161.29 111.76))
+    (stroke (width 0) (type default))
+  )
+  (wire (pts (xy 132.08 100.33) (xy 132.08 86.36))
     (stroke (width 0) (type default))
   )
@@
     )
   )
-  (symbol (lib_id "power:+5V") (at 129.54 90.17 0) (unit 1)
-    (in_bom yes) (on_board yes) (dnp no) (fields_autoplaced)
-    (property "Reference" "#PWR05" (at 129.54 93.98 0)
-      (effects (font (size 1.27 1.27)) hide)
-    )
-    (property "Value" "+5V" (at 129.54 85.09 0)
-      (effects (font (size 1.27 1.27)))
-    )
-    (property "Footprint" "" (at 129.54 90.17 0)
-      (effects (font (size 1.27 1.27)) hide)
-    )
-    (property "Datasheet" "" (at 129.54 90.17 0)
+  (symbol (lib_id "power:+5V") (at 127 90.17 0) (unit 1)
+    (in_bom yes) (on_board yes) (dnp no) (fields_autoplaced)
+    (property "Reference" "#PWR05" (at 127 93.98 0)
+      (effects (font (size 1.27 1.27)) hide)
+    )
+    (property "Value" "+5V" (at 127 85.09 0)
+      (effects (font (size 1.27 1.27)))
+    )
+    (property "Footprint" "" (at 127 90.17 0)
+      (effects (font (size 1.27 1.27)) hide)
+    )
+    (property "Datasheet" "" (at 127 90.17 0)
       (effects (font (size 1.27 1.27)) hide)
     )
@@
         )
       )
+    )
+  )
+  (symbol (lib_id "Device:R") (at 176.53 86.36 90) (unit 1)
+    (in_bom yes) (on_board yes) (dnp no) (fields_autoplaced)
+    (property "Reference" "R21" (at 176.53 80.01 90)
+      (effects (font (size 1.27 1.27)))
+    )
+    (property "Value" "DNP" (at 176.53 82.55 90)
+      (effects (font (size 1.27 1.27)))
+    )
+    (property "Footprint" "Resistor_SMD:R_0805_2012Metric" (at 176.53 88.138 90)
+      (effects (font (size 1.27 1.27)) hide)
+    )
+    (property "Datasheet" "~" (at 176.53 86.36 0)
+      (effects (font (size 1.27 1.27)) hide)
+    )
+    (pin "1")
+    (pin "2")
+    (instances
+      (project "DaisySeedPedal1590b"
+        (path "/1d54e6f4-7c7a-4f03-b2db-a136bdff5b99/52799331-6b0e-4f5c-8576-655b01bd4c42"
+          (reference "R21") (unit 1)
+        )
+      )
