File: Hardware/GuitarPedal125b/pcb/Audio_Input_Buffer.kicad_sch (KiCad schematic)
At the start: 11 parts, among them U3 MCP6004

Commit message: Hardware Rev 6
* Removed PDS1 to reduce cost and because it wasn't really helping anything
* Added low pass filter to address Rev7 Seed Noise issue
* Modified schematics and footprints to make it easier to have assembled by JLCPCB
Parts:
- renumbered C7 to C5, C8 to C6, C9 to C7, C10 to C8, U3 to U2
Connections:
- net +5V_ISOLATED_POWER renamed +5V
