File: Hardware/GuitarPedal125b/pcb/Audio_True_Bypass_Stereo.kicad_sch (KiCad schematic)
At the start: 10 parts, among them K1 G6K-2, K2 G6K-2, Q1 SS8050, U7 CPC1018N, U8 CPC1018N

Commit message: Rev6 WIP
Working on a fresh layout of the board.
Connections:
- net +5V_ISOLATED_POWER renamed +5V
Changed lines of the file:
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@@
-    )
-  )
-  (global_label "+5V_ISOLATED_POWER" (shape input) (at 135.89 40.64 90) (fields_autoplaced)
-    (effects (font (size 1.27 1.27)) (justify left))
-    (property "Intersheetrefs" "${INTERSHEET_REFS}" (at 135.89 16.8095 90)
-      (effects (font (size 1.27 1.27)) (justify left) hide)
     )
   )
@@
         )
       )
+    )
+  )
+  (symbol (lib_id "power:+5V") (at 135.89 40.64 0) (unit 1)
+    (in_bom yes) (on_board yes) (dnp no) (fields_autoplaced)
+    (property "Reference" "#PWR059" (at 135.89 44.45 0)
+      (effects (font (size 1.27 1.27)) hide)
+    )
+    (property "Value" "+5V" (at 135.89 35.56 0)
+      (effects (font (size 1.27 1.27)))
+    )
+    (property "Footprint" "" (at 135.89 40.64 0)
+      (effects (font (size 1.27 1.27)) hide)
+    )
+    (property "Datasheet" "" (at 135.89 40.64 0)
+      (effects (font (size 1.27 1.27)) hide)
+    )
+    (pin "1")
+    (instances
+      (project "DaisySeedPedal125b"
+        (path "/1d54e6f4-7c7a-4f03-b2db-a136bdff5b99/d5b1af0e-2179-4bcd-8e24-55fd6680ab7e"
+          (reference "#PWR059") (unit 1)
+        )
+      )
