File: Hardware/GuitarPedal125b/pcb/Audio_True_Bypass_Stereo.kicad_sch (KiCad schematic)
At the start: 10 parts, among them K1 G6K-2, K2 G6K-2, Q1 SS8050, U7 CPC1018N, U8 CPC1018N

Commit message: Hardware Rev 6
* Removed PDS1 to reduce cost and because it wasn't really helping anything
* Added low pass filter to address Rev7 Seed Noise issue
* Modified schematics and footprints to make it easier to have assembled by JLCPCB
Parts:
- renumbered R24 to R22, R25 to R23, U7 to U5, U8 to U6
Connections:
- net +5V_ISOLATED_POWER renamed +5V
Changed lines of the file:
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@@
   (title_block
     (title "Daisy Seed Guitar Pedal 125B")
-    (date "2023-06-30")
-    (rev "5")
+    (date "2024-02-25")
+    (rev "6")
     (company "Made by Keith Shepherd (kshep@mac.com)")
   )
@@
     )
   )
-  (global_label "+5V_ISOLATED_POWER" (shape input) (at 135.89 40.64 90) (fields_autoplaced)
-    (effects (font (size 1.27 1.27)) (justify left))
-    (property "Intersheetrefs" "${INTERSHEET_REFS}" (at 135.89 16.8095 90)
-      (effects (font (size 1.27 1.27)) (justify left) hide)
-    )
-  )
   (global_label "BYPASS_RIGHT_SEND" (shape output) (at 101.6 130.81 180) (fields_autoplaced)
     (effects (font (size 1.27 1.27)) (justify right))
     (property "Intersheetrefs" "${INTERSHEET_REFS}" (at 79.7136 130.8894 0)
       (effects (font (size 1.27 1.27)) (justify right) hide)
+    )
+  )
+  (symbol (lib_id "power:+5V") (at 135.89 40.64 0) (unit 1)
+    (in_bom yes) (on_board yes) (dnp no) (fields_autoplaced)
+    (property "Reference" "#PWR041" (at 135.89 44.45 0)
+      (effects (font (size 1.27 1.27)) hide)
+    )
+    (property "Value" "+5V" (at 135.89 35.56 0)
+      (effects (font (size 1.27 1.27)))
+    )
+    (property "Footprint" "" (at 135.89 40.64 0)
+      (effects (font (size 1.27 1.27)) hide)
+    )
+    (property "Datasheet" "" (at 135.89 40.64 0)
+      (effects (font (size 1.27 1.27)) hide)
+    )
+    (pin "1")
+    (instances
+      (project "DaisySeedPedal125b"
+        (path "/1d54e6f4-7c7a-4f03-b2db-a136bdff5b99/d5b1af0e-2179-4bcd-8e24-55fd6680ab7e"
+          (reference "#PWR041") (unit 1)
+        )
+      )
     )
   )
@@
   (symbol (lib_id "power:GND") (at 140.97 128.27 0) (unit 1)
     (in_bom yes) (on_board yes) (dnp no) (fields_autoplaced)
-    (property "Reference" "#PWR029" (at 140.97 134.62 0)
+    (property "Reference" "#PWR043" (at 140.97 134.62 0)
       (effects (font (size 1.27 1.27)) hide)
     )
@@
       (project "DaisySeedPedal125b"
         (path "/1d54e6f4-7c7a-4f03-b2db-a136bdff5b99/d5b1af0e-2179-4bcd-8e24-55fd6680ab7e"
-          (reference "#PWR029") (unit 1)
+          (reference "#PWR043") (unit 1)
         )
       )
@@
   (symbol (lib_id "Relay_SolidState:CPC1017N") (at 90.17 160.02 0) (unit 1)
     (in_bom yes) (on_board yes) (dnp no) (fields_autoplaced)
-    (property "Reference" "U7" (at 90.17 152.4 0)
+    (property "Reference" "U5" (at 90.17 152.4 0)
       (effects (font (size 1.27 1.27)))
     )
@@
       (project "DaisySeedPedal125b"
         (path "/1d54e6f4-7c7a-4f03-b2db-a136bdff5b99/d5b1af0e-2179-4bcd-8e24-55fd6680ab7e"
-          (reference "U7") (unit 1)
+          (reference "U5") (unit 1)
         )
       )
@@
   (symbol (lib_id "power:GND") (at 97.79 162.56 0) (unit 1)
     (in_bom yes) (on_board yes) (dnp no) (fields_autoplaced)
-    (property "Reference" "#PWR043" (at 97.79 168.91 0)
+    (property "Reference" "#PWR039" (at 97.79 168.91 0)
       (effects (font (size 1.27 1.27)) hide)
     )
@@
       (project "DaisySeedPedal125b"
         (path "/1d54e6f4-7c7a-4f03-b2db-a136bdff5b99/d5b1af0e-2179-4bcd-8e24-55fd6680ab7e"
-          (reference "#PWR043") (unit 1)
+          (reference "#PWR039") (unit 1)
         )
       )
@@
   (symbol (lib_id "Device:R") (at 78.74 157.48 90) (unit 1)
     (in_bom yes) (on_board yes) (dnp no) (fields_autoplaced)
-    (property "Reference" "R24" (at 78.74 152.4 90)
+    (property "Reference" "R22" (at 78.74 152.4 90)
       (effects (font (size 1.27 1.27)))
     )
@@
       (project "DaisySeedPedal125b"
         (path "/1d54e6f4-7c7a-4f03-b2db-a136bdff5b99/d5b1af0e-2179-4bcd-8e24-55fd6680ab7e"
-          (reference "R24") (unit 1)
+          (reference "R22") (unit 1)
         )
       )
@@
   (symbol (lib_id "power:GND") (at 40.64 95.25 0) (unit 1)
     (in_bom yes) (on_board yes) (dnp no)
-    (property "Reference" "#PWR018" (at 40.64 101.6 0)
+    (property "Reference" "#PWR036" (at 40.64 101.6 0)
       (effects (font (size 1.27 1.27)) hide)
     )
@@
       (project "DaisySeedPedal125b"
         (path "/1d54e6f4-7c7a-4f03-b2db-a136bdff5b99/d5b1af0e-2179-4bcd-8e24-55fd6680ab7e"
-          (reference "#PWR018") (unit 1)
+          (reference "#PWR036") (unit 1)
         )
       )
@@
   (symbol (lib_id "power:GND") (at 82.55 162.56 0) (unit 1)
     (in_bom yes) (on_board yes) (dnp no) (fields_autoplaced)
-    (property "Reference" "#PWR041" (at 82.55 168.91 0)
+    (property "Reference" "#PWR037" (at 82.55 168.91 0)
       (effects (font (size 1.27 1.27)) hide)
     )
@@
       (project "DaisySeedPedal125b"
         (path "/1d54e6f4-7c7a-4f03-b2db-a136bdff5b99/d5b1af0e-2179-4bcd-8e24-55fd6680ab7e"
-          (reference "#PWR041") (unit 1)
+          (reference "#PWR037") (unit 1)
         )
       )
@@
   (symbol (lib_id "Relay_SolidState:CPC1017N") (at 90.17 187.96 0) (unit 1)
     (in_bom yes) (on_board yes) (dnp no) (fields_autoplaced)
-    (property "Reference" "U8" (at 90.17 180.34 0)
+    (property "Reference" "U6" (at 90.17 180.34 0)
       (effects (font (size 1.27 1.27)))
     )
@@
       (project "DaisySeedPedal125b"
         (path "/1d54e6f4-7c7a-4f03-b2db-a136bdff5b99/d5b1af0e-2179-4bcd-8e24-55fd6680ab7e"
-          (reference "U8") (unit 1)
+          (reference "U6") (unit 1)
         )
       )
@@
   (symbol (lib_id "power:GND") (at 140.97 71.12 0) (unit 1)
     (in_bom yes) (on_board yes) (dnp no) (fields_autoplaced)
-    (property "Reference" "#PWR020" (at 140.97 77.47 0)
+    (property "Reference" "#PWR042" (at 140.97 77.47 0)
       (effects (font (size 1.27 1.27)) hide)
     )
@@
       (project "DaisySeedPedal125b"
         (path "/1d54e6f4-7c7a-4f03-b2db-a136bdff5b99/d5b1af0e-2179-4bcd-8e24-55fd6680ab7e"
-          (reference "#PWR020") (unit 1)
+          (reference "#PWR042") (unit 1)
         )
       )
@@
   (symbol (lib_id "power:GND") (at 97.79 190.5 0) (unit 1)
     (in_bom yes) (on_board yes) (dnp no) (fields_autoplaced)
-    (property "Reference" "#PWR044" (at 97.79 196.85 0)
+    (property "Reference" "#PWR040" (at 97.79 196.85 0)
       (effects (font (size 1.27 1.27)) hide)
     )
@@
       (project "DaisySeedPedal125b"
         (path "/1d54e6f4-7c7a-4f03-b2db-a136bdff5b99/d5b1af0e-2179-4bcd-8e24-55fd6680ab7e"
-          (reference "#PWR044") (unit 1)
+          (reference "#PWR040") (unit 1)
         )
       )
@@
   (symbol (lib_id "power:GND") (at 82.55 190.5 0) (unit 1)
     (in_bom yes) (on_board yes) (dnp no) (fields_autoplaced)
-    (property "Reference" "#PWR042" (at 82.55 196.85 0)
+    (property "Reference" "#PWR038" (at 82.55 196.85 0)
       (effects (font (size 1.27 1.27)) hide)
     )
@@
       (project "DaisySeedPedal125b"
         (path "/1d54e6f4-7c7a-4f03-b2db-a136bdff5b99/d5b1af0e-2179-4bcd-8e24-55fd6680ab7e"
-          (reference "#PWR042") (unit 1)
+          (reference "#PWR038") (unit 1)
         )
       )
@@
   (symbol (lib_id "Device:R") (at 78.74 185.42 90) (unit 1)
     (in_bom yes) (on_board yes) (dnp no) (fields_autoplaced)
-    (property "Reference" "R25" (at 78.74 180.34 90)
+    (property "Reference" "R23" (at 78.74 180.34 90)
       (effects (font (size 1.27 1.27)))
     )
@@
       (project "DaisySeedPedal125b"
         (path "/1d54e6f4-7c7a-4f03-b2db-a136bdff5b99/d5b1af0e-2179-4bcd-8e24-55fd6680ab7e"
-          (reference "R25") (unit 1)
-        )
-      )
+          (reference "R23") (unit 1)
+        )
+      )
