File: Hardware/GuitarPedal125b/pcb/Power.kicad_sch (KiCad schematic)
At the start: 10 parts, among them U1 LD1117S50TR_SOT223, U2 PDS1-S5-S5-M

Commit message: Rev6 WIP
Working on a fresh layout of the board.
Parts:
- removed C5: 10UF, Capacitor_SMD:C_0805_2012Metric, symbol Device:C
- removed C6: 22UF, Capacitor_SMD:C_0805_2012Metric, symbol Device:C
- removed L1: 2.2uH, Inductor_SMD:L_0805_2012Metric, symbol Device:L_Iron
- removed U2: PDS1-S5-S5-M, PDS1-S5-S5-M:CONV_PDS1-S5-S5-M, symbol PDS1-S5-S5-M:PDS1-S5-S5-M
