File: Hardware/GuitarPedal125b/pcb/Power.kicad_sch (KiCad schematic)
At the start: 10 parts, among them U1 LD1117S50TR_SOT223, U2 PDS1-S5-S5-M

Commit message: Hardware Rev 6
* Removed PDS1 to reduce cost and because it wasn't really helping anything
* Added low pass filter to address Rev7 Seed Noise issue
* Modified schematics and footprints to make it easier to have assembled by JLCPCB
Parts:
- removed C5: 10UF, Capacitor_SMD:C_0805_2012Metric, symbol Device:C
- removed C6: 22UF, Capacitor_SMD:C_0805_2012Metric, symbol Device:C
- removed L1: 2.2uH, Inductor_SMD:L_0805_2012Metric, symbol Device:L_Iron
- removed U2: PDS1-S5-S5-M, PDS1-S5-S5-M:CONV_PDS1-S5-S5-M, symbol PDS1-S5-S5-M:PDS1-S5-S5-M
