File: Hardware/GuitarPedal125b/pcb/Audio_Output_Buffer.kicad_sch (KiCad schematic)
At the start: 15 parts, among them U4 OPA1652AID

Commit message: Rev6 WIP
Working on a fresh layout of the board.
Connections:
- net +5V_ISOLATED_POWER renamed +5V
Changed lines of the file:
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@@
-    (stroke (width 0) (type default))
-  )
-  (wire (pts (xy 110.49 50.8) (xy 114.3 50.8))
     (stroke (width 0) (type default))
   )
@@
     (stroke (width 0) (type default))
   )
-  (wire (pts (xy 110.49 90.17) (xy 114.3 90.17))
-    (stroke (width 0) (type default))
-  )
   (wire (pts (xy 127 109.22) (xy 127 115.57))
     (stroke (width 0) (type default))
@@
     (stroke (width 0) (type default))
   )
-  (wire (pts (xy 114.3 93.98) (xy 114.3 90.17))
+  (wire (pts (xy 114.3 93.98) (xy 114.3 92.71))
     (stroke (width 0) (type default))
   )
@@
   (wire (pts (xy 147.32 106.68) (xy 147.32 115.57))
     (stroke (width 0) (type default))
-  )
-  (global_label "+5V_ISOLATED_POWER" (shape input) (at 110.49 50.8 180) (fields_autoplaced)
-    (effects (font (size 1.27 1.27)) (justify right))
-    (property "Intersheetrefs" "${INTERSHEET_REFS}" (at 87.1521 50.7206 0)
-      (effects (font (size 1.27 1.27)) (justify right) hide)
-    )
   )
   (global_label "AUDIO_OUT_BUFFER_RIGHT" (shape input) (at 77.47 104.14 180) (fields_autoplaced)
@@
     )
   )
-  (global_label "+5V_ISOLATED_POWER" (shape input) (at 137.16 134.62 180) (fields_autoplaced)
-    (effects (font (size 1.27 1.27)) (justify right))
-    (property "Intersheetrefs" "${INTERSHEET_REFS}" (at 113.8221 134.5406 0)
-      (effects (font (size 1.27 1.27)) (justify right) hide)
-    )
-  )
   (global_label "BYPASS_RIGHT_RETURN" (shape output) (at 203.2 87.63 0) (fields_autoplaced)
     (effects (font (size 1.27 1.27)) (justify left))
@@
     (effects (font (size 1.27 1.27)) (justify right))
     (property "Intersheetrefs" "${INTERSHEET_REFS}" (at 51.4712 64.6906 0)
-      (effects (font (size 1.27 1.27)) (justify right) hide)
-    )
-  )
-  (global_label "+5V_ISOLATED_POWER" (shape input) (at 110.49 90.17 180) (fields_autoplaced)
-    (effects (font (size 1.27 1.27)) (justify right))
-    (property "Intersheetrefs" "${INTERSHEET_REFS}" (at 87.1521 90.0906 0)
       (effects (font (size 1.27 1.27)) (justify right) hide)
     )
@@
     )
   )
+  (symbol (lib_id "power:+5V") (at 114.3 92.71 0) (unit 1)
+    (in_bom yes) (on_board yes) (dnp no) (fields_autoplaced)
+    (property "Reference" "#PWR057" (at 114.3 96.52 0)
+      (effects (font (size 1.27 1.27)) hide)
+    )
+    (property "Value" "+5V" (at 114.3 87.63 0)
+      (effects (font (size 1.27 1.27)))
+    )
+    (property "Footprint" "" (at 114.3 92.71 0)
+      (effects (font (size 1.27 1.27)) hide)
+    )
+    (property "Datasheet" "" (at 114.3 92.71 0)
+      (effects (font (size 1.27 1.27)) hide)
+    )
+    (pin "1")
+    (instances
+      (project "DaisySeedPedal125b"
+        (path "/1d54e6f4-7c7a-4f03-b2db-a136bdff5b99/56549882-0be3-4804-9aec-d28049bb2b53"
+          (reference "#PWR057") (unit 1)
+        )
+      )
+    )
+  )
   (symbol (lib_id "power:GND") (at 175.26 78.74 0) (unit 1)
     (in_bom yes) (on_board yes) (dnp no) (fields_autoplaced)
@@
         (path "/1d54e6f4-7c7a-4f03-b2db-a136bdff5b99/56549882-0be3-4804-9aec-d28049bb2b53"
           (reference "R8") (unit 1)
+        )
+      )
+    )
+  )
+  (symbol (lib_id "power:+5V") (at 137.16 134.62 0) (unit 1)
+    (in_bom yes) (on_board yes) (dnp no) (fields_autoplaced)
+    (property "Reference" "#PWR058" (at 137.16 138.43 0)
+      (effects (font (size 1.27 1.27)) hide)
+    )
+    (property "Value" "+5V" (at 137.16 129.54 0)
+      (effects (font (size 1.27 1.27)))
+    )
+    (property "Footprint" "" (at 137.16 134.62 0)
+      (effects (font (size 1.27 1.27)) hide)
+    )
+    (property "Datasheet" "" (at 137.16 134.62 0)
+      (effects (font (size 1.27 1.27)) hide)
+    )
+    (pin "1")
+    (instances
+      (project "DaisySeedPedal125b"
+        (path "/1d54e6f4-7c7a-4f03-b2db-a136bdff5b99/56549882-0be3-4804-9aec-d28049bb2b53"
+          (reference "#PWR058") (unit 1)
         )
       )
@@
         )
       )
+    )
+  )
+  (symbol (lib_id "power:+5V") (at 114.3 50.8 0) (unit 1)
+    (in_bom yes) (on_board yes) (dnp no) (fields_autoplaced)
+    (property "Reference" "#PWR056" (at 114.3 54.61 0)
+      (effects (font (size 1.27 1.27)) hide)
+    )
+    (property "Value" "+5V" (at 114.3 45.72 0)
+      (effects (font (size 1.27 1.27)))
+    )
+    (property "Footprint" "" (at 114.3 50.8 0)
+      (effects (font (size 1.27 1.27)) hide)
+    )
+    (property "Datasheet" "" (at 114.3 50.8 0)
+      (effects (font (size 1.27 1.27)) hide)
+    )
+    (pin "1")
+    (instances
+      (project "DaisySeedPedal125b"
+        (path "/1d54e6f4-7c7a-4f03-b2db-a136bdff5b99/56549882-0be3-4804-9aec-d28049bb2b53"
+          (reference "#PWR056") (unit 1)
+        )
+      )

Commit message: Initial layout of all major component blocks
Got all the components on the board, starting routing signals, maybe about half complete.
Parts:
- added C5, C6: 1.5NF, Capacitor_SMD:C_0805_2012Metric, symbol Device:C
- added R28, R29: 4.7K, Resistor_SMD:R_0805_2012Metric, symbol Device:R
Connections:
- net AUDIO_OUT_BUFFER_LEFT: now also R28.1; no longer C11.2
- net AUDIO_OUT_BUFFER_RIGHT: now also R29.1; no longer C12.2
- net GND: now also C5.2, C6.2
- new net: C11.2, C5.1, R28.2
- new net: C12.2, C6.1, R29.2
Other:
- note added: "Simple RC Low Pass Filter at 22kHz to remove out of band noise from Seed Rev7"
Changed lines of the file:
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@@
   (junction (at 147.32 106.68) (diameter 0) (color 0 0 0 0)
   )
+  (junction (at 77.47 104.14) (diameter 0) (color 0 0 0 0)
+  )
   (junction (at 152.4 153.67) (diameter 0) (color 0 0 0 0)
   )
@@
   (junction (at 114.3 104.14) (diameter 0) (color 0 0 0 0)
   )
+  (junction (at 77.47 64.77) (diameter 0) (color 0 0 0 0)
+  )
   (junction (at 114.3 64.77) (diameter 0) (color 0 0 0 0)
   )
@@
     (stroke (width 0) (type default))
   )
+  (wire (pts (xy 77.47 64.77) (xy 101.6 64.77))
+    (stroke (width 0) (type default))
+  )
   (wire (pts (xy 152.4 153.67) (xy 165.1 153.67))
     (stroke (width 0) (type default))
@@
     (stroke (width 0) (type default))
   )
+  (wire (pts (xy 77.47 104.14) (xy 101.6 104.14))
+    (stroke (width 0) (type default))
+  )
+  (wire (pts (xy 74.93 64.77) (xy 77.47 64.77))
+    (stroke (width 0) (type default))
+  )
   (wire (pts (xy 191.77 67.31) (xy 191.77 82.55))
     (stroke (width 0) (type default))
@@
     (stroke (width 0) (type default))
   )
+  (wire (pts (xy 77.47 76.2) (xy 77.47 78.74))
+    (stroke (width 0) (type default))
+  )
   (wire (pts (xy 137.16 138.43) (xy 152.4 138.43))
     (stroke (width 0) (type default))
@@
     (stroke (width 0) (type default))
   )
-  (wire (pts (xy 77.47 64.77) (xy 101.6 64.77))
+  (wire (pts (xy 77.47 115.57) (xy 77.47 118.11))
+    (stroke (width 0) (type default))
+  )
+  (wire (pts (xy 50.8 64.77) (xy 67.31 64.77))
     (stroke (width 0) (type default))
   )
@@
     (stroke (width 0) (type default))
   )
+  (wire (pts (xy 77.47 107.95) (xy 77.47 104.14))
+    (stroke (width 0) (type default))
+  )
   (wire (pts (xy 152.4 138.43) (xy 165.1 138.43))
     (stroke (width 0) (type default))
@@
     (stroke (width 0) (type default))
   )
+  (wire (pts (xy 76.2 104.14) (xy 77.47 104.14))
+    (stroke (width 0) (type default))
+  )
   (wire (pts (xy 147.32 115.57) (xy 127 115.57))
     (stroke (width 0) (type default))
@@
     (stroke (width 0) (type default))
   )
+  (wire (pts (xy 77.47 68.58) (xy 77.47 64.77))
+    (stroke (width 0) (type default))
+  )
   (wire (pts (xy 114.3 93.98) (xy 114.3 92.71))
     (stroke (width 0) (type default))
   )
-  (wire (pts (xy 77.47 104.14) (xy 101.6 104.14))
+  (wire (pts (xy 50.8 104.14) (xy 68.58 104.14))
     (stroke (width 0) (type default))
   )
@@
     (stroke (width 0) (type default))
   )
-  (global_label "AUDIO_OUT_BUFFER_RIGHT" (shape input) (at 77.47 104.14 180) (fields_autoplaced)
+  (rectangle (start 63.5 45.72) (end 92.71 129.54)
+    (stroke (width 0) (type default))
+    (fill (type none))
+  )
+  (text "Simple RC Low Pass Filter\nat 22kHz to remove out of\nband noise from Seed Rev7"
+    (at 64.77 53.34 0)
+    (effects (font (size 1.27 1.27)) (justify left bottom))
+  )
+  (global_label "AUDIO_OUT_BUFFER_RIGHT" (shape input) (at 50.8 104.14 180) (fields_autoplaced)
     (effects (font (size 1.27 1.27)) (justify right))
-    (property "Intersheetrefs" "${INTERSHEET_REFS}" (at 50.2617 104.0606 0)
+    (property "Intersheetrefs" "${INTERSHEET_REFS}" (at 23.5917 104.0606 0)
       (effects (font (size 1.27 1.27)) (justify right) hide)
     )
@@
     )
   )
-  (global_label "AUDIO_OUT_BUFFER_LEFT" (shape input) (at 77.47 64.77 180) (fields_autoplaced)
+  (global_label "AUDIO_OUT_BUFFER_LEFT" (shape input) (at 50.8 64.77 180) (fields_autoplaced)
     (effects (font (size 1.27 1.27)) (justify right))
-    (property "Intersheetrefs" "${INTERSHEET_REFS}" (at 51.4712 64.6906 0)
+    (property "Intersheetrefs" "${INTERSHEET_REFS}" (at 24.8012 64.6906 0)
       (effects (font (size 1.27 1.27)) (justify right) hide)
     )
@@
     )
   )
+  (symbol (lib_id "power:GND") (at 77.47 78.74 0) (unit 1)
+    (in_bom yes) (on_board yes) (dnp no) (fields_autoplaced)
+    (property "Reference" "#PWR061" (at 77.47 85.09 0)
+      (effects (font (size 1.27 1.27)) hide)
+    )
+    (property "Value" "GND" (at 77.47 83.82 0)
+      (effects (font (size 1.27 1.27)))
+    )
+    (property "Footprint" "" (at 77.47 78.74 0)
+      (effects (font (size 1.27 1.27)) hide)
+    )
+    (property "Datasheet" "" (at 77.47 78.74 0)
+      (effects (font (size 1.27 1.27)) hide)
+    )
+    (pin "1")
+    (instances
+      (project "DaisySeedPedal125b"
+        (path "/1d54e6f4-7c7a-4f03-b2db-a136bdff5b99/56549882-0be3-4804-9aec-d28049bb2b53"
+          (reference "#PWR061") (unit 1)
+        )
+      )
+    )
+  )
+  (symbol (lib_id "Device:R") (at 71.12 64.77 90) (unit 1)
+    (in_bom yes) (on_board yes) (dnp no) (fields_autoplaced)
+    (property "Reference" "R28" (at 71.12 58.42 90)
+      (effects (font (size 1.27 1.27)))
+    )
+    (property "Value" "4.7K" (at 71.12 60.96 90)
+      (effects (font (size 1.27 1.27)))
+    )
+    (property "Footprint" "Resistor_SMD:R_0805_2012Metric" (at 71.12 66.548 90)
+      (effects (font (size 1.27 1.27)) hide)
+    )
+    (property "Datasheet" "~" (at 71.12 64.77 0)
+      (effects (font (size 1.27 1.27)) hide)
+    )
+    (pin "1")
+    (pin "2")
+    (instances
+      (project "DaisySeedPedal125b"
+        (path "/1d54e6f4-7c7a-4f03-b2db-a136bdff5b99/56549882-0be3-4804-9aec-d28049bb2b53"
+          (reference "R28") (unit 1)
+        )
+      )
+    )
+  )
   (symbol (lib_id "power:+5V") (at 114.3 92.71 0) (unit 1)
     (in_bom yes) (on_board yes) (dnp no) (fields_autoplaced)
@@
         (path "/1d54e6f4-7c7a-4f03-b2db-a136bdff5b99/56549882-0be3-4804-9aec-d28049bb2b53"
           (reference "R7") (unit 1)
+        )
+      )
+    )
+  )
+  (symbol (lib_id "Device:C") (at 77.47 111.76 0) (unit 1)
+    (in_bom yes) (on_board yes) (dnp no) (fields_autoplaced)
+    (property "Reference" "C6" (at 81.28 110.49 0)
+      (effects (font (size 1.27 1.27)) (justify left))
+    )
+    (property "Value" "1.5NF" (at 81.28 113.03 0)
+      (effects (font (size 1.27 1.27)) (justify left))
+    )
+    (property "Footprint" "Capacitor_SMD:C_0805_2012Metric" (at 78.4352 115.57 0)
+      (effects (font (size 1.27 1.27)) hide)
+    )
+    (property "Datasheet" "~" (at 77.47 111.76 0)
+      (effects (font (size 1.27 1.27)) hide)
+    )
+    (pin "1")
+    (pin "2")
+    (instances
+      (project "DaisySeedPedal125b"
+        (path "/1d54e6f4-7c7a-4f03-b2db-a136bdff5b99/56549882-0be3-4804-9aec-d28049bb2b53"
+          (reference "C6") (unit 1)
         )
       )
@@
     )
   )
+  (symbol (lib_id "Device:R") (at 72.39 104.14 90) (unit 1)
+    (in_bom yes) (on_board yes) (dnp no) (fields_autoplaced)
+    (property "Reference" "R29" (at 72.39 97.79 90)
+      (effects (font (size 1.27 1.27)))
+    )
+    (property "Value" "4.7K" (at 72.39 100.33 90)
+      (effects (font (size 1.27 1.27)))
+    )
+    (property "Footprint" "Resistor_SMD:R_0805_2012Metric" (at 72.39 105.918 90)
+      (effects (font (size 1.27 1.27)) hide)
+    )
+    (property "Datasheet" "~" (at 72.39 104.14 0)
+      (effects (font (size 1.27 1.27)) hide)
+    )
+    (pin "2")
+    (pin "1")
+    (instances
+      (project "DaisySeedPedal125b"
+        (path "/1d54e6f4-7c7a-4f03-b2db-a136bdff5b99/56549882-0be3-4804-9aec-d28049bb2b53"
+          (reference "R29") (unit 1)
+        )
+      )
+    )
+  )
   (symbol (lib_id "Device:C") (at 167.64 67.31 90) (unit 1)
     (in_bom yes) (on_board yes) (dnp no) (fields_autoplaced)
@@
         (path "/1d54e6f4-7c7a-4f03-b2db-a136bdff5b99/56549882-0be3-4804-9aec-d28049bb2b53"
           (reference "C15") (unit 1)
+        )
+      )
+    )
+  )
+  (symbol (lib_id "Device:C") (at 77.47 72.39 0) (unit 1)
+    (in_bom yes) (on_board yes) (dnp no) (fields_autoplaced)
+    (property "Reference" "C5" (at 81.28 71.12 0)
+      (effects (font (size 1.27 1.27)) (justify left))
+    )
+    (property "Value" "1.5NF" (at 81.28 73.66 0)
+      (effects (font (size 1.27 1.27)) (justify left))
+    )
+    (property "Footprint" "Capacitor_SMD:C_0805_2012Metric" (at 78.4352 76.2 0)
+      (effects (font (size 1.27 1.27)) hide)
+    )
+    (property "Datasheet" "~" (at 77.47 72.39 0)
+      (effects (font (size 1.27 1.27)) hide)
+    )
+    (pin "1")
+    (pin "2")
+    (instances
+      (project "DaisySeedPedal125b"
+        (path "/1d54e6f4-7c7a-4f03-b2db-a136bdff5b99/56549882-0be3-4804-9aec-d28049bb2b53"
+          (reference "C5") (unit 1)
         )
       )
@@
         )
       )
+    )
+  )
+  (symbol (lib_id "power:GND") (at 77.47 118.11 0) (unit 1)
+    (in_bom yes) (on_board yes) (dnp no) (fields_autoplaced)
+    (property "Reference" "#PWR062" (at 77.47 124.46 0)
+      (effects (font (size 1.27 1.27)) hide)
+    )
+    (property "Value" "GND" (at 77.47 123.19 0)
+      (effects (font (size 1.27 1.27)))
+    )
+    (property "Footprint" "" (at 77.47 118.11 0)
+      (effects (font (size 1.27 1.27)) hide)
+    )
+    (property "Datasheet" "" (at 77.47 118.11 0)
+      (effects (font (size 1.27 1.27)) hide)
+    )
+    (pin "1")
+    (instances
+      (project "DaisySeedPedal125b"
+        (path "/1d54e6f4-7c7a-4f03-b2db-a136bdff5b99/56549882-0be3-4804-9aec-d28049bb2b53"
+          (reference "#PWR062") (unit 1)
+        )
+      )
