File: Hardware/GuitarPedal125b/pcb/Audio_Output_Buffer.kicad_sch (KiCad schematic)
At the start: 15 parts, among them U4 OPA1652AID

Commit message: Hardware Rev 6
* Removed PDS1 to reduce cost and because it wasn't really helping anything
* Added low pass filter to address Rev7 Seed Noise issue
* Modified schematics and footprints to make it easier to have assembled by JLCPCB
Parts:
- added C10, C9: 2.2NF, Capacitor_SMD:C_0805_2012Metric, symbol Device:C
- added R7, R8: 3.3K, Resistor_SMD:R_0805_2012Metric, symbol Device:R
- renumbered R8 to R10, R9 to R11, R10 to R12, R11 to R13, R12 to R14, R13 to R15, R14 to R16, R7 to R9, U4 to U3
Connections:
- net AUDIO_OUT_BUFFER_LEFT: now also R7.1; no longer C11.2
- net AUDIO_OUT_BUFFER_RIGHT: now also R8.1; no longer C12.2
- net GND: now also C10.2, C9.2
- net +5V_ISOLATED_POWER renamed +5V
- new net: C11.2, C9.1, R7.2
- new net: C10.1, C12.2, R8.2
Other:
- note added: "Simple RC Low Pass Filter at ~22kHz to remove out of band noise from Seed Rev7"
