File: Hardware/GuitarPedal125b/pcb/DaisySeedPedal125b.kicad_pcb (KiCad board)
At the start: 4 copper layers, 60 x 94 mm, 79 parts, among them J1 Barrel_Jack_Switch, J2 AUDIO_IN_TRS, J3 AUDIO_OUT_TRS, J4 MIDI IN JACK, J5 MIDI OUT JACK, K1 G6K-2, K2 G6K-2, Q1 SS8050, U1 LD1117S50TR_SOT223, U2 PDS1-S5-S5-M, U3 MCP6004, U4 OPA1652AID, U5 H11L1, U6 OLED_DISPLAY_SSD1306_SPI, U7 CPC1018N, U8 CPC1018N

Commit message: Rev6 WIP
Working on a fresh layout of the board.
Parts:
- removed A1: Electrosmith_Daisy_Seed_Rev4, Module:Electrosmith_Daisy_Seed
- removed C5: 10UF, Capacitor_SMD:C_0805_2012Metric
- removed C6: 22UF, Capacitor_SMD:C_0805_2012Metric
- removed L1: 2.2uH, Inductor_SMD:L_0805_2012Metric
- removed U2: PDS1-S5-S5-M, PDS1-S5-S5-M:CONV_PDS1-S5-S5-M
- added J4: AUDIO_OUT_LEFT, GuitarPedal125B:Generic_Pads_AudioTS, F.Cu at (167.0, 100.8)
- added J7: MIDI_OUT, GuitarPedal125B:Generic_Pads_AudioTRS, F.Cu at (156.0, 45.2)
- added J8: Conn_01x20_Socket, Connector_PinSocket_2.54mm:PinSocket_1x20_P2.54mm_Vertical, F.Cu at (134.4, 91.8)
- added J9: Conn_01x20_Socket, Connector_PinSocket_2.54mm:PinSocket_1x20_P2.54mm_Vertical, F.Cu at (149.6, 43.5)
- J1: value Barrel_Jack_Switch -> POWER_JACK; footprint GuitarPedal125B:Generic_PowerJack -> GuitarPedal125B:Generic_Pads_Power
- J2: value AUDIO_IN_TRS -> AUDIO_IN_LEFT; footprint NMJ6HCD2:NEUTRIK_NMJ6HCD2 -> GuitarPedal125B:Generic_Pads_AudioTS
- J3: value AUDIO_OUT_TRS -> AUDIO_IN_RIGHT; footprint NMJ6HCD2:NEUTRIK_NMJ6HCD2 -> GuitarPedal125B:Generic_Pads_AudioTS
- J5: value MIDI OUT JACK -> AUDIO_OUT_RIGHT; footprint AudioConnector-PJ320A:TRRS-PJ-320A -> GuitarPedal125B:Generic_Pads_AudioTS
- J6: renamed from J4; value MIDI IN JACK -> MIDI_IN; footprint AudioConnector-PJ320A:TRRS-PJ-320A -> GuitarPedal125B:Generic_Pads_AudioTRS
- moved C10 95.1 mm to (225.4, 84.8)
- moved C11 95.1 mm to (252.0, 81.0)
- moved C12 95.1 mm to (254.3, 81.0)
- moved C14 95.1 mm to (245.8, 90.2)
- moved C15 95.1 mm to (227.6, 95.5)
- moved C16 95.1 mm to (225.3, 88.9)
- moved C7 95.1 mm to (235.3, 87.9)
- moved C8 95.1 mm to (235.3, 90.2)
- moved C9 95.1 mm to (225.3, 81.0)
- moved D3 95.1 mm to (210.0, 96.4)
- moved D4 95.1 mm to (210.0, 84.4)
- moved K1 95.1 mm to (216.8, 82.7)
- moved R1 95.1 mm to (223.1, 81.0)
- moved R10 95.1 mm to (254.3, 84.7)
- moved R12 95.1 mm to (227.5, 88.9)
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Connections:
- C13 pad 1: +5V_ISOLATED_POWER -> +5V
- C14 pad 1: +5V_ISOLATED_POWER -> +5V
- C7 pad 1: +5V_ISOLATED_POWER -> +5V
- C8 pad 1: +5V_ISOLATED_POWER -> +5V
- D3 pad 1: +5V_ISOLATED_POWER -> +5V
- D4 pad 1: +5V_ISOLATED_POWER -> +5V
- J3 pad T: AUDIO_OUT_JACK_LEFT -> AUDIO_IN_JACK_RIGHT
- J5 pad T: MIDI_OUT_JACK_PIN5 -> AUDIO_OUT_JACK_RIGHT
- K1 pad 1: +5V_ISOLATED_POWER -> +5V
- K2 pad 1: +5V_ISOLATED_POWER -> +5V
- R3 pad 1: +5V_ISOLATED_POWER -> +5V
- R7 pad 1: +5V_ISOLATED_POWER -> +5V
- R9 pad 1: +5V_ISOLATED_POWER -> +5V
- U3 pad 4: +5V_ISOLATED_POWER -> +5V
- U4 pad 8: +5V_ISOLATED_POWER -> +5V
Routing:
- net Net-(LED1-A): track 124.9 -> 0.00 mm, vias 1 -> 0
- net +3.3VA: track 81.6 -> 0.00 mm
- net Net-(LED2-A): track 80.1 -> 0.00 mm, vias 1 -> 0
- net FOOT_SWITCH_1: track 69.5 -> 0.00 mm
- net AUDIO_OUT_JACK_LEFT: track 62.0 -> 0.00 mm, vias 2 -> 0
- net FOOT_SWITCH_2: track 59.3 -> 0.00 mm
- net AUDIO_OUT_JACK_RIGHT: track 57.1 -> 0.00 mm, vias 2 -> 0
- net ENCODER_1_CLICK: track 54.1 -> 0.00 mm
- net Net-(ENC1-PadA): track 55.6 -> 5.59 mm, vias 1 -> 0
- net +5V_ISOLATED_POWER: track 48.5 -> 0.00 mm
- net MIDI_OUT: track 43.9 -> 0.00 mm
- net Net-(ENC1-PadB): track 49.1 -> 5.48 mm, vias 1 -> 0
- net POT_3: track 38.4 -> 0.00 mm
- net AUDIO_IN_JACK_LEFT: track 46.9 -> 11.7 mm, vias 1 -> 0
- net GND: track 55.4 -> 20.4 mm, vias 40 -> 9
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- added copper zone on B.Cu, net +3.3VA
- added copper zone on F.Cu, net +5V
- removed copper zone on F.Cu, net +5V_ISOLATED_POWER
Other:
- board text added: "Daisy Seed Guitar Pedal 125B (Rev 6 Test) Made by Keith Shepherd 1/19/2024"
- board text removed: "Daisy Seed Guitar Pedal 125B (Rev 5) Made by Keith Shepherd 6/30/2023"
- board text removed: "J4"
- board text removed: "J5"

Commit message: Initial layout of all major component blocks
Got all the components on the board, starting routing signals, maybe about half complete.
Parts:
- added C5: 1.5NF, Capacitor_SMD:C_0805_2012Metric, F.Cu at (164.5, 92.6)
- added C6: 1.5NF, Capacitor_SMD:C_0805_2012Metric, F.Cu at (157.9, 92.6)
- added R28: 4.7K, Resistor_SMD:R_0805_2012Metric, F.Cu at (166.7, 92.6)
- added R29: 4.7K, Resistor_SMD:R_0805_2012Metric, F.Cu at (155.7, 92.6)
- moved C10 108.4 mm to (117.5, 96.3)
- moved C7 108.4 mm to (127.5, 99.5)
- moved C8 108.4 mm to (127.5, 101.8)
- moved C9 108.4 mm to (117.5, 92.6)
- moved R1 108.4 mm to (115.3, 92.6)
- moved R2 108.4 mm to (115.3, 96.3)
- moved R3 108.4 mm to (124.2, 100.5)
- moved R4 108.4 mm to (119.8, 92.6)
- moved R5 108.4 mm to (119.8, 96.3)
- moved R6 108.4 mm to (122.0, 100.5)
- moved U3 108.4 mm to (125.8, 94.5)
- moved R9 99.3 mm to (157.9, 96.3)
- moved U8 96.3 mm to (164.4, 118.7), turned to 180 degrees
- moved R10 95.0 mm to (160.0, 96.3), turned to 90 degrees
- moved C12 94.9 mm to (160.1, 92.6)
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Connections:
- C11 pad 2: AUDIO_OUT_BUFFER_LEFT -> Net-(C11-Pad2)
- C12 pad 2: AUDIO_OUT_BUFFER_RIGHT -> Net-(C12-Pad2)
Routing:
- net AUDIO_OUT_BUFFER_LEFT: track 0.00 -> 39.3 mm
- net AUDIO_OUT_JACK_LEFT: track 0.00 -> 30.9 mm
- net AUDIO_OUT_BUFFER_RIGHT: track 0.00 -> 28.1 mm
- net AUDIO_IN_JACK_RIGHT: track 11.8 -> 38.0 mm
- net AUDIO_OUT_JACK_RIGHT: track 0.00 -> 23.7 mm
- net Net-(U4A--): track 26.5 -> 3.80 mm, vias 2 -> 0
- net AUDIO_IN_BUFFER_LEFT: track 1.27 -> 19.0 mm
- net BYPASS_LEFT_RETURN: track 18.8 -> 1.97 mm, vias 2 -> 0
- net BYPASS_RIGHT_SEND: track 18.6 -> 2.27 mm
- net AUDIO_IN_BUFFER_RIGHT: track 1.27 -> 15.6 mm
- net Net-(U4B--): track 19.9 -> 6.10 mm, vias 2 -> 0
- net GND: track 20.4 -> 30.5 mm, vias 9 -> 18
- net AUDIO_IN_JACK_LEFT: track 11.7 -> 18.5 mm
- net BYPASS_LEFT_SEND: track 8.48 -> 2.23 mm
- net Net-(C12-Pad2): track 0.00 -> 5.16 mm
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
Commit message: More routing
Parts:
- moved R1 15.0 mm to (126.6, 102.4)
- moved R2 15.0 mm to (126.6, 106.1)
- moved C9 12.0 mm to (124.4, 102.4)
- moved C10 11.9 mm to (124.4, 106.0)
- moved C8 11.5 mm to (117.0, 96.9), turned to -90 degrees
- moved R4 10.0 mm to (122.2, 102.3)
- moved R5 9.87 mm to (122.2, 105.9)
- moved R6 9.76 mm to (118.3, 91.4), turned to 180 degrees
- moved R3 9.01 mm to (118.3, 93.7), turned to 0 degrees
- moved C7 8.55 mm to (119.3, 96.9), turned to -90 degrees
- moved C18 2.45 mm to (144.2, 120.8)
- moved C19 2.45 mm to (144.2, 116.5)
- moved R22 2.45 mm to (141.9, 120.8)
- moved R23 2.45 mm to (141.9, 116.5)
- moved R26 2.45 mm to (139.7, 120.8)
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Routing:
- net Net-(LED1-A): track 0.00 -> 108.0 mm, vias 0 -> 1
- net Net-(LED2-A): track 0.00 -> 74.3 mm, vias 0 -> 1
- net OLED_DISPLAY_SPI_SCK: track 0.00 -> 58.8 mm, vias 0 -> 1
- net OLED_DISPLAY_SPI_CS: track 0.00 -> 55.9 mm
- net OLED_DISPLAY_SPI_MOSI: track 0.00 -> 51.1 mm, vias 0 -> 1
- net OLED_DISPLAY_SPI_DC: track 0.00 -> 50.4 mm
- net OLED_DISPLAY_SPI_RESET: track 0.00 -> 48.3 mm
- net POT_3: track 0.00 -> 46.3 mm, vias 0 -> 1
- net MIDI_IN: track 2.70 -> 42.3 mm, vias 0 -> 1
- net POT_2: track 0.00 -> 37.9 mm, vias 0 -> 1
- net POT_1: track 0.00 -> 35.6 mm
- net POT_6: track 0.00 -> 35.3 mm, vias 0 -> 1
- net BYPASS_RIGHT_SEND: track 2.27 -> 23.5 mm
- net +3.3V: track 23.8 -> 44.9 mm, vias 0 -> 2
- net GND: track 30.5 -> 48.9 mm, vias 18 -> 30
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
Commit message: Continuing to work on Rev 6
Parts:
- added J10: Conn_01x07_Pin, Connector_Molex:Molex_PicoBlade_53398-0771_1x07-1MP_P1.25mm_Vertical, F.Cu at (141.2, 70.8)
- added J11: Conn_01x05_Pin, Connector_PinHeader_2.54mm:PinHeader_1x05_P2.54mm_Vertical, F.Cu at (153.2, 66.4)
- added J12: Conn_01x02_Pin, Connector_PinHeader_2.54mm:PinHeader_1x02_P2.54mm_Vertical, F.Cu at (130.8, 76.6)
- added J13: Conn_01x01_Pin, Connector_PinHeader_2.54mm:PinHeader_1x01_P2.54mm_Vertical, F.Cu at (130.8, 43.6)
- U6: footprint GuitarPedal125B:HiLetgo_OLED_SPI -> GuitarPedal125B:HiLetgo_OLED_SPI_NOPINS
- moved R18 12.6 mm to (115.2, 75.6), turned to 0 degrees
- moved C17 11.7 mm to (120.6, 75.6), turned to 180 degrees
- moved R21 3.23 mm to (143.7, 92.0), turned to -90 degrees
- moved U5 1.92 mm to (117.9, 68.4), turned to -90 degrees
- moved Q1 1.81 mm to (140.2, 92.0)
- moved U6 0.47 mm to (142.0, 98.0), turned to 180 degrees
Routing:
- net OLED_DISPLAY_SPI_SCK: track 58.8 -> 9.31 mm, vias 1 -> 0
- net POT_3: track 46.3 -> 0.00 mm, vias 1 -> 0
- net OLED_DISPLAY_SPI_CS: track 55.9 -> 10.6 mm
- net OLED_DISPLAY_SPI_MOSI: track 51.1 -> 7.37 mm, vias 1 -> 0
- net OLED_DISPLAY_SPI_DC: track 50.4 -> 8.02 mm
- net MIDI_IN: track 42.3 -> 0.00 mm, vias 1 -> 0
- net OLED_DISPLAY_SPI_RESET: track 48.3 -> 6.84 mm
- net MIDI_IN_JACK_PIN5: track 28.6 -> 6.22 mm
- net Net-(D2-K): track 21.0 -> 2.56 mm
- net ENABLE_AUDIO_MUTE: track 17.7 -> 7.05 mm, vias 1 -> 0
- net +3.3V: track 44.9 -> 39.7 mm
- net POT_6: track 35.3 -> 30.7 mm
- net MIDI_OUT: track 16.9 -> 12.9 mm
- net Net-(J13-Pin_1): track 0.00 -> 3.57 mm
- net Net-(J12-Pin_1): track 0.00 -> 3.56 mm
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
Commit message: more work on layout
Parts:
- moved K2 3.69 mm to (146.6, 105.3)
- moved K1 3.62 mm to (137.4, 105.3)
- moved R21 3.60 mm to (143.7, 95.6)
- moved D3 3.60 mm to (144.5, 98.6)
- moved D4 3.60 mm to (139.5, 98.6)
- moved Q1 3.60 mm to (140.2, 95.6)
Routing:
- net BYPASS_LEFT_RETURN: track 1.97 -> 23.7 mm
- net BYPASS_RIGHT_RETURN: track 1.97 -> 10.0 mm
- net AUDIO_IN_JACK_RIGHT: track 38.0 -> 31.1 mm
- net AUDIO_OUT_JACK_LEFT: track 31.4 -> 27.5 mm, vias 0 -> 2
- net BYPASS_LEFT_SEND: track 9.77 -> 11.7 mm
- net AUDIO_OUT_JACK_RIGHT: track 23.7 -> 25.0 mm, vias 0 -> 2
- net AUDIO_OUT_BUFFER_LEFT: track 39.1 -> 38.0 mm
- net AUDIO_OUT_BUFFER_RIGHT: track 26.5 -> 25.5 mm
- net BYPASS_RIGHT_SEND: track 23.5 -> 24.2 mm
- net Net-(D3-A): track 16.8 -> 16.1 mm

Commit message: More work on layout
Parts:
- J11: value Conn_01x05_Pin -> Conn_01x07_Pin; footprint Connector_PinHeader_2.54mm:PinHeader_1x05_P2.54mm_Vertical -> Connector_PinHeader_2.54mm:PinHeader_1x07_P2.54mm_Vertical
- J12: value Conn_01x02_Pin -> ALT_POWER_JACK; footprint Connector_PinHeader_2.54mm:PinHeader_1x02_P2.54mm_Vertical -> GuitarPedal125B:Generic_Pads_Power
- J6, J7: moved to B.Cu
- moved R17 39.8 mm to (131.5, 75.7)
- moved R16 39.5 mm to (129.4, 75.7)
- moved J7 36.6 mm to (130.7, 71.7), turned to 0 degrees
- moved J12 30.4 mm to (130.3, 46.1), turned to 180 degrees
- moved J6 18.2 mm to (130.6, 61.7), turned to 0 degrees
- moved D2 15.9 mm to (115.4, 63.9), turned to 180 degrees
- moved C17 15.0 mm to (127.8, 62.5), turned to 90 degrees
- moved R15 14.2 mm to (116.7, 60.4), turned to -90 degrees
- moved R18 9.60 mm to (124.7, 74.0)
- moved J13 7.45 mm to (130.3, 51.0)
- moved U5 2.72 mm to (120.6, 68.6), turned to 0 degrees
- moved J1 2.66 mm to (138.5, 46.1), turned to 180 degrees
Connections:
- J10 pad 1: OLED_DISPLAY_SPI_RESET -> OLED_DISPLAY_SPI_CS
- J10 pad 2: OLED_DISPLAY_SPI_MOSI -> OLED_DISPLAY_SPI_DC
- J10 pad 3: OLED_DISPLAY_SPI_DC -> OLED_DISPLAY_SPI_RESET
- J10 pad 4: OLED_DISPLAY_SPI_SCK -> OLED_DISPLAY_SPI_MOSI
- J10 pad 5: OLED_DISPLAY_SPI_CS -> OLED_DISPLAY_SPI_SCK
- J12 pad 1: Net-(J12-Pin_1) -> GND
- J12 pad 2: Net-(J12-Pin_2) -> POWER_JACK_PWR
- J8 pad 6: Net-(J12-Pin_2) -> MIDI_IN
- J8 pad 7: Net-(J12-Pin_1) -> MIDI_OUT
- J9 pad 4: MIDI_IN -> Net-(J11-Pin_7)
- J9 pad 5: MIDI_OUT -> Net-(J11-Pin_6)
Routing:
- net MIDI_OUT: track 12.9 -> 2.89 mm
- net MIDI_OUT_JACK_PIN5: track 0.00 -> 8.79 mm
- net POWER_JACK_PWR: track 4.81 -> 13.1 mm
- net MIDI_OUT_JACK_PIN4: track 0.00 -> 7.44 mm
- net MIDI_IN_JACK_PIN5: track 6.22 -> 0.00 mm
- net OLED_DISPLAY_SPI_CS: track 10.6 -> 16.5 mm, vias 0 -> 1
- net OLED_DISPLAY_SPI_DC: track 8.02 -> 13.7 mm
- net Net-(J13-Pin_1): track 3.57 -> 0.00 mm
- net Net-(J12-Pin_1): track 3.56 -> 0.00 mm
- net Net-(J12-Pin_2): track 3.56 -> 0.00 mm
- net Net-(J11-Pin_7): track 0.00 -> 3.56 mm
- net Net-(J11-Pin_6): track 0.00 -> 3.56 mm
- net MIDI_IN_JACK_PIN4: track 3.23 -> 0.00 mm
- net Net-(D2-K): track 2.56 -> 0.00 mm
- net GND: track 45.3 -> 46.6 mm, vias 28 -> 29
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