File: Hardware/GuitarPedal125b/pcb/DaisySeedPedal125b.kicad_pcb (KiCad board)
At the start: 4 copper layers, 60 x 94 mm, 79 parts, among them J1 Barrel_Jack_Switch, J2 AUDIO_IN_TRS, J3 AUDIO_OUT_TRS, J4 MIDI IN JACK, J5 MIDI OUT JACK, K1 G6K-2, K2 G6K-2, Q1 SS8050, U1 LD1117S50TR_SOT223, U2 PDS1-S5-S5-M, U3 MCP6004, U4 OPA1652AID, U5 H11L1, U6 OLED_DISPLAY_SSD1306_SPI, U7 CPC1018N, U8 CPC1018N

Commit message: Hardware Rev 6
* Removed PDS1 to reduce cost and because it wasn't really helping anything
* Added low pass filter to address Rev7 Seed Noise issue
* Modified schematics and footprints to make it easier to have assembled by JLCPCB
Parts:
- removed A1: Electrosmith_Daisy_Seed_Rev4, Module:Electrosmith_Daisy_Seed
- removed the C5 at (151.0, 55.5)
- removed the C6 at (160.8, 66.0)
- removed L1: 2.2uH, Inductor_SMD:L_0805_2012Metric
- removed the U2 at (152.9, 63.2)
- added C10: 2.2NF, Capacitor_SMD:C_0805_2012Metric, F.Cu at (163.2, 96.0)
- added C9: 2.2NF, Capacitor_SMD:C_0805_2012Metric, F.Cu at (156.4, 96.0)
- added J6: Conn_01x20_Socket, GuitarPedal125B:PinSocket1x20_P2.54mm_Vertical_JLCPCB, F.Cu at (138.4, 74.0)
- added J7: Conn_01x20_Socket, GuitarPedal125B:PinSocket1x20_P2.54mm_Vertical_JLCPCB, F.Cu at (138.4, 89.3)
- added R7: 3.3K, Resistor_SMD:R_0805_2012Metric, F.Cu at (158.1, 92.4)
- added R8: 3.3K, Resistor_SMD:R_0805_2012Metric, F.Cu at (161.6, 92.4)
- J3: renamed from J4; footprint AudioConnector-PJ320A:TRRS-PJ-320A -> GuitarPedal125B:PJ-320A
- J5: footprint AudioConnector-PJ320A:TRRS-PJ-320A -> GuitarPedal125B:PJ-320A
- moved J3 7.27 mm to (121.8, 48.5), turned to -90 degrees
- moved J5 7.27 mm to (162.2, 48.5), turned to -90 degrees
- moved J1 3.72 mm to (130.2, 50.2)
- moved C11 0.99 mm to (158.7, 96.0)
- moved C12 0.99 mm to (160.9, 96.0)
- moved R11 0.99 mm to (163.2, 99.6)
- moved R9 0.99 mm to (156.4, 99.6)
- moved R10 0.96 mm to (158.7, 99.6)
- moved R12 0.89 mm to (160.9, 99.6)
- moved C4 0.29 mm to (150.9, 51.8)
- turned U4 to 180 degrees
- renumbered C7 to C5, C8 to C6, C9 to C7, C10 to C8, J3 to J4, R8 to R10, R9 to R11, R10 to R12, R11 to R13, R12 to R14, R13 to R15, R14 to R16, R15 to R17, R17 to R18, R16 to R19, R18 to R20, R24 to R22, R25 to R23, R19 to R24, R20 to R25, R22 to R26, R23 to R27, R26 to R28, R27 to R29, R7 to R9, U3 to U2, U4 to U3, U5 to U4, U7 to U5, U8 to U6, U6 to U7
Connections:
- C11 pad 2: AUDIO_OUT_BUFFER_LEFT -> Net-(C11-Pad2)
- C12 pad 2: AUDIO_OUT_BUFFER_RIGHT -> Net-(C10-Pad1)
- C13 pad 1: +5V_ISOLATED_POWER -> +5V
- C14 pad 1: +5V_ISOLATED_POWER -> +5V
- C5 pad 1: +5V_ISOLATED_POWER -> +5V
- C6 pad 1: +5V_ISOLATED_POWER -> +5V
- D3 pad 1: +5V_ISOLATED_POWER -> +5V
- D4 pad 1: +5V_ISOLATED_POWER -> +5V
- K1 pad 1: +5V_ISOLATED_POWER -> +5V
- K2 pad 1: +5V_ISOLATED_POWER -> +5V
- R11 pad 1: +5V_ISOLATED_POWER -> +5V
- R3 pad 1: +5V_ISOLATED_POWER -> +5V
- R9 pad 1: +5V_ISOLATED_POWER -> +5V
- U2 pad 4: +5V_ISOLATED_POWER -> +5V
- U3 pad 8: +5V_ISOLATED_POWER -> +5V
Routing:
- net +5V: track 11.2 -> 73.7 mm, vias 0 -> 2
- net +5V_ISOLATED_POWER: track 48.5 -> 0.00 mm
- net /Power/VIN: track 10.5 -> 0.00 mm
- net GND: track 55.4 -> 49.5 mm, vias 40 -> 38
- net Net-(C11-Pad2): track 0.00 -> 5.28 mm
- net Net-(C10-Pad1): track 0.00 -> 5.21 mm
- net AUDIO_OUT_BUFFER_RIGHT: track 5.22 -> 3.45 mm
- net AUDIO_OUT_BUFFER_LEFT: track 5.34 -> 3.81 mm
- net Net-(U3B-+): track 11.6 -> 12.5 mm
- net Net-(U3A-+): track 16.2 -> 16.8 mm
- added copper zone on F.Cu, net +5V
- removed copper zone on F.Cu, net +5V_ISOLATED_POWER
Other:
- board text added: "Daisy Seed Guitar Pedal 125B (Rev 6) Made by Keith Shepherd 2/25/2024"
- board text removed: "Daisy Seed Guitar Pedal 125B (Rev 5) Made by Keith Shepherd 6/30/2023"
