File: Hardware/GuitarPedal125b/pcb/DaisySeedPedal125b.kicad_sch (KiCad schematic)
At the start: 6 parts, among them J1 Barrel_Jack_Switch, J2 AUDIO_IN_TRS, J3 AUDIO_OUT_TRS, J4 MIDI IN JACK, J5 MIDI OUT JACK

Commit message: Rev6 WIP
Working on a fresh layout of the board.
Parts:
- removed J3: AUDIO_OUT_TRS, NMJ6HCD2:NEUTRIK_NMJ6HCD2, symbol NMJ6HCD2:NMJ6HCD2
- removed J5: MIDI OUT JACK, AudioConnector-PJ320A:TRRS-PJ-320A, symbol Connector_Audio:AudioJack4
- added J3: AUDIO_IN_RIGHT, GuitarPedal125B:Generic_Pads_AudioTS, symbol Connector_Audio:AudioJack2
- added J4: AUDIO_OUT_LEFT, GuitarPedal125B:Generic_Pads_AudioTS, symbol Connector_Audio:AudioJack2
- added J5: AUDIO_OUT_RIGHT, GuitarPedal125B:Generic_Pads_AudioTS, symbol Connector_Audio:AudioJack2
- added J7: MIDI_OUT, GuitarPedal125B:Generic_Pads_AudioTRS, symbol Connector_Audio:AudioJack3
- added J8, J9: Conn_01x20_Socket, Connector_PinSocket_2.54mm:PinSocket_1x20_P2.54mm_Vertical, symbol Connector:Conn_01x20_Socket
- A1: value Electrosmith_Daisy_Seed_Rev4 -> Electrosmith_Daisy_Seed_Rev7; footprint Module:Electrosmith_Daisy_Seed -> (none); symbol MCU_Module:Electrosmith_Daisy_Seed_Rev4 -> GuitarPedal125B:Electrosmith_Daisy_Seed_Rev7; now left out of the parts list
- J1: value Barrel_Jack_Switch -> POWER_JACK; footprint GuitarPedal125B:Generic_PowerJack -> GuitarPedal125B:Generic_Pads_Power; symbol Connector:Barrel_Jack_Switch -> Connector:Barrel_Jack
- J2: value AUDIO_IN_TRS -> AUDIO_IN_LEFT; footprint NMJ6HCD2:NEUTRIK_NMJ6HCD2 -> GuitarPedal125B:Generic_Pads_AudioTS; symbol NMJ6HCD2:NMJ6HCD2 -> Connector_Audio:AudioJack2
- J6: renamed from J4; value MIDI IN JACK -> MIDI_IN; footprint AudioConnector-PJ320A:TRRS-PJ-320A -> GuitarPedal125B:Generic_Pads_AudioTRS; symbol Connector_Audio:AudioJack4 -> Connector_Audio:AudioJack3
Connections:
- net +3.3V: now also J9.3 (Pin_3)
- net +3.3VA: now also J9.20 (Pin_20)
- net +9V: now also J9.2 (Pin_2)
- net AUDIO_IN_BUFFER_LEFT: now also J8.5 (Pin_5)
- net AUDIO_IN_BUFFER_RIGHT: now also J8.4 (Pin_4)
- net AUDIO_IN_JACK_RIGHT: now also J3.T; no longer J2.R
- net AUDIO_OUT_BUFFER_LEFT: now also J8.3 (Pin_3)
- net AUDIO_OUT_BUFFER_RIGHT: now also J8.2 (Pin_2)
- net AUDIO_OUT_JACK_LEFT: now also J4.T
- net AUDIO_OUT_JACK_RIGHT: now also J5.T
- net DISABLE_AUDIO_BYPASS: now also J8.19 (Pin_19)
- net ENABLE_AUDIO_MUTE: now also J8.8 (Pin_8)
- net ENCODER_1_A: now also J8.18 (Pin_18)
- net ENCODER_1_B: now also J8.17 (Pin_17)
- net ENCODER_1_CLICK: now also J8.16 (Pin_16)
- net FOOT_SWITCH_1: now also J8.14 (Pin_14)
- net FOOT_SWITCH_2: now also J8.15 (Pin_15)
- net GND: now also J3.S, J4.S, J5.S, J7.S, J8.1 (Pin_1), J9.1 (Pin_1); no longer J1.3, J2.RN, J2.SN, J2.TN
- net LED_1: now also J9.12 (Pin_12)
- net LED_2: now also J9.11 (Pin_11)
- net MIDI_IN: now also J9.4 (Pin_4)
- net MIDI_IN_JACK_PIN4: now also J6.R; no longer J6.R1
- net MIDI_OUT: now also J9.5 (Pin_5)
- net MIDI_OUT_JACK_PIN4: now also J7.R
- net MIDI_OUT_JACK_PIN5: now also J7.T
- net OLED_DISPLAY_SPI_CS: now also J8.13 (Pin_13)
- net OLED_DISPLAY_SPI_DC: now also J8.11 (Pin_11)
- net OLED_DISPLAY_SPI_MOSI: now also J8.10 (Pin_10)
- net OLED_DISPLAY_SPI_RESET: now also J8.9 (Pin_9)
- net OLED_DISPLAY_SPI_SCK: now also J8.12 (Pin_12)
- net POT_1: now also J9.19 (Pin_19)
- net POT_2: now also J9.18 (Pin_18)
- net POT_3: now also J9.17 (Pin_17)
- net POT_4: now also J9.16 (Pin_16)
- net POT_5: now also J9.15 (Pin_15)
- net POT_6: now also J9.14 (Pin_14)
- net at A1.1 (USB_ID): now also J8.20 (Pin_20)
- net at A1.14 (USART1_TX): now also J8.7 (Pin_7)
- net at A1.15 (USART1_RX): now also J8.6 (Pin_6)
- net at A1.28 (ADC_6): now also J9.13 (Pin_13)
- net at A1.31 (SAI2_MCLK): now also J9.10 (Pin_10)
- net at A1.32 (SAI2_SD_B): now also J9.9 (Pin_9)
- net at A1.33 (SAI2_SD_A): now also J9.8 (Pin_8)
- net at A1.34 (SAI2_FS): now also J9.7 (Pin_7)
- net at A1.35 (SAI2_SCK): now also J9.6 (Pin_6)
- no-connect marks 11 -> 0
Other:
- moved on the sheet: A1

Commit message: Continuing to work on Rev 6
Parts:
- added J11: Conn_01x05_Pin, Connector_PinHeader_2.54mm:PinHeader_1x05_P2.54mm_Vertical, symbol Connector:Conn_01x05_Pin
- added J12: Conn_01x02_Pin, Connector_PinHeader_2.54mm:PinHeader_1x02_P2.54mm_Vertical, symbol Connector:Conn_01x02_Pin
- added J13: Conn_01x01_Pin, Connector_PinHeader_2.54mm:PinHeader_1x01_P2.54mm_Vertical, symbol Connector:Conn_01x01_Pin
Connections:
- net at A1.1 (USB_ID), J8.20 (Pin_20): now also J13.1 (Pin_1)
- net at A1.14 (USART1_TX), J8.7 (Pin_7): now also J12.1 (Pin_1)
- net at A1.15 (USART1_RX), J8.6 (Pin_6): now also J12.2 (Pin_2)
- net at A1.31 (SAI2_MCLK), J9.10 (Pin_10): now also J11.1 (Pin_1)
- net at A1.32 (SAI2_SD_B), J9.9 (Pin_9): now also J11.2 (Pin_2)
- net at A1.33 (SAI2_SD_A), J9.8 (Pin_8): now also J11.3 (Pin_3)
- net at A1.34 (SAI2_FS), J9.7 (Pin_7): now also J11.4 (Pin_4)
- net at A1.35 (SAI2_SCK), J9.6 (Pin_6): now also J11.5 (Pin_5)
Changed lines of the file:
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@@
   (junction (at 130.81 95.25) (diameter 0) (color 0 0 0 0)
   )
+  (junction (at 64.77 120.65) (diameter 0) (color 0 0 0 0)
+  )
+  (junction (at 64.77 113.03) (diameter 0) (color 0 0 0 0)
+  )
   (junction (at 130.81 120.65) (diameter 0) (color 0 0 0 0)
   )
@@
   (junction (at 64.77 128.27) (diameter 0) (color 0 0 0 0)
   )
+  (junction (at 64.77 110.49) (diameter 0) (color 0 0 0 0)
+  )
   (junction (at 224.79 53.34) (diameter 0) (color 0 0 0 0)
   )
@@
   (junction (at 130.81 90.17) (diameter 0) (color 0 0 0 0)
   )
+  (junction (at 130.81 100.33) (diameter 0) (color 0 0 0 0)
+  )
   (junction (at 64.77 130.81) (diameter 0) (color 0 0 0 0)
   )
@@
   (junction (at 130.81 85.09) (diameter 0) (color 0 0 0 0)
   )
+  (junction (at 64.77 115.57) (diameter 0) (color 0 0 0 0)
+  )
   (junction (at 130.81 107.95) (diameter 0) (color 0 0 0 0)
   )
@@
   (junction (at 64.77 107.95) (diameter 0) (color 0 0 0 0)
   )
+  (junction (at 64.77 118.11) (diameter 0) (color 0 0 0 0)
+  )
   (junction (at 130.81 87.63) (diameter 0) (color 0 0 0 0)
   )
@@
   (junction (at 64.77 123.19) (diameter 0) (color 0 0 0 0)
   )
+  (junction (at 130.81 133.35) (diameter 0) (color 0 0 0 0)
+  )
+  (junction (at 130.81 97.79) (diameter 0) (color 0 0 0 0)
+  )
   (junction (at 130.81 130.81) (diameter 0) (color 0 0 0 0)
   )
@@
     (stroke (width 0) (type default))
   )
+  (wire (pts (xy 130.81 97.79) (xy 138.43 97.79))
+    (stroke (width 0) (type default))
+  )
   (wire (pts (xy 222.25 110.49) (xy 228.6 110.49))
     (stroke (width 0) (type default))
@@
     (stroke (width 0) (type default))
   )
+  (wire (pts (xy 57.15 118.11) (xy 64.77 118.11))
+    (stroke (width 0) (type default))
+  )
   (wire (pts (xy 127 105.41) (xy 130.81 105.41))
     (stroke (width 0) (type default))
@@
     (stroke (width 0) (type default))
   )
+  (wire (pts (xy 57.15 113.03) (xy 64.77 113.03))
+    (stroke (width 0) (type default))
+  )
   (wire (pts (xy 130.81 120.65) (xy 148.59 120.65))
     (stroke (width 0) (type default))
@@
     (stroke (width 0) (type default))
   )
+  (wire (pts (xy 130.81 133.35) (xy 148.59 133.35))
+    (stroke (width 0) (type default))
+  )
   (wire (pts (xy 127 123.19) (xy 130.81 123.19))
     (stroke (width 0) (type default))
   )
+  (wire (pts (xy 57.15 120.65) (xy 64.77 120.65))
+    (stroke (width 0) (type default))
+  )
   (wire (pts (xy 64.77 120.65) (xy 68.58 120.65))
     (stroke (width 0) (type default))
@@
     (stroke (width 0) (type default))
   )
+  (wire (pts (xy 57.15 110.49) (xy 64.77 110.49))
+    (stroke (width 0) (type default))
+  )
   (wire (pts (xy 222.25 97.79) (xy 228.6 97.79))
     (stroke (width 0) (type default))
@@
     (stroke (width 0) (type default))
   )
+  (wire (pts (xy 130.81 100.33) (xy 138.43 100.33))
+    (stroke (width 0) (type default))
+  )
   (wire (pts (xy 25.4 123.19) (xy 25.4 130.81))
     (stroke (width 0) (type default))
@@
   )
   (wire (pts (xy 64.77 113.03) (xy 68.58 113.03))
+    (stroke (width 0) (type default))
+  )
+  (wire (pts (xy 57.15 115.57) (xy 64.77 115.57))
     (stroke (width 0) (type default))
   )
@@
     )
   )
+  (symbol (lib_id "Connector:Conn_01x02_Pin") (at 143.51 100.33 180) (unit 1)
+    (in_bom yes) (on_board yes) (dnp no) (fields_autoplaced)
+    (property "Reference" "J12" (at 144.78 97.79 0)
+      (effects (font (size 1.27 1.27)) (justify right))
+    )
+    (property "Value" "Conn_01x02_Pin" (at 144.78 100.33 0)
+      (effects (font (size 1.27 1.27)) (justify right))
+    )
+    (property "Footprint" "Connector_PinHeader_2.54mm:PinHeader_1x02_P2.54mm_Vertical" (at 143.51 100.33 0)
+      (effects (font (size 1.27 1.27)) hide)
+    )
+    (property "Datasheet" "~" (at 143.51 100.33 0)
+      (effects (font (size 1.27 1.27)) hide)
+    )
+    (pin "1")
+    (pin "2")
+    (instances
+      (project "DaisySeedPedal125b"
+        (path "/1d54e6f4-7c7a-4f03-b2db-a136bdff5b99"
+          (reference "J12") (unit 1)
+        )
+      )
+    )
+  )
   (symbol (lib_id "Connector:Barrel_Jack") (at 214.63 50.8 0) (mirror x) (unit 1)
     (in_bom yes) (on_board yes) (dnp no) (fields_autoplaced)
@@
     )
   )
+  (symbol (lib_id "Connector:Conn_01x05_Pin") (at 52.07 115.57 0) (unit 1)
+    (in_bom yes) (on_board yes) (dnp no)
+    (property "Reference" "J11" (at 49.53 113.03 0)
+      (effects (font (size 1.27 1.27)))
+    )
+    (property "Value" "Conn_01x05_Pin" (at 43.18 115.57 0)
+      (effects (font (size 1.27 1.27)))
+    )
+    (property "Footprint" "Connector_PinHeader_2.54mm:PinHeader_1x05_P2.54mm_Vertical" (at 52.07 115.57 0)
+      (effects (font (size 1.27 1.27)) hide)
+    )
+    (property "Datasheet" "~" (at 52.07 115.57 0)
+      (effects (font (size 1.27 1.27)) hide)
+    )
+    (pin "1")
+    (pin "2")
+    (pin "4")
+    (pin "3")
+    (pin "5")
+    (instances
+      (project "DaisySeedPedal125b"
+        (path "/1d54e6f4-7c7a-4f03-b2db-a136bdff5b99"
+          (reference "J11") (unit 1)
+        )
+      )
+    )
+  )
   (symbol (lib_id "power:+3.3VA") (at 33.02 72.39 0) (unit 1)
     (in_bom yes) (on_board yes) (dnp no)
@@
         )
       )
+    )
+  )
+  (symbol (lib_id "Connector:Conn_01x01_Pin") (at 153.67 133.35 180) (unit 1)
+    (in_bom yes) (on_board yes) (dnp no)
+    (property "Reference" "J13" (at 153.67 138.43 0)
+      (effects (font (size 1.27 1.27)))
+    )
+    (property "Value" "Conn_01x01_Pin" (at 153.67 135.89 0)
+      (effects (font (size 1.27 1.27)))
+    )
+    (property "Footprint" "Connector_PinHeader_2.54mm:PinHeader_1x01_P2.54mm_Vertical" (at 153.67 133.35 0)
+      (effects (font (size 1.27 1.27)) hide)
+    )
+    (property "Datasheet" "~" (at 153.67 133.35 0)
+      (effects (font (size 1.27 1.27)) hide)
+    )
+    (pin "1")
+    (instances
+      (project "DaisySeedPedal125b"
+        (path "/1d54e6f4-7c7a-4f03-b2db-a136bdff5b99"
+          (reference "J13") (unit 1)
+        )
+      )

Commit message: More work on layout
Parts:
- removed J11: Conn_01x05_Pin, Connector_PinHeader_2.54mm:PinHeader_1x05_P2.54mm_Vertical, symbol Connector:Conn_01x05_Pin
- added J11: Conn_01x07_Pin, Connector_PinHeader_2.54mm:PinHeader_1x07_P2.54mm_Vertical, symbol Connector:Conn_01x07_Pin
- J12: value Conn_01x02_Pin -> ALT_POWER_JACK; footprint Connector_PinHeader_2.54mm:PinHeader_1x02_P2.54mm_Vertical -> GuitarPedal125B:Generic_Pads_Power
Connections:
- net GND: now also J12.1 (Pin_1)
- net MIDI_IN: now also A1.15 (USART1_RX), J8.6 (Pin_6); no longer A1.37 (USB_D_+), J9.4 (Pin_4)
- net MIDI_OUT: now also A1.14 (USART1_TX), J8.7 (Pin_7); no longer A1.36 (USB_D_-), J9.5 (Pin_5)
- net POWER_JACK_PWR: now also J12.2 (Pin_2)
- net at A1.31 (SAI2_MCLK), J9.10 (Pin_10): now also J11.1 (Pin_1)
- net at A1.32 (SAI2_SD_B), J9.9 (Pin_9): now also J11.2 (Pin_2)
- net at A1.33 (SAI2_SD_A), J9.8 (Pin_8): now also J11.3 (Pin_3)
- net at A1.34 (SAI2_FS), J9.7 (Pin_7): now also J11.4 (Pin_4)
- net at A1.35 (SAI2_SCK), J9.6 (Pin_6): now also J11.5 (Pin_5)
- new net: A1.36 (USB_D_-), J11.6 (Pin_6), J9.5 (Pin_5)
- new net: A1.37 (USB_D_+), J11.7 (Pin_7), J9.4 (Pin_4)
Changed lines of the file:
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@@
   (junction (at 130.81 120.65) (diameter 0) (color 0 0 0 0)
   )
+  (junction (at 64.77 123.19) (diameter 0) (color 0 0 0 0)
+  )
   (junction (at 64.77 105.41) (diameter 0) (color 0 0 0 0)
   )
@@
   (junction (at 130.81 105.41) (diameter 0) (color 0 0 0 0)
   )
+  (junction (at 130.81 128.27) (diameter 0) (color 0 0 0 0)
+  )
+  (junction (at 130.81 90.17) (diameter 0) (color 0 0 0 0)
+  )
+  (junction (at 130.81 100.33) (diameter 0) (color 0 0 0 0)
+  )
   (junction (at 64.77 125.73) (diameter 0) (color 0 0 0 0)
   )
-  (junction (at 130.81 128.27) (diameter 0) (color 0 0 0 0)
-  )
-  (junction (at 130.81 90.17) (diameter 0) (color 0 0 0 0)
-  )
-  (junction (at 130.81 100.33) (diameter 0) (color 0 0 0 0)
-  )
   (junction (at 64.77 130.81) (diameter 0) (color 0 0 0 0)
   )
@@
   (junction (at 64.77 100.33) (diameter 0) (color 0 0 0 0)
   )
+  (junction (at 222.758 48.26) (diameter 0) (color 0 0 0 0)
+  )
   (junction (at 130.81 115.57) (diameter 0) (color 0 0 0 0)
   )
-  (junction (at 64.77 123.19) (diameter 0) (color 0 0 0 0)
-  )
   (junction (at 130.81 133.35) (diameter 0) (color 0 0 0 0)
   )
@@
     (stroke (width 0) (type default))
   )
-  (wire (pts (xy 130.81 97.79) (xy 138.43 97.79))
-    (stroke (width 0) (type default))
-  )
   (wire (pts (xy 222.25 110.49) (xy 228.6 110.49))
     (stroke (width 0) (type default))
@@
     (stroke (width 0) (type default))
   )
-  (wire (pts (xy 222.25 48.26) (xy 229.87 48.26))
+  (wire (pts (xy 222.25 48.26) (xy 222.758 48.26))
     (stroke (width 0) (type default))
   )
@@
     (stroke (width 0) (type default))
   )
+  (wire (pts (xy 222.758 42.926) (xy 222.758 48.26))
+    (stroke (width 0) (type default))
+  )
   (wire (pts (xy 64.77 110.49) (xy 68.58 110.49))
     (stroke (width 0) (type default))
@@
     (stroke (width 0) (type default))
   )
-  (wire (pts (xy 48.26 123.19) (xy 64.77 123.19))
-    (stroke (width 0) (type default))
-  )
   (wire (pts (xy 127 128.27) (xy 130.81 128.27))
     (stroke (width 0) (type default))
@@
     (stroke (width 0) (type default))
   )
+  (wire (pts (xy 57.15 125.73) (xy 64.77 125.73))
+    (stroke (width 0) (type default))
+  )
   (wire (pts (xy 64.77 130.81) (xy 68.58 130.81))
     (stroke (width 0) (type default))
@@
     (stroke (width 0) (type default))
   )
-  (wire (pts (xy 48.26 125.73) (xy 64.77 125.73))
-    (stroke (width 0) (type default))
-  )
   (wire (pts (xy 127 87.63) (xy 130.81 87.63))
     (stroke (width 0) (type default))
@@
     (stroke (width 0) (type default))
   )
+  (wire (pts (xy 224.79 40.386) (xy 224.79 53.34))
+    (stroke (width 0) (type default))
+  )
   (wire (pts (xy 127 133.35) (xy 130.81 133.35))
     (stroke (width 0) (type default))
@@
     (stroke (width 0) (type default))
   )
+  (wire (pts (xy 57.15 123.19) (xy 64.77 123.19))
+    (stroke (width 0) (type default))
+  )
+  (wire (pts (xy 219.456 42.926) (xy 222.758 42.926))
+    (stroke (width 0) (type default))
+  )
   (wire (pts (xy 222.25 127) (xy 229.87 127))
     (stroke (width 0) (type default))
@@
     (stroke (width 0) (type default))
   )
+  (wire (pts (xy 130.81 100.33) (xy 148.59 100.33))
+    (stroke (width 0) (type default))
+  )
+  (wire (pts (xy 130.81 97.79) (xy 148.59 97.79))
+    (stroke (width 0) (type default))
+  )
   (wire (pts (xy 48.26 107.95) (xy 64.77 107.95))
     (stroke (width 0) (type default))
@@
     (stroke (width 0) (type default))
   )
+  (wire (pts (xy 222.758 48.26) (xy 229.87 48.26))
+    (stroke (width 0) (type default))
+  )
   (wire (pts (xy 130.81 110.49) (xy 148.59 110.49))
     (stroke (width 0) (type default))
@@
     (stroke (width 0) (type default))
   )
-  (wire (pts (xy 130.81 100.33) (xy 138.43 100.33))
-    (stroke (width 0) (type default))
-  )
   (wire (pts (xy 25.4 123.19) (xy 25.4 130.81))
     (stroke (width 0) (type default))
@@
     (stroke (width 0) (type default))
   )
+  (wire (pts (xy 219.456 40.386) (xy 224.79 40.386))
+    (stroke (width 0) (type default))
+  )
   (wire (pts (xy 64.77 113.03) (xy 68.58 113.03))
     (stroke (width 0) (type default))
@@
     )
   )
-  (global_label "MIDI_IN" (shape input) (at 48.26 125.73 180) (fields_autoplaced)
-    (effects (font (size 1.27 1.27)) (justify right))
-    (property "Intersheetrefs" "${INTERSHEET_REFS}" (at 38.4409 125.73 0)
-      (effects (font (size 1.27 1.27)) (justify right) hide)
+  (global_label "MIDI_IN" (shape input) (at 148.59 97.79 0) (fields_autoplaced)
+    (effects (font (size 1.27 1.27)) (justify left))
+    (property "Intersheetrefs" "${INTERSHEET_REFS}" (at 158.4091 97.79 0)
+      (effects (font (size 1.27 1.27)) (justify left) hide)
     )
   )
@@
     )
   )
-  (global_label "MIDI_OUT" (shape output) (at 48.26 123.19 180) (fields_autoplaced)
-    (effects (font (size 1.27 1.27)) (justify right))
-    (property "Intersheetrefs" "${INTERSHEET_REFS}" (at 36.7476 123.19 0)
-      (effects (font (size 1.27 1.27)) (justify right) hide)
+  (global_label "MIDI_OUT" (shape output) (at 148.59 100.33 0) (fields_autoplaced)
+    (effects (font (size 1.27 1.27)) (justify left))
+    (property "Intersheetrefs" "${INTERSHEET_REFS}" (at 160.1024 100.33 0)
+      (effects (font (size 1.27 1.27)) (justify left) hide)
     )
   )
@@
     )
   )
+  (symbol (lib_id "Connector:Conn_01x07_Pin") (at 52.07 118.11 0) (unit 1)
+    (in_bom yes) (on_board yes) (dnp no)
+    (property "Reference" "J11" (at 49.022 121.412 0)
+      (effects (font (size 1.27 1.27)))
+    )
+    (property "Value" "Conn_01x07_Pin" (at 42.926 123.952 0)
+      (effects (font (size 1.27 1.27)))
+    )
+    (property "Footprint" "Connector_PinHeader_2.54mm:PinHeader_1x07_P2.54mm_Vertical" (at 52.07 118.11 0)
+      (effects (font (size 1.27 1.27)) hide)
+    )
+    (property "Datasheet" "~" (at 52.07 118.11 0)
+      (effects (font (size 1.27 1.27)) hide)
+    )
+    (pin "1")
+    (pin "6")
+    (pin "3")
+    (pin "4")
+    (pin "2")
+    (pin "5")
+    (pin "7")
+    (instances
+      (project "DaisySeedPedal125b"
+        (path "/1d54e6f4-7c7a-4f03-b2db-a136bdff5b99"
+          (reference "J11") (unit 1)
+        )
+      )
+    )
+  )
   (symbol (lib_id "Connector_Audio:AudioJack2") (at 217.17 81.28 0) (mirror x) (unit 1)
     (in_bom yes) (on_board yes) (dnp no)
@@
         (path "/1d54e6f4-7c7a-4f03-b2db-a136bdff5b99"
           (reference "#PWR0111") (unit 1)
-        )
-      )
-    )
-  )
-  (symbol (lib_id "Connector:Conn_01x02_Pin") (at 143.51 100.33 180) (unit 1)
-    (in_bom yes) (on_board yes) (dnp no) (fields_autoplaced)
-    (property "Reference" "J12" (at 144.78 97.79 0)
-      (effects (font (size 1.27 1.27)) (justify right))
-    )
-    (property "Value" "Conn_01x02_Pin" (at 144.78 100.33 0)
-      (effects (font (size 1.27 1.27)) (justify right))
-    )
-    (property "Footprint" "Connector_PinHeader_2.54mm:PinHeader_1x02_P2.54mm_Vertical" (at 143.51 100.33 0)
-      (effects (font (size 1.27 1.27)) hide)
-    )
-    (property "Datasheet" "~" (at 143.51 100.33 0)
-      (effects (font (size 1.27 1.27)) hide)
-    )
-    (pin "1")
-    (pin "2")
-    (instances
-      (project "DaisySeedPedal125b"
-        (path "/1d54e6f4-7c7a-4f03-b2db-a136bdff5b99"
-          (reference "J12") (unit 1)
         )
       )
@@
     )
   )
+  (symbol (lib_id "Connector:Conn_01x02_Pin") (at 214.376 40.386 0) (unit 1)
+    (in_bom yes) (on_board yes) (dnp no)
+    (property "Reference" "J12" (at 218.44 34.798 0)
+      (effects (font (size 1.27 1.27)))
+    )
+    (property "Value" "ALT_POWER_JACK" (at 215.011 37.338 0)
+      (effects (font (size 1.27 1.27)))
+    )
+    (property "Footprint" "GuitarPedal125B:Generic_Pads_Power" (at 214.376 40.386 0)
+      (effects (font (size 1.27 1.27)) hide)
+    )
+    (property "Datasheet" "~" (at 214.376 40.386 0)
+      (effects (font (size 1.27 1.27)) hide)
+    )
+    (pin "1")
+    (pin "2")
+    (instances
+      (project "DaisySeedPedal125b"
+        (path "/1d54e6f4-7c7a-4f03-b2db-a136bdff5b99"
+          (reference "J12") (unit 1)
+        )
+      )
+    )
+  )
   (symbol (lib_id "power:GND") (at 222.25 100.33 0) (unit 1)
     (in_bom yes) (on_board yes) (dnp no) (fields_autoplaced)
@@
         )
       )
-    )
-  )
-  (symbol (lib_id "Connector:Conn_01x05_Pin") (at 52.07 115.57 0) (unit 1)
-    (in_bom yes) (on_board yes) (dnp no)
-    (property "Reference" "J11" (at 49.53 113.03 0)
-      (effects (font (size 1.27 1.27)))
-    )
-    (property "Value" "Conn_01x05_Pin" (at 43.18 115.57 0)
-      (effects (font (size 1.27 1.27)))
-    )
-    (property "Footprint" "Connector_PinHeader_2.54mm:PinHeader_1x05_P2.54mm_Vertical" (at 52.07 115.57 0)
-      (effects (font (size 1.27 1.27)) hide)
-    )
-    (property "Datasheet" "~" (at 52.07 115.57 0)
-      (effects (font (size 1.27 1.27)) hide)
-    )
-    (pin "1")
-    (pin "2")
-    (pin "4")
-    (pin "3")
-    (pin "5")
-    (instances
-      (project "DaisySeedPedal125b"
-        (path "/1d54e6f4-7c7a-4f03-b2db-a136bdff5b99"
-          (reference "J11") (unit 1)
-        )
-      )
