File: Hardware/GuitarPedal125b/pcb/DaisySeedPedal125b.kicad_sch (KiCad schematic)
At the start: 6 parts, among them J1 Barrel_Jack_Switch, J2 AUDIO_IN_TRS, J3 AUDIO_OUT_TRS, J4 MIDI IN JACK, J5 MIDI OUT JACK

Commit message: Hardware Rev 6
* Removed PDS1 to reduce cost and because it wasn't really helping anything
* Added low pass filter to address Rev7 Seed Noise issue
* Modified schematics and footprints to make it easier to have assembled by JLCPCB
Parts:
- removed A1: Electrosmith_Daisy_Seed_Rev4, Module:Electrosmith_Daisy_Seed, symbol MCU_Module:Electrosmith_Daisy_Seed_Rev4
- added A1: Electrosmith_Daisy_Seed_Rev7, symbol GuitarPedal125B:Electrosmith_Daisy_Seed_Rev7
- added J6, J7: Conn_01x20_Socket, GuitarPedal125B:PinSocket1x20_P2.54mm_Vertical_JLCPCB, symbol Connector:Conn_01x20_Socket
- J3: renamed from J4; footprint AudioConnector-PJ320A:TRRS-PJ-320A -> GuitarPedal125B:PJ-320A
- J5: footprint AudioConnector-PJ320A:TRRS-PJ-320A -> GuitarPedal125B:PJ-320A
- renumbered J3 to J4
Connections:
- net +3.3V: now also A1.38 (3V3_D), J6.3 (Pin_3)
- net +3.3VA: now also A1.21 (3V3_A), J6.20 (Pin_20)
- net +9V: now also A1.39 (VIN), J6.2 (Pin_2)
- net AUDIO_IN_BUFFER_LEFT: now also A1.16 (AUDIO_IN_1), J7.5 (Pin_5)
- net AUDIO_IN_BUFFER_RIGHT: now also A1.17 (AUDIO_IN_2), J7.4 (Pin_4)
- net AUDIO_OUT_BUFFER_LEFT: now also A1.18 (AUDIO_OUT_1), J7.3 (Pin_3)
- net AUDIO_OUT_BUFFER_RIGHT: now also A1.19 (AUDIO_OUT_2), J7.2 (Pin_2)
- net DISABLE_AUDIO_BYPASS: now also A1.2 (SD_DATA_3), J7.19 (Pin_19)
- net ENABLE_AUDIO_MUTE: now also A1.13 (I2C1_SDA), J7.8 (Pin_8)
- net ENCODER_1_A: now also A1.3 (SD_DATA_2), J7.18 (Pin_18)
- net ENCODER_1_B: now also A1.4 (SD_DATA_1), J7.17 (Pin_17)
- net ENCODER_1_CLICK: now also A1.5 (SD_DATA_0), J7.16 (Pin_16)
- net FOOT_SWITCH_1: now also A1.7 (SD_CLK), J7.14 (Pin_14)
- net FOOT_SWITCH_2: now also A1.6 (SD_CMD), J7.15 (Pin_15)
- net GND: now also A1.20 (AGND), A1.40 (DGND), J6.1 (Pin_1), J7.1 (Pin_1)
- net LED_1: now also A1.29 (DAC_OUT2), J6.12 (Pin_12)
- net LED_2: now also A1.30 (DAC_OUT1), J6.11 (Pin_11)
- net MIDI_IN: now also A1.37 (USB_D_+), J6.4 (Pin_4)
- net MIDI_OUT: now also A1.36 (USB_D_-), J6.5 (Pin_5)
- net OLED_DISPLAY_SPI_CS: now also A1.8 (SPI1_CS), J7.13 (Pin_13)
- net OLED_DISPLAY_SPI_DC: now also A1.10 (SPI1_POCI), J7.11 (Pin_11)
- net OLED_DISPLAY_SPI_MOSI: now also A1.11 (SPI1_PICO), J7.10 (Pin_10)
- net OLED_DISPLAY_SPI_RESET: now also A1.12 (I2C1_SCL), J7.9 (Pin_9)
- net OLED_DISPLAY_SPI_SCK: now also A1.9 (SPI1_SCK), J7.12 (Pin_12)
- net POT_1: now also A1.22 (ADC_0), J6.19 (Pin_19)
- net POT_2: now also A1.23 (ADC_1), J6.18 (Pin_18)
- net POT_3: now also A1.24 (ADC_2), J6.17 (Pin_17)
- net POT_4: now also A1.25 (ADC_3), J6.16 (Pin_16)
- net POT_5: now also A1.26 (ADC_4), J6.15 (Pin_15)
- net POT_6: now also A1.27 (ADC_5), J6.14 (Pin_14)
- new net: A1.1 (USB_ID), J7.20 (Pin_20)
- new net: A1.15 (USART1_RX), J7.6 (Pin_6)
- new net: A1.14 (USART1_TX), J7.7 (Pin_7)
- new net: A1.28 (ADC_6), J6.13 (Pin_13)
- new net: A1.31 (SAI2_MCLK), J6.10 (Pin_10)
- new net: A1.32 (SAI2_SD_B), J6.9 (Pin_9)
- new net: A1.33 (SAI2_SD_A), J6.8 (Pin_8)
- new net: A1.34 (SAI2_FS), J6.7 (Pin_7)
- new net: A1.35 (SAI2_SCK), J6.6 (Pin_6)
