File: Hardware/GuitarPedal125b/pcb/SSD1306_Screen_SPI.kicad_sch (KiCad schematic)
At the start: 1 part, among them U6 OLED_DISPLAY_SSD1306_SPI

Commit message: Hardware Rev 6
* Removed PDS1 to reduce cost and because it wasn't really helping anything
* Added low pass filter to address Rev7 Seed Noise issue
* Modified schematics and footprints to make it easier to have assembled by JLCPCB
Parts:
- renumbered U6 to U7
Changed lines of the file:
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@@
   (title_block
     (title "Daisy Seed Guitar Pedal 125B")
-    (date "2023-06-30")
-    (rev "5")
+    (date "2024-02-25")
+    (rev "6")
     (company "Made by Keith Shepherd (kshep@mac.com)")
   )
@@
   (symbol (lib_id "power:GND") (at 138.43 113.03 0) (unit 1)
     (in_bom yes) (on_board yes) (dnp no) (fields_autoplaced)
-    (property "Reference" "#PWR08" (at 138.43 119.38 0)
+    (property "Reference" "#PWR045" (at 138.43 119.38 0)
       (effects (font (size 1.27 1.27)) hide)
     )
@@
       (project "DaisySeedPedal125b"
         (path "/1d54e6f4-7c7a-4f03-b2db-a136bdff5b99/05a79108-cb22-4356-96de-706d080a4feb"
-          (reference "#PWR08") (unit 1)
+          (reference "#PWR045") (unit 1)
         )
       )
@@
   (symbol (lib_id "GuitarPedal125B:OLED_DISPLAY_SSD1306_SPI") (at 138.43 102.87 0) (unit 1)
     (in_bom yes) (on_board yes) (dnp no)
-    (property "Reference" "U6" (at 137.16 100.33 0)
+    (property "Reference" "U7" (at 137.16 100.33 0)
       (effects (font (size 1.27 1.27)) (justify left))
     )
@@
       (project "DaisySeedPedal125b"
         (path "/1d54e6f4-7c7a-4f03-b2db-a136bdff5b99/05a79108-cb22-4356-96de-706d080a4feb"
-          (reference "U6") (unit 1)
+          (reference "U7") (unit 1)
         )
       )
@@
   (symbol (lib_id "power:+3.3V") (at 138.43 83.82 0) (unit 1)
     (in_bom yes) (on_board yes) (dnp no) (fields_autoplaced)
-    (property "Reference" "#PWR01" (at 138.43 87.63 0)
+    (property "Reference" "#PWR044" (at 138.43 87.63 0)
       (effects (font (size 1.27 1.27)) hide)
     )
@@
       (project "DaisySeedPedal125b"
         (path "/1d54e6f4-7c7a-4f03-b2db-a136bdff5b99/05a79108-cb22-4356-96de-706d080a4feb"
-          (reference "#PWR01") (unit 1)
+          (reference "#PWR044") (unit 1)
         )
       )
