File: Hardware/GuitarPedal125b/pcb/Controls.kicad_sch (KiCad schematic)
At the start: 19 parts

Commit message: Hardware Rev 6
* Removed PDS1 to reduce cost and because it wasn't really helping anything
* Added low pass filter to address Rev7 Seed Noise issue
* Modified schematics and footprints to make it easier to have assembled by JLCPCB
Parts:
- renumbered R19 to R24, R20 to R25, R22 to R26, R23 to R27, R26 to R28, R27 to R29
