File: Hardware/GuitarPedal125b/pcb/Midi_InOut.kicad_sch (KiCad schematic)
At the start: 7 parts, among them U5 H11L1

Commit message: Hardware Rev 6
* Removed PDS1 to reduce cost and because it wasn't really helping anything
* Added low pass filter to address Rev7 Seed Noise issue
* Modified schematics and footprints to make it easier to have assembled by JLCPCB
Parts:
- renumbered R15 to R17, R17 to R18, R16 to R19, R18 to R20, U5 to U4
Changed lines of the file:
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@@
   (title_block
     (title "Daisy Seed Guitar Pedal 125B")
-    (date "2023-06-30")
-    (rev "5")
+    (date "2024-02-25")
+    (rev "6")
     (company "Made by Keith Shepherd (kshep@mac.com)")
     (comment 1 "https://diyelectromusic.wordpress.com/2022/08/29/3v3-midi-module-pcb/")
@@
   (symbol (lib_id "Device:R") (at 116.84 91.44 90) (unit 1)
     (in_bom yes) (on_board yes) (dnp no) (fields_autoplaced)
-    (property "Reference" "R15" (at 116.84 85.09 90)
+    (property "Reference" "R17" (at 116.84 85.09 90)
       (effects (font (size 1.27 1.27)))
     )
@@
       (project "DaisySeedPedal125b"
         (path "/1d54e6f4-7c7a-4f03-b2db-a136bdff5b99/9c4d00d6-afa1-4803-8527-08af930a10bd"
-          (reference "R15") (unit 1)
+          (reference "R17") (unit 1)
         )
       )
@@
   (symbol (lib_id "power:+3.3V") (at 144.78 80.01 0) (unit 1)
     (in_bom yes) (on_board yes) (dnp no) (fields_autoplaced)
-    (property "Reference" "#PWR022" (at 144.78 83.82 0)
+    (property "Reference" "#PWR033" (at 144.78 83.82 0)
       (effects (font (size 1.27 1.27)) hide)
     )
@@
       (project "DaisySeedPedal125b"
         (path "/1d54e6f4-7c7a-4f03-b2db-a136bdff5b99/9c4d00d6-afa1-4803-8527-08af930a10bd"
-          (reference "#PWR022") (unit 1)
+          (reference "#PWR033") (unit 1)
         )
       )
@@
   (symbol (lib_id "Device:R") (at 139.7 135.89 270) (unit 1)
     (in_bom yes) (on_board yes) (dnp no) (fields_autoplaced)
-    (property "Reference" "R16" (at 139.7 142.24 90)
+    (property "Reference" "R19" (at 139.7 142.24 90)
       (effects (font (size 1.27 1.27)))
     )
@@
       (project "DaisySeedPedal125b"
         (path "/1d54e6f4-7c7a-4f03-b2db-a136bdff5b99/9c4d00d6-afa1-4803-8527-08af930a10bd"
-          (reference "R16") (unit 1)
+          (reference "R19") (unit 1)
         )
       )
@@
   (symbol (lib_id "Device:R") (at 166.37 87.63 0) (unit 1)
     (in_bom yes) (on_board yes) (dnp no) (fields_autoplaced)
-    (property "Reference" "R18" (at 168.91 86.3599 0)
+    (property "Reference" "R20" (at 168.91 86.3599 0)
       (effects (font (size 1.27 1.27)) (justify left))
     )
@@
       (project "DaisySeedPedal125b"
         (path "/1d54e6f4-7c7a-4f03-b2db-a136bdff5b99/9c4d00d6-afa1-4803-8527-08af930a10bd"
-          (reference "R18") (unit 1)
+          (reference "R20") (unit 1)
         )
       )
@@
   (symbol (lib_id "power:GND") (at 144.78 102.87 0) (unit 1)
     (in_bom yes) (on_board yes) (dnp no) (fields_autoplaced)
-    (property "Reference" "#PWR023" (at 144.78 109.22 0)
+    (property "Reference" "#PWR034" (at 144.78 109.22 0)
       (effects (font (size 1.27 1.27)) hide)
     )
@@
       (project "DaisySeedPedal125b"
         (path "/1d54e6f4-7c7a-4f03-b2db-a136bdff5b99/9c4d00d6-afa1-4803-8527-08af930a10bd"
-          (reference "#PWR023") (unit 1)
+          (reference "#PWR034") (unit 1)
         )
       )
@@
   (symbol (lib_id "power:GND") (at 184.15 87.63 0) (unit 1)
     (in_bom yes) (on_board yes) (dnp no) (fields_autoplaced)
-    (property "Reference" "#PWR021" (at 184.15 93.98 0)
+    (property "Reference" "#PWR035" (at 184.15 93.98 0)
       (effects (font (size 1.27 1.27)) hide)
     )
@@
       (project "DaisySeedPedal125b"
         (path "/1d54e6f4-7c7a-4f03-b2db-a136bdff5b99/9c4d00d6-afa1-4803-8527-08af930a10bd"
-          (reference "#PWR021") (unit 1)
+          (reference "#PWR035") (unit 1)
         )
       )
@@
   (symbol (lib_id "Isolator:H11L1") (at 144.78 95.25 0) (unit 1)
     (in_bom yes) (on_board yes) (dnp no) (fields_autoplaced)
-    (property "Reference" "U5" (at 154.94 90.805 0)
+    (property "Reference" "U4" (at 154.94 90.805 0)
       (effects (font (size 1.27 1.27)))
     )
@@
       (project "DaisySeedPedal125b"
         (path "/1d54e6f4-7c7a-4f03-b2db-a136bdff5b99/9c4d00d6-afa1-4803-8527-08af930a10bd"
-          (reference "U5") (unit 1)
+          (reference "U4") (unit 1)
         )
       )
@@
   (symbol (lib_id "power:+3.3V") (at 130.81 134.62 0) (unit 1)
     (in_bom yes) (on_board yes) (dnp no) (fields_autoplaced)
-    (property "Reference" "#PWR024" (at 130.81 138.43 0)
+    (property "Reference" "#PWR032" (at 130.81 138.43 0)
       (effects (font (size 1.27 1.27)) hide)
     )
@@
       (project "DaisySeedPedal125b"
         (path "/1d54e6f4-7c7a-4f03-b2db-a136bdff5b99/9c4d00d6-afa1-4803-8527-08af930a10bd"
-          (reference "#PWR024") (unit 1)
+          (reference "#PWR032") (unit 1)
         )
       )
@@
   (symbol (lib_id "Device:R") (at 139.7 123.19 270) (unit 1)
     (in_bom yes) (on_board yes) (dnp no) (fields_autoplaced)
-    (property "Reference" "R17" (at 139.7 129.54 90)
+    (property "Reference" "R18" (at 139.7 129.54 90)
       (effects (font (size 1.27 1.27)))
     )
@@
       (project "DaisySeedPedal125b"
         (path "/1d54e6f4-7c7a-4f03-b2db-a136bdff5b99/9c4d00d6-afa1-4803-8527-08af930a10bd"
-          (reference "R17") (unit 1)
-        )
-      )
+          (reference "R18") (unit 1)
+        )
+      )
